File: kicad-pcbs/adxi/lpf-10m-smt.kicad_sch (KiCad schematic)
At the start: 18 parts

Commit message: More bands
Parts:
- renumbered C31 to C30, C30 to C31, L15 to L5, L16 to L6, L17 to L7, L10 to L8, L11 to L9
Changed lines of the file:
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@@
 		(on_board yes)
 		(dnp no)
-		(property "Reference" "L10"
+		(property "Reference" "L8"
 			(at 99.822 80.01 90)
 			(effects
@@
 			(project "adxi"
 				(path "/c3abf330-1856-4368-a03b-0e6191ae29a9/4bed0468-3ef3-43ae-86cd-7d15afd655b3"
-					(reference "L10")
+					(reference "L8")
 					(unit 1)
 				)
@@
 		(dnp no)
 		(fields_autoplaced yes)
-		(property "Reference" "L16"
+		(property "Reference" "L6"
 			(at 78.74 80.01 90)
 			(effects
@@
 			(project "adxi"
 				(path "/c3abf330-1856-4368-a03b-0e6191ae29a9/4bed0468-3ef3-43ae-86cd-7d15afd655b3"
-					(reference "L16")
+					(reference "L6")
 					(unit 1)
 				)
@@
 		(dnp no)
 		(fields_autoplaced yes)
-		(property "Reference" "L17"
+		(property "Reference" "L7"
 			(at 86.36 80.01 90)
 			(effects
@@
 			(project "adxi"
 				(path "/c3abf330-1856-4368-a03b-0e6191ae29a9/4bed0468-3ef3-43ae-86cd-7d15afd655b3"
-					(reference "L17")
+					(reference "L7")
 					(unit 1)
 				)
@@
 		(dnp no)
 		(fields_autoplaced yes)
-		(property "Reference" "C31"
+		(property "Reference" "C30"
 			(at 121.92 87.6362 0)
 			(effects
@@
 			(project "adxi"
 				(path "/c3abf330-1856-4368-a03b-0e6191ae29a9/4bed0468-3ef3-43ae-86cd-7d15afd655b3"
-					(reference "C31")
+					(reference "C30")
 					(unit 1)
 				)
@@
 		(dnp no)
 		(fields_autoplaced yes)
-		(property "Reference" "C30"
+		(property "Reference" "C31"
 			(at 132.08 87.6362 0)
 			(effects
@@
 			(project "adxi"
 				(path "/c3abf330-1856-4368-a03b-0e6191ae29a9/4bed0468-3ef3-43ae-86cd-7d15afd655b3"
-					(reference "C30")
+					(reference "C31")
 					(unit 1)
 				)
@@
 		(dnp no)
 		(fields_autoplaced yes)
-		(property "Reference" "L15"
+		(property "Reference" "L5"
 			(at 71.12 80.01 90)
 			(effects
@@
 		)
 		(pin "1"
+		)
+		(instances
+			(project ""
+				(path "/c3abf330-1856-4368-a03b-0e6191ae29a9/4bed0468-3ef3-43ae-86cd-7d15afd655b3"
+					(reference "L5")
+					(unit 1)
+				)
+			)
 		)
 	)
@@
 		(on_board yes)
 		(dnp no)
-		(property "Reference" "L11"
+		(property "Reference" "L9"
 			(at 107.442 80.01 90)
 			(effects
@@
 			(project "adxi"
 				(path "/c3abf330-1856-4368-a03b-0e6191ae29a9/4bed0468-3ef3-43ae-86cd-7d15afd655b3"
-					(reference "L11")
-					(unit 1)
-				)
+					(reference "L9")
+					(unit 1)
+				)
