File: kicad-pcbs/adxi/lpf-12m-smt.kicad_sch (KiCad schematic)
At the start: 12 parts

Commit message: More bands
Parts:
- removed C86, C87: 1pF, Capacitor_SMD:C_1206_3216Metric, symbol Device:C_Small
- removed D68, D69: 13V 5W, Diode_SMD:D_0603_1608Metric, symbol Diode:SD15_SOD323
- added C79, C80: 1pF, Capacitor_SMD:C_1206_3216Metric, symbol Device:C_Small
- added D72, D73: 13V 5W, Diode_SMD:D_0603_1608Metric, symbol Diode:SD15_SOD323
- renumbered L14 to L34
Connections:
- net GND: now also C79.2, C80.2, D72.1 (A1), D73.1 (A1)
- net INPUT: now also D70.2 (A2), D71.2 (A2)
- net OUTPUT: now also C79.1, C80.1, D72.2 (A2), D73.2 (A2); no longer D70.2 (A2), D71.2 (A2)
