File: kicad-pcbs/adxi/lpf-15m-smt.kicad_sch (KiCad schematic)
At the start: 11 parts

Commit message: More bands
Parts:
- renumbered C64 to C56, C52 to C57, C53 to C58, C54 to C59, L22 to L14, L23 to L15
