File: kicad-pcbs/adxi/lpf-17m-smt.kicad_sch (KiCad schematic)
At the start: 7 parts

Commit message: More bands
Parts:
- renumbered C55 to C74, C68 to C75, L13 to L32
Changed lines of the file:
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@@
 		(dnp no)
 		(fields_autoplaced yes)
-		(property "Reference" "L13"
+		(property "Reference" "L32"
 			(at 133.35 87.63 90)
 			(effects
@@
 			(project ""
 				(path "/c3abf330-1856-4368-a03b-0e6191ae29a9/f4e82807-25d6-477e-92aa-6d05f3573797"
-					(reference "L13")
+					(reference "L32")
 					(unit 1)
 				)
@@
 		(dnp no)
 		(fields_autoplaced yes)
-		(property "Reference" "C55"
+		(property "Reference" "C74"
 			(at 143.51 95.2562 0)
 			(effects
@@
 			(project "adxi"
 				(path "/c3abf330-1856-4368-a03b-0e6191ae29a9/f4e82807-25d6-477e-92aa-6d05f3573797"
-					(reference "C55")
+					(reference "C74")
 					(unit 1)
 				)
@@
 		(dnp no)
 		(fields_autoplaced yes)
-		(property "Reference" "C68"
+		(property "Reference" "C75"
 			(at 153.67 95.2562 0)
 			(effects
@@
 			(project "adxi"
 				(path "/c3abf330-1856-4368-a03b-0e6191ae29a9/f4e82807-25d6-477e-92aa-6d05f3573797"
-					(reference "C68")
+					(reference "C75")
 					(unit 1)
 				)
