File: kicad-pcbs/adxi/lpf-20m-smt.kicad_sch (KiCad schematic)
At the start: 11 parts

Commit message: More bands
Parts:
- renumbered C48 to C43, C49 to C44, C46 to C45, C47 to C46, C44 to C47, C50 to C48, L8 to L11
Changed lines of the file:
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@@
 		(dnp no)
 		(fields_autoplaced yes)
-		(property "Reference" "C46"
+		(property "Reference" "C45"
 			(at 147.32 91.4462 0)
 			(effects
@@
 			(project "adxi"
 				(path "/c3abf330-1856-4368-a03b-0e6191ae29a9/c4c14f2a-5eed-4fbd-84fc-7dedf7e1d431"
-					(reference "C46")
+					(reference "C45")
 					(unit 1)
 				)
@@
 		(dnp no)
 		(fields_autoplaced yes)
-		(property "Reference" "C47"
+		(property "Reference" "C46"
 			(at 156.21 91.4462 0)
 			(effects
@@
 			(project "adxi"
 				(path "/c3abf330-1856-4368-a03b-0e6191ae29a9/c4c14f2a-5eed-4fbd-84fc-7dedf7e1d431"
-					(reference "C47")
+					(reference "C46")
 					(unit 1)
 				)
@@
 		(dnp no)
 		(fields_autoplaced yes)
-		(property "Reference" "C44"
+		(property "Reference" "C47"
 			(at 165.1 91.4462 0)
 			(effects
@@
 			(project "adxi"
 				(path "/c3abf330-1856-4368-a03b-0e6191ae29a9/c4c14f2a-5eed-4fbd-84fc-7dedf7e1d431"
-					(reference "C44")
+					(reference "C47")
 					(unit 1)
 				)
@@
 		(dnp no)
 		(fields_autoplaced yes)
-		(property "Reference" "C49"
+		(property "Reference" "C44"
 			(at 137.16 91.4462 0)
 			(effects
@@
 			(project "adxi"
 				(path "/c3abf330-1856-4368-a03b-0e6191ae29a9/c4c14f2a-5eed-4fbd-84fc-7dedf7e1d431"
-					(reference "C49")
+					(reference "C44")
 					(unit 1)
 				)
@@
 		(dnp no)
 		(fields_autoplaced yes)
-		(property "Reference" "C50"
+		(property "Reference" "C48"
 			(at 173.99 91.4462 0)
 			(effects
@@
 			(project "adxi"
 				(path "/c3abf330-1856-4368-a03b-0e6191ae29a9/c4c14f2a-5eed-4fbd-84fc-7dedf7e1d431"
-					(reference "C50")
+					(reference "C48")
 					(unit 1)
 				)
@@
 		(dnp no)
 		(fields_autoplaced yes)
-		(property "Reference" "L8"
+		(property "Reference" "L11"
 			(at 115.57 83.82 90)
 			(effects
@@
 			(project ""
 				(path "/c3abf330-1856-4368-a03b-0e6191ae29a9/c4c14f2a-5eed-4fbd-84fc-7dedf7e1d431"
-					(reference "L8")
+					(reference "L11")
 					(unit 1)
 				)
@@
 		(dnp no)
 		(fields_autoplaced yes)
-		(property "Reference" "C48"
+		(property "Reference" "C43"
 			(at 127 91.4462 0)
 			(effects
@@
 			(project "adxi"
 				(path "/c3abf330-1856-4368-a03b-0e6191ae29a9/c4c14f2a-5eed-4fbd-84fc-7dedf7e1d431"
-					(reference "C48")
+					(reference "C43")
 					(unit 1)
 				)
