File: kicad-pcbs/adxi/lpf-2m-smt.kicad_sch (KiCad schematic)
At the start: 9 parts

Commit message: More bands
Parts:
- removed C51: 1pF, Capacitor_SMD:C_1206_3216Metric, symbol Device:C_Small
- added C42: 1pF, Capacitor_SMD:C_1206_3216Metric, symbol Device:C_Small
- renumbered L6 to L10
Connections:
- net GND: now also C42.2
- net OUTPUT: now also C42.1
