File: kicad-pcbs/adxi/lpf-30m-smt.kicad_sch (KiCad schematic)
At the start: 10 parts

Commit message: More bands
Parts:
- renumbered C63 to C70, C66 to C71, C67 to C72, C65 to C73, L7 to L30, L12 to L31
