File: kicad-pcbs/adxi/lpf-40m-smt.kicad_sch (KiCad schematic)
At the start: 10 parts

Commit message: More bands
Parts:
- renumbered C56 to C49, C45 to C50, C57 to C51, C58 to C52, C59 to C53, L5 to L12
Changed lines of the file:
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@@
 		(dnp no)
 		(fields_autoplaced yes)
-		(property "Reference" "C57"
+		(property "Reference" "C51"
 			(at 147.32 101.6062 0)
 			(effects
@@
 			(project "adxi"
 				(path "/c3abf330-1856-4368-a03b-0e6191ae29a9/8c898856-4b06-4fe5-9f12-ccd8c8eabd99"
-					(reference "C57")
+					(reference "C51")
 					(unit 1)
 				)
@@
 		(dnp no)
 		(fields_autoplaced yes)
-		(property "Reference" "C56"
+		(property "Reference" "C49"
 			(at 137.16 101.6062 0)
 			(effects
@@
 			(project "adxi"
 				(path "/c3abf330-1856-4368-a03b-0e6191ae29a9/8c898856-4b06-4fe5-9f12-ccd8c8eabd99"
-					(reference "C56")
+					(reference "C49")
 					(unit 1)
 				)
@@
 		(dnp no)
 		(fields_autoplaced yes)
-		(property "Reference" "C59"
+		(property "Reference" "C53"
 			(at 167.64 101.6062 0)
 			(effects
@@
 			(project "adxi"
 				(path "/c3abf330-1856-4368-a03b-0e6191ae29a9/8c898856-4b06-4fe5-9f12-ccd8c8eabd99"
-					(reference "C59")
+					(reference "C53")
 					(unit 1)
 				)
@@
 		(dnp no)
 		(fields_autoplaced yes)
-		(property "Reference" "L5"
+		(property "Reference" "L12"
 			(at 134.62 87.63 90)
 			(effects
@@
 			(project ""
 				(path "/c3abf330-1856-4368-a03b-0e6191ae29a9/8c898856-4b06-4fe5-9f12-ccd8c8eabd99"
-					(reference "L5")
+					(reference "L12")
 					(unit 1)
 				)
@@
 		(dnp no)
 		(fields_autoplaced yes)
-		(property "Reference" "C58"
+		(property "Reference" "C52"
 			(at 157.48 101.6062 0)
 			(effects
@@
 			(project "adxi"
 				(path "/c3abf330-1856-4368-a03b-0e6191ae29a9/8c898856-4b06-4fe5-9f12-ccd8c8eabd99"
-					(reference "C58")
+					(reference "C52")
 					(unit 1)
 				)
@@
 		(dnp no)
 		(fields_autoplaced yes)
-		(property "Reference" "C45"
+		(property "Reference" "C50"
 			(at 147.32 95.2562 0)
 			(effects
@@
 			(project ""
 				(path "/c3abf330-1856-4368-a03b-0e6191ae29a9/8c898856-4b06-4fe5-9f12-ccd8c8eabd99"
-					(reference "C45")
+					(reference "C50")
 					(unit 1)
 				)
