File: kicad-pcbs/adxi/lpf-60m-smt.kicad_sch (KiCad schematic)
At the start: 27 parts

Commit message: More bands
Parts:
- renumbered C70 to C62, C62 to C63, C72 to C64, C73 to C65, C74 to C66, C75 to C67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
