File: kicad-pcbs/adxi/lpf-6m-smt.kicad_sch (KiCad schematic)
At the start: 8 parts

Commit message: More bands
Parts:
- renumbered C69 to C76, C71 to C77, C79 to C78, D62 to D64, D63 to D65, D64 to D66, D65 to D67, L18 to L33
Changed lines of the file:
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@@
 		(dnp no)
 		(fields_autoplaced yes)
-		(property "Reference" "C79"
+		(property "Reference" "C78"
 			(at 162.56 99.0662 0)
 			(effects
@@
 			(project "adxi"
 				(path "/c3abf330-1856-4368-a03b-0e6191ae29a9/89243ecd-733d-4cae-bfd5-43b5bae8c7f3"
-					(reference "C79")
+					(reference "C78")
 					(unit 1)
 				)
@@
 		(dnp no)
 		(fields_autoplaced yes)
-		(property "Reference" "C71"
+		(property "Reference" "C77"
 			(at 152.4 99.0662 0)
 			(effects
@@
 			(project "adxi"
 				(path "/c3abf330-1856-4368-a03b-0e6191ae29a9/89243ecd-733d-4cae-bfd5-43b5bae8c7f3"
-					(reference "C71")
+					(reference "C77")
 					(unit 1)
 				)
@@
 		(on_board yes)
 		(dnp no)
-		(property "Reference" "D65"
+		(property "Reference" "D67"
 			(at 186.69 99.06 90)
 			(effects
@@
 			(project "adxi"
 				(path "/c3abf330-1856-4368-a03b-0e6191ae29a9/89243ecd-733d-4cae-bfd5-43b5bae8c7f3"
-					(reference "D65")
+					(reference "D67")
 					(unit 1)
 				)
@@
 		(on_board yes)
 		(dnp no)
-		(property "Reference" "D62"
+		(property "Reference" "D64"
 			(at 111.76 99.06 90)
 			(effects
@@
 			(project "adxi"
 				(path "/c3abf330-1856-4368-a03b-0e6191ae29a9/89243ecd-733d-4cae-bfd5-43b5bae8c7f3"
-					(reference "D62")
+					(reference "D64")
 					(unit 1)
 				)
@@
 		(on_board yes)
 		(dnp no)
-		(property "Reference" "D64"
+		(property "Reference" "D66"
 			(at 175.26 99.06 90)
 			(effects
@@
 			(project "adxi"
 				(path "/c3abf330-1856-4368-a03b-0e6191ae29a9/89243ecd-733d-4cae-bfd5-43b5bae8c7f3"
-					(reference "D64")
+					(reference "D66")
 					(unit 1)
 				)
@@
 		(on_board yes)
 		(dnp no)
-		(property "Reference" "D63"
+		(property "Reference" "D65"
 			(at 123.19 99.06 90)
 			(effects
@@
 			(project "adxi"
 				(path "/c3abf330-1856-4368-a03b-0e6191ae29a9/89243ecd-733d-4cae-bfd5-43b5bae8c7f3"
-					(reference "D63")
+					(reference "D65")
 					(unit 1)
 				)
@@
 		(dnp no)
 		(fields_autoplaced yes)
-		(property "Reference" "L18"
+		(property "Reference" "L33"
 			(at 129.54 91.44 90)
 			(effects
@@
 			(project "adxi"
 				(path "/c3abf330-1856-4368-a03b-0e6191ae29a9/89243ecd-733d-4cae-bfd5-43b5bae8c7f3"
-					(reference "L18")
+					(reference "L33")
 					(unit 1)
 				)
@@
 		(dnp no)
 		(fields_autoplaced yes)
-		(property "Reference" "C69"
+		(property "Reference" "C76"
 			(at 142.24 99.0662 0)
 			(effects
@@
 			(project "adxi"
 				(path "/c3abf330-1856-4368-a03b-0e6191ae29a9/89243ecd-733d-4cae-bfd5-43b5bae8c7f3"
-					(reference "C69")
+					(reference "C76")
 					(unit 1)
 				)
