File: kicad-pcbs/adxi/lpf-160m-smt.kicad_sch (KiCad schematic)
At the start: 4 parts

Commit message: More bands
Parts:
- added C87: 680pF, Capacitor_SMD:C_1206_3216Metric, symbol Device:C_Small
- added L36: 100nH, Inductor_SMD:L_1008_2520Metric, symbol Device:L
- renumbered D74 to D76, D75 to D77, D76 to D78, D77 to D79
Connections:
- net GND: now also C87.2
- net INPUT: now also L36.1
- net OUTPUT: now also C87.1, L36.2
Other:
- note added: "2% SRF>1GHz, DCR=0.56, I=650mA, Q=45@F, V=?"
- note added: "Inductor (L): 100 nH Capacitor (C): 680 pF"
- note removed: "?% SRF=?MHz, DCR=?, I=?, Q=?"
- note removed: "Inductor (L): x uH Capacitor (C): x pF"

Commit message: Updates
Parts:
- renumbered C87 to C86, L36 to L35
