File: kicad-pcbs/adxi/lpf-2200m-smt.kicad_sch (KiCad schematic)
At the start: 4 parts

Commit message: More bands
Parts:
- removed D86, D87: 13V 5W, Diode_SMD:D_0603_1608Metric, symbol Diode:SD15_SOD323
- added C89: 100nF, Capacitor_SMD:C_1206_3216Metric, symbol Device:C_Small
- added D90, D91: 13V 5W, Diode_SMD:D_0603_1608Metric, symbol Diode:SD15_SOD323
- added L38: 100nH, Inductor_SMD:L_1008_2520Metric, symbol Device:L
Connections:
- net GND: now also C89.2, D90.1 (A1), D91.1 (A1)
- net INPUT: now also D88.2 (A2), D89.2 (A2), L38.1
- net OUTPUT: now also C89.1, D90.2 (A2), D91.2 (A2), L38.2; no longer D88.2 (A2), D89.2 (A2)
Other:
- note added: "2% SRF>1GHz, DCR=0.56, I=650mA, Q=45@F"
- note added: "Inductor (L): 100 nH Capacitor (C): 100 nF"
- note removed: "?% SRF=?MHz, DCR=?, I=?, Q=?"
- note removed: "Inductor (L): x uH Capacitor (C): x pF"

Commit message: Updates
Parts:
- renumbered C89 to C88, L38 to L37
Changed lines of the file:
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@@
 		(on_board yes)
 		(dnp no)
-		(property "Reference" "C89"
+		(property "Reference" "C88"
 			(at 156.21 96.5262 0)
 			(effects
@@
 			(project ""
 				(path "/c3abf330-1856-4368-a03b-0e6191ae29a9/01440e7e-6957-4f7e-93d9-c375eb2e2686"
-					(reference "C89")
+					(reference "C88")
 					(unit 1)
 				)
@@
 		(on_board yes)
 		(dnp no)
-		(property "Reference" "L38"
+		(property "Reference" "L37"
 			(at 135.89 91.694 90)
 			(effects
@@
 			(project "adxi"
 				(path "/c3abf330-1856-4368-a03b-0e6191ae29a9/01440e7e-6957-4f7e-93d9-c375eb2e2686"
-					(reference "L38")
+					(reference "L37")
 					(unit 1)
 				)
