File: kicad-pcbs/adxi/lpf-630m-smt.kicad_sch (KiCad schematic)
At the start: 6 parts

Commit message: Updates
Parts:
- renumbered C88 to C87, L37 to L36
Changed lines of the file:
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@@
 		(on_board yes)
 		(dnp no)
-		(property "Reference" "L37"
+		(property "Reference" "L36"
 			(at 135.89 91.694 90)
 			(effects
@@
 			(project "adxi"
 				(path "/c3abf330-1856-4368-a03b-0e6191ae29a9/45b077a6-c9ac-48b9-a42a-6627340441cd"
-					(reference "L37")
+					(reference "L36")
 					(unit 1)
 				)
@@
 		(on_board yes)
 		(dnp no)
-		(property "Reference" "C88"
+		(property "Reference" "C87"
 			(at 156.21 96.5262 0)
 			(effects
@@
 			(project ""
 				(path "/c3abf330-1856-4368-a03b-0e6191ae29a9/45b077a6-c9ac-48b9-a42a-6627340441cd"
-					(reference "C88")
+					(reference "C87")
 					(unit 1)
 				)
