File: kicad-pcbs/adxi/lpf-70cm-smt.kicad_sch (KiCad schematic)
At the start: 6 parts

Commit message: More bands
Parts:
- removed C88: 1nF, Capacitor_SMD:C_1206_3216Metric, symbol Device:C_Small
- removed D82, D83, D84, D85: 13V 5W, Diode_SMD:D_0603_1608Metric, symbol Diode:SD15_SOD323
- removed L37: 100nH, Inductor_SMD:L_1008_2520Metric, symbol Device:L
- added C86: 6.8pF, Capacitor_SMD:C_0805_2012Metric, symbol Device:C_Small
- added D94, D95, D96, D97: 13V 5W, Diode_SMD:D_0603_1608Metric, symbol Diode:SD15_SOD323
- added L35: 100nH, Inductor_SMD:L_1008_2520Metric, symbol Device:L
Connections:
- net GND: now also C86.2, D94.1 (A1), D95.1 (A1), D96.1 (A1), D97.1 (A1)
- net INPUT: now also D94.2 (A2), D95.2 (A2), L35.1
- net OUTPUT: now also C86.1, D96.2 (A2), D97.2 (A2), L35.2
Other:
- note added: "2% SRF>1GHz, DCR=0.56, I=650mA, Q=45@F, V=?"
- note added: "70CM Band (420-450MHz)"
- note added: "Inductor (L): 100 nH Capacitor (C): 6.8 pF"
- note removed: "2% SRF>1GHz, DCR=0.56, I=650mA, Q=45@F"
- note removed: "630M Band (472-479 KHz)"
- note removed: "Inductor (L): 100 nH Capacitor (C): 1 nF"

Commit message: Updates
Parts:
- renumbered C86 to C89, L35 to L38
Changed lines of the file:
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@@
 		(on_board yes)
 		(dnp no)
-		(property "Reference" "C86"
+		(property "Reference" "C89"
 			(at 156.21 96.5262 0)
 			(effects
@@
 			(project ""
 				(path "/c3abf330-1856-4368-a03b-0e6191ae29a9/44dd9bca-6161-4d06-84e0-0f48363b8396"
-					(reference "C86")
+					(reference "C89")
 					(unit 1)
 				)
@@
 		(on_board yes)
 		(dnp no)
-		(property "Reference" "L35"
+		(property "Reference" "L38"
 			(at 135.89 91.694 90)
 			(effects
@@
 			(project "adxi"
 				(path "/c3abf330-1856-4368-a03b-0e6191ae29a9/44dd9bca-6161-4d06-84e0-0f48363b8396"
-					(reference "L35")
+					(reference "L38")
 					(unit 1)
 				)
