File: kicad-pcbs/adxi/adxi.kicad_sch (KiCad schematic)
At the start: 143 parts, among them J1 FROM-PC-SPK, J2 TO-PC-MIC, J3 12V SUPPLY, J4 Conn_Coaxial, J5 Conn_Coaxial_Small, Q1 MMBF170, Q2 MMBF170, Q3 MMBF170, Q4 MMBF170, SW1 UP, SW2 DOWN, SW3 TRANSMIT, U1 CD2003, U2 Si5351A-B-GT, U3 74ACT244, U4 L7812

Commit message: LPFs, footprints, component selection, switching
Parts:
- removed C33, C34, C35, C37, C38, C39, C40, C41, C42, C43, C47, C48, C49, C50, C51, C52, C53, C54, C55: 1pF, Capacitor_SMD:C_1206_3216Metric, symbol Device:C_Small
- removed C36: 0.47pF, Capacitor_SMD:C_1206_3216Metric, symbol Device:C_Small
- removed C44, C45, C46: 10pF, Capacitor_SMD:C_1206_3216Metric, symbol Device:C_Small
- removed C56, C57, C58: 33pF, Capacitor_SMD:C_1206_3216Metric, symbol Device:C_Small
- removed D1, D19, D2, D20, D25, D26, D27, D28, D29, D3, D30, D4, D5: LED, Resistor_SMD:R_0805_2012Metric, symbol Device:LED
- removed D10, D11, D12, D13, D14, D15, D16, D17, D8, D9: 24V 1ns, Diode_SMD:D_0603_1608Metric, symbol Diode:SD15_SOD323
- removed L10: 100nH, Inductor_SMD:L_0603_1608Metric, symbol Device:L
- removed L3, L5, L6: 2.2uH, Inductor_SMD:L_1008_2520Metric, symbol Device:L
- removed L4: 560nH, Inductor_SMD:L_1008_2520Metric, symbol Device:L
- removed L7: 4.7uH, Inductor_SMD:L_Vishay_IFSC-1515AH_4x4x1.8mm, symbol Device:L
- removed Q1, Q2, Q3: MMBF170, Package_TO_SOT_SMD:SOT-23, symbol Transistor_FET:MMBF170
- removed R11, R12, R14, R15, R19, R20, R25, R26, R27, R28, R29, R30: 120, Resistor_SMD:R_0805_2012Metric, symbol Device:R_Small_US
- removed R5, R6, R7: 10K, Resistor_SMD:R_1206_3216Metric, symbol Device:R_Small_US
- removed SW1: UP, symbol Switch:SW_Push
- removed SW2: DOWN, symbol Switch:SW_Push
- removed SW3: TRANSMIT, symbol Switch:SW_Push
- added Q2: HY1904C2, kicad-parts:HY1904C2, symbol kicad-parts:HY1904C2
- J3: renamed from J4; value Conn_Coaxial -> BNC
- J4: renamed from J5; value Conn_Coaxial_Small -> SMA
- R13: value 120 -> 100K; footprint Resistor_SMD:R_0805_2012Metric -> Resistor_SMD:R_1206_3216Metric; LCSC Part # C17547 -> C17900; MPN 0805W8F2103T5E -> 1206W4F1003T5E
- renumbered C26 to C1, C23 to C10, C7 to C11, C16 to C12, C10 to C13, C22 to C14, C18 to C15, C29 to C16, C30 to C18, C21 to C19, C1 to C2, C31 to C21, C11 to C22, C32 to C23, C14 to C24, C12 to C25, C13 to C26, C15 to C27, C6 to C28, C8 to C29, C5 to C3, C2 to C4, C25 to C5, C3 to C6, C4 to C7, C9 to C8, C19 to C9, D21 to D1, D23 to D2, D22 to D3, D24 to D4, D6 to D5, D7 to D6, D18 to D7, J3 to J5, L12 to L1, L11 to L2, L2 to L3, L8 to L4, Q4 to Q1, R21 to R1, R3 to R10, R8 to R11, R16 to R12, R10 to R14, R9 to R15, R23 to R2, R17 to R3, R1 to R5, R2 to R6, R22 to R7, R24 to R8, R18 to R9, U4 to U2, U2 to U4
Connections:
- net GND: now also J3.2 (Ext), J4.2 (Ext), R13.1, Q2.1 (SOURCE_1), Q2.2 (SOURCE_2), Q2.3 (SOURCE_3); no longer A1.8 (D5), A1.9 (D6)
- net at C27.2: now also R13.2, Q2.4 (GATE)
- net ANTENNA: now reaches J3.1 (In)
- net ANTENNA: now also J4.1 (In)
- net LED-FT4: no longer names the net of A1.14 (D11)
- net LED-FT4: no longer R13.1
- net LED-FT8: no longer names the net of A1.15 (D12)
- net LED-JS8: no longer names the net of A1.13 (D10)
- net LED-TX: no longer names the net of A1.16 (D13)
- net LED-WSPR: no longer names the net of A1.12 (D9)
- net SWITCH-1-UP: no longer names the net of A1.5 (D2)
- net SWITCH-2-DOWN renamed PA-POWER-PWM
- net SWITCH-3-TRANSMIT: no longer names the net of A1.7 (D4)
- new net PA-DRAIN: Q2.5 (DRAIN_5), Q2.6 (DRAIN_6), Q2.7 (DRAIN_7), Q2.8 (DRAIN_8)
Other:
- added sheet 10M LPF IN (nfet-highside-load-switch.kicad_sch)
- added sheet 10M LPF OUT (nfet-highside-load-switch.kicad_sch)
- added sheet 10m LPF (SMT) (lpf-10m-smt.kicad_sch)
- added sheet 12M LPF IN (nfet-highside-load-switch.kicad_sch)
- added sheet 12M LPF OUT (nfet-highside-load-switch.kicad_sch)
- added sheet 12m LPF (SMT) (lpf-12m-smt.kicad_sch)
- added sheet 15M LPF IN (nfet-highside-load-switch.kicad_sch)
- added sheet 15M LPF OUT (nfet-highside-load-switch.kicad_sch)
- added sheet 15m LPF (SMT) (lpf-15m-smt.kicad_sch)
- added sheet 160M LPF IN (nfet-highside-load-switch.kicad_sch)
- added sheet 160M LPF OUT (nfet-highside-load-switch.kicad_sch)
- added sheet 160m LPF (SMT) (lpf-160m-smt.kicad_sch)
- added sheet 17M LPF IN (nfet-highside-load-switch.kicad_sch)
- added sheet 17M LPF OUT (nfet-highside-load-switch.kicad_sch)
- added sheet 17m LPF (SMT) (lpf-17m-smt.kicad_sch)
- added sheet 20M LPF IN (nfet-highside-load-switch.kicad_sch)
- added sheet 20M LPF OUT (nfet-highside-load-switch.kicad_sch)
- added sheet 20m LPF (SMT) (lpf-20m-smt.kicad_sch)
- added sheet 2200M LPF IN (nfet-highside-load-switch.kicad_sch)
- added sheet 2200M LPF OUT (nfet-highside-load-switch.kicad_sch)
- added sheet 2200m LPF (SMT) (lpf-2200m-smt.kicad_sch)
- added sheet 2M LPF IN (nfet-highside-load-switch.kicad_sch)
- added sheet 2M LPF OUT (nfet-highside-load-switch.kicad_sch)
- added sheet 2m LPF (SMT) (lpf-2m-smt.kicad_sch)
- added sheet 30M LPF IN (nfet-highside-load-switch.kicad_sch)
- added sheet 30M LPF OUT (nfet-highside-load-switch.kicad_sch)
- added sheet 30m LPF (SMT) (lpf-30m-smt.kicad_sch)
- added sheet 40M LPF IN (nfet-highside-load-switch.kicad_sch)
- added sheet 40M LPF OUT (nfet-highside-load-switch.kicad_sch)
- added sheet 40m LPF (SMT) (lpf-40m-smt.kicad_sch)
- added sheet 60M LPF IN (nfet-highside-load-switch.kicad_sch)
- added sheet 60M LPF OUT (nfet-highside-load-switch.kicad_sch)
- added sheet 60m LPF (SMT) (lpf-60m-smt.kicad_sch)
- added sheet 630M LPF IN (nfet-highside-load-switch.kicad_sch)
- added sheet 630M LPF OUT (nfet-highside-load-switch.kicad_sch)
- added sheet 630m LPF (SMT) (lpf-630m-smt.kicad_sch)
- added sheet 6M LPF IN (nfet-highside-load-switch.kicad_sch)
- added sheet 6M LPF OUT (nfet-highside-load-switch.kicad_sch)
- added sheet 6m LPF (SMT) (lpf-6m-smt.kicad_sch)
- added sheet 80M LPF IN (nfet-highside-load-switch.kicad_sch)
- added sheet 80M LPF OUT (nfet-highside-load-switch.kicad_sch)
- added sheet 80m LPF (SMT) (lpf-80m-smt.kicad_sch)
- note added: "10M"
- note added: "12M"
- note added: "15M"
- note added: "160M"
- note added: "17M"
- note added: "20M"
- note added: "2200M"
- note added: "2M"
- note added: "30M"
- note added: "40M"
- note added: "60M"
- note added: "630M"
- note added: "6M"
- note added: "80M"
- note added: "ADD PULLUPS/PULLDOWNS FOR ALL IMPORTANT PINS CLASS E INDUCTOR FOR PA / ATS ANTENNA MATCHING NETWORK OR ATU ADD/TEST AUDIO+ANTENNA CABLE DETECTION ADD MORE MOSFET SWITCHES ADD SOME KIND OF MULTIPLEXING? ADD OPTIONAL INTERFACE PCB - EASY MOUNTING AT RIGHT ANGLES ADD TEST POINTS EITHER PREVENT RADIO POWERUP USING USB-SUPPLIED POWER (EG. 12V SUPPLY PRESENCE ENABLES 5V LINE) OR CONSIDER POWER LIMITS O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"
- note added: "INTERFACE FOR ANTENNA BAND PASS FILTERS"
- note added: "NB. IN A CLASS E RF POWER AMPLIFIER THE PA-DRAIN FLOWS INWARD WHEN ENABLED AND IS SUNK AT THE MOSFET SOURCE PINS."
- note added: "These filters are very likely to change. Therefore it makes sense to keep them on a separate board. PA -> Interface -> LPF board -> Interface back to mainboard -> Antenna How does the system know which board is plugged in? It should be able to query somehow to determine the frequency range. How can this be done easily? Allow the board to provide some data to read back to the master board describi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"
- note added: "docs/filter-models/cd2003-supply-low-pass-filter"
- note removed: "(CLAIM: "RF POWER OUTPUT VARIES FROM BAND TO BAND AROUND 5 WATTS" [3xBS170])"
- note removed: "0.05"
- note removed: "0.06"
- note removed: "0.08"
- note removed: "0.1"
- note removed: "0.13"
- note removed: "1.5A"
- note removed: "1650MHz"
- note removed: "2.35/1.34"
- note removed: "2.6/1.9A"
- note removed: "2M Band (144-148 MHz) Inductor (L): ~100 nH Capacitor (C): ~100 pF 10M Band (28-29.7 MHz) Inductor (L): ~560 nH Capacitor (C): ~27 pF 20M Band (14-14.35 MHz) Inductor (L): ~1.1 μH Capacitor (C): ~12 pF 40M Band (7-7.3 MHz) Inductor (L): ~2.2 μH Capacitor (C): ~6.8 pF 80M Band (3.5-4 MHz) Inductor (L): ~4.7 μH Capacitor (C): ~3.3 pF"
- note removed: "32MHz"
- note removed: "42MHz"
- note removed: "5 LEDs and three tactile pushbutton switches for user visual interface and controls. No fancy displays or rotary encoders!"
- note removed: "5.2/3.8A"
- note removed: ">400mA"
- note removed: ">70MHz"
- note removed: "ADD CABLE DETECTION ADD 12V REGULATOR ADD MOSFET SWITCHES ADD BAND INDICATOR LEDS ADD SOME KIND OF MULTIPLEXING ADD SCREEN? ADD BUTTONS? ADD INTERFACE PCB FOR EASY MOUNTING? ADD TEST POINTS"
- note removed: "C"
- note removed: "CAN FIX WITH DUPLICATION BUT CREATES PARASITICS TOWARD 1GHZ (BENEATH 2M)"
- note removed: "Example Calculation for 10M Band For a central frequency of 29 MHz: Target Frequency (f): 29 MHz Assuming L = 560 nH Calculate C: C=1(2πf)2LC=(2πf)2L1​ C=1(2π⋅29×106)2⋅560×10−9C=(2π⋅29×106)2⋅560×10−91​ C≈27 pFC≈27 pF"
- note removed: "HIGH POWER RATING VAGUE IMPRECISE RATING (20%) UNREPEATABLE HARD TO SIMULATE LOW SRF"
- note removed: "HIGH POWER RATING VAGUE IMPRECISE RATING (>20%) REQUIRES MANUAL WINDING AND TUNING UNREPEATABLE HARD TO SIMULATE LOW SRF"
- note removed: "INTERFACE"
- note removed: "L"
- note removed: "L.DCR"
- note removed: "L.I"
- note removed: "L.SRF"
- note removed: "LARGER SMT COMPONENTS"
- note removed: "LOW POWER RATING PRECISE (10%) OPTIONAL TUNING REPEATABLE SIMULATABLE HIGH SRF"
- note removed: "MANUALLY WOUND COILS"
- note removed: "MOSFET-SWITCHED TUNING COMPONENTS OR GAAS FETs (LOW INSERTION LOSS)"
- note removed: "POTENTIAL IMPROVEMENT: IMPEDANCE MATCHING RESISTOR IN SERIES. NOMINAL IMPROVEMENT, WILL REQUIRE DETAILED MEASUREMENT."
- note removed: "POTENTIAL IMPROVEMENT: MCU CONFIGURABLE OUTPUT POWER LEVEL. (ADD 2×MMBF170)"
- note removed: "POTENTIAL IMPROVEMENT: MCU OUTPUT POWER MONITOR. USE 2x SAME 1% RESISTORS TO HALVE VOLTAGE THEN FEED TO MCU ADC VIA ZENER DIODE."
- note removed: "POTENTIAL IMPROVEMENT: MCU SHUTDOWN OF LINE DRIVER IN CASE OF SWR ANOMALY OR SIMILAR."
- note removed: "POTENTIAL IMPROVEMENT: SWITCHABLE TUNING COMPONENTS"
- note removed: "REALITY: - Not easily possible to tune SMT based resonant circuits due to lack of ability to alter 'turns' - Even if switching in compnents with a GaaS FET, these would need to be frequency band specific due to SRF concerns. - Probably requires a broader view of the tuning problem including the ability to add or remove loads - Given that inductance drops with power, some ability to tune for power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"
- note removed: "SMALLER SMT COMPONENTS"
- moved on the sheet: A1, C1, C24, C25, C26, C27, C28, C29, C5, D1, D2, D3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

Commit message: More bands
Other:
- added sheet 70CM LPF IN (nfet-highside-load-switch.kicad_sch)
- added sheet 70CM LPF OUT (nfet-highside-load-switch.kicad_sch)
- added sheet 70cm LPF (SMT) (lpf-70cm-smt.kicad_sch)
- note added: "70CM"

Commit message: Updates
Parts:
- added J10: BANDMODULE3-ANT, Connector_PinSocket_2.54mm:PinSocket_1x07_P2.54mm_Vertical, symbol Connector_Generic:Conn_01x07
- added J11: BANDMODULE4-ANT, Connector_PinSocket_2.54mm:PinSocket_1x07_P2.54mm_Vertical, symbol Connector_Generic:Conn_01x07
- added J12: BANDMODULE3-PA, Connector_PinSocket_2.54mm:PinSocket_1x07_P2.54mm_Vertical, symbol Connector_Generic:Conn_01x07
- added J13: BANDMODULE4-PA, Connector_PinSocket_2.54mm:PinSocket_1x07_P2.54mm_Vertical, symbol Connector_Generic:Conn_01x07
- added J14: BANDMODULE5-ANT, Connector_PinSocket_2.54mm:PinSocket_1x07_P2.54mm_Vertical, symbol Connector_Generic:Conn_01x07
- added J15: BANDMODULE6-ANT, Connector_PinSocket_2.54mm:PinSocket_1x07_P2.54mm_Vertical, symbol Connector_Generic:Conn_01x07
- added J16: BANDMODULE5-PA, Connector_PinSocket_2.54mm:PinSocket_1x07_P2.54mm_Vertical, symbol Connector_Generic:Conn_01x07
- added J17: BANDMODULE6-PA, Connector_PinSocket_2.54mm:PinSocket_1x07_P2.54mm_Vertical, symbol Connector_Generic:Conn_01x07
- added J18: MMCX, Connector_Coaxial:MMCX_Molex_73415-1471_Vertical, symbol Connector:Conn_Coaxial_Small
- added J19: IPEX-1, symbol Connector:Conn_Coaxial_Small
- added J20: LCD-2004, Connector_PinHeader_2.54mm:PinHeader_1x04_P2.54mm_Vertical, symbol Connector_Generic:Conn_01x04
- added J6: BANDMODULE1-ANT, Connector_PinSocket_2.54mm:PinSocket_1x07_P2.54mm_Vertical, symbol Connector_Generic:Conn_01x07
- added J7: BANDMODULE1-PA, Connector_PinSocket_2.54mm:PinSocket_1x07_P2.54mm_Vertical, symbol Connector_Generic:Conn_01x07
- added J8: BANDMODULE2-ANT, Connector_PinSocket_2.54mm:PinSocket_1x07_P2.54mm_Vertical, symbol Connector_Generic:Conn_01x07
- added J9: BANDMODULE2-PA, Connector_PinSocket_2.54mm:PinSocket_1x07_P2.54mm_Vertical, symbol Connector_Generic:Conn_01x07
- added L5: L, symbol Device:L
- J1, J2: footprint Connector_Audio:Jack_3.5mm_CUI_SJ2-3593D-SMT_Horizontal -> Connector_Audio:Jack_3.5mm_CUI_SJ1-3525N_Horizontal
Connections:
- net 3.3V: now also J20.2 (Pin_2)
- net ANTENNA: now also J18.1 (In), J19.1 (In)
- net GND: now also J10.1 (Pin_1), J10.3 (Pin_3), J10.5 (Pin_5), J11.1 (Pin_1), J11.3 (Pin_3), J11.5 (Pin_5), J12.1 (Pin_1), J12.3 (Pin_3), J12.5 (Pin_5), J12.7 (Pin_7), J13.1 (Pin_1), J13.3 (Pin_3), J13.5 (Pin_5), J13.7 (Pin_7), J14.1 (Pin_1), J14.3 (Pin_3), J14.5 (Pin_5), J15.1 (Pin_1), J15.3 (Pin_3), J15.5 (Pin_5), J16.1 (Pin_1), J16.3 (Pin_3), J16.5 (Pin_5), J16.7 (Pin_7), J17.1 (Pin_1), J17.3 (Pin_3), J17.5 (Pin_5), J17.7 (Pin_7), J18.2 (Ext), J19.2 (Ext), J20.1 (Pin_1), J6.1 (Pin_1), J6.3 (Pin_3), J6.5 (Pin_5), J7.1 (Pin_1), J7.3 (Pin_3), J7.5 (Pin_5), J7.7 (Pin_7), J8.1 (Pin_1), J8.3 (Pin_3), J8.5 (Pin_5), J9.1 (Pin_1), J9.3 (Pin_3), J9.5 (Pin_5), J9.7 (Pin_7)
- net I2C-SCL-3.3V: now also J20.4 (Pin_4)
- net I2C-SDA-3.3V: now also J20.3 (Pin_3)
- new net BM1-ANT: J6.2 (Pin_2), J6.4 (Pin_4), J6.6 (Pin_6)
- new net BM1-PA: J7.2 (Pin_2), J7.4 (Pin_4), J7.6 (Pin_6)
- new net BM1-PRESENT: J15.7 (Pin_7), J6.7 (Pin_7)
- new net BM2-ANT: J8.2 (Pin_2), J8.4 (Pin_4), J8.6 (Pin_6)
- new net BM2-PA: J9.2 (Pin_2), J9.4 (Pin_4), J9.6 (Pin_6)
- new net BM2-PRESENT: J8.7 (Pin_7)
- new net BM3-ANT: J10.2 (Pin_2), J10.4 (Pin_4), J10.6 (Pin_6)
- new net BM3-PA: J12.2 (Pin_2), J12.4 (Pin_4), J12.6 (Pin_6)
- new net BM3-PRESENT: J10.7 (Pin_7)
- new net BM4-ANT: J11.2 (Pin_2), J11.4 (Pin_4), J11.6 (Pin_6)
- new net BM4-PA: J13.2 (Pin_2), J13.4 (Pin_4), J13.6 (Pin_6)
- new net BM4-PRESENT: J11.7 (Pin_7)
- new net BM5-ANT: J14.2 (Pin_2), J14.4 (Pin_4), J14.6 (Pin_6)
- new net BM5-PA: J16.2 (Pin_2), J16.4 (Pin_4), J16.6 (Pin_6)
- new net BM5-PRESENT: J14.7 (Pin_7)
- new net BM6-ANT: J15.2 (Pin_2), J15.4 (Pin_4), J15.6 (Pin_6)
- new net BM6-PA: J17.2 (Pin_2), J17.4 (Pin_4), J17.6 (Pin_6)
- new net PA-12V: L5.1
Other:
- removed sheet 10M LPF IN
- removed sheet 10M LPF OUT
- removed sheet 10m LPF (SMT)
- removed sheet 12M LPF IN
- removed sheet 12M LPF OUT
- removed sheet 12m LPF (SMT)
- removed sheet 15M LPF IN
- removed sheet 15M LPF OUT
- removed sheet 15m LPF (SMT)
- removed sheet 160M LPF IN
- removed sheet 160M LPF OUT
- removed sheet 160m LPF (SMT)
- removed sheet 17M LPF IN
- removed sheet 17M LPF OUT
- removed sheet 17m LPF (SMT)
- removed sheet 20M LPF IN
- removed sheet 20M LPF OUT
- removed sheet 20m LPF (SMT)
- removed sheet 2200M LPF IN
- removed sheet 2200M LPF OUT
- removed sheet 2200m LPF (SMT)
- removed sheet 2M LPF IN
- removed sheet 2M LPF OUT
- removed sheet 2m LPF (SMT)
- removed sheet 30M LPF IN
- removed sheet 30M LPF OUT
- removed sheet 30m LPF (SMT)
- removed sheet 40M LPF IN
- removed sheet 40M LPF OUT
- removed sheet 40m LPF (SMT)
- removed sheet 60M LPF IN
- removed sheet 60M LPF OUT
- removed sheet 60m LPF (SMT)
- removed sheet 630M LPF IN
- removed sheet 630M LPF OUT
- removed sheet 630m LPF (SMT)
- removed sheet 6M LPF IN
- removed sheet 6M LPF OUT
- removed sheet 6m LPF (SMT)
- removed sheet 70CM LPF IN
- removed sheet 70CM LPF OUT
- removed sheet 70cm LPF (SMT)
- removed sheet 80M LPF IN
- removed sheet 80M LPF OUT
- removed sheet 80m LPF (SMT)
- added sheet BM1-SWITCH-ANT (nfet-highside-load-switch.kicad_sch)
- added sheet BM1-SWITCH-PA (nfet-highside-load-switch.kicad_sch)
- added sheet BM2-SWITCH-ANT (nfet-highside-load-switch.kicad_sch)
- added sheet BM2-SWITCH-PA (nfet-highside-load-switch.kicad_sch)
- added sheet BM3-SWITCH-ANT (nfet-highside-load-switch.kicad_sch)
- added sheet BM3-SWITCH-PA (nfet-highside-load-switch.kicad_sch)
- added sheet BM4-SWITCH-ANT (nfet-highside-load-switch.kicad_sch)
- added sheet BM4-SWITCH-PA (nfet-highside-load-switch.kicad_sch)
- added sheet BM5-SWITCH-ANT (nfet-highside-load-switch.kicad_sch)
- added sheet BM5-SWITCH-PA (nfet-highside-load-switch.kicad_sch)
- added sheet BM6-SWITCH-ANT (nfet-highside-load-switch.kicad_sch)
- added sheet BM6-SWITCH-PA5 (nfet-highside-load-switch.kicad_sch)
- added sheet PA-POWER-PWM (nfet-highside-load-switch.kicad_sch)
- note added: "DIFFICULT TO ACHIEVE WITH OBSERVED SMT PRODUCTS: - HIGH DCR AND LOW ACCURACY ON HIGH I INDUCTORS. - LOW I ON HIGH SRF LOW DCR HIGH ACCURACY INDUCTORS. SOLUTION: SERIES-PARALLEL CONFIGURATION."
- note added: "DISPLAY"
- note added: "DRAIN"
- note added: "OPERATION ON ALL FREQUENCIES. SOLE OPERATION ON 70CM (430 MHz) TO 160M (1.8 MHz)."
- note added: "POSSIBLE TO USE THIS OUTPUT TO TEST THE FILTER CONFIGURATION?"
- note added: "PRIMARY RF CHOKE INDUCTOR"
- note added: "SECONDARY/ TERTIARY SWITCHABLE RF CHOKE INDUCTORS"
- note added: "SRF > 1.2GHz HIGH Q (50+) DCR <=0.1"
- note removed: "10M"
- note removed: "12M"
- note removed: "15M"
- note removed: "160M"
- note removed: "17M"
- note removed: "20M"
- note removed: "2200M"
- note removed: "2M"
- note removed: "30M"
- note removed: "40M"
- note removed: "60M"
- note removed: "630M"
- note removed: "6M"
- note removed: "70CM"
- note removed: "80M"
- note removed: "BAND-SPECIFIC LOW PASS FILTERS"
- note removed: "INTERFACE FOR ANTENNA BAND PASS FILTERS"
- note removed: "POTENTIAL IMPROVEMENT: UPGRADE TO CHEBYSHEV 7TH ORDER OR SOME OTHER EXOTIC FILTER TOPOLOGIES. FOR DIGITAL DATA WHICH IS THIS SYSTEM'S FOCUS THAT MAY BE OVERKILL."
- note removed: "SELECTION OF COMPONENTS HERE IS NON-TRIVIAL. THERE ARE A LOT OF COMPETING CONCERNS INCLUDING SRF, CURRENT RATING, VOLTAGE RATING, FORM FACTOR, REPEATABILITY, ACCURACY/TUNABILITY, AND AVAILABILITY. THE CURRENT DESIGN USES SOME APPROXIMATIONS TO REDUCE UNIQUE COMPONENT COUNT WHILE MAINTAINING A THEORETICALLY RELATIVELY ACCURATE AND PROTECTED APPROACH."
- note removed: "These filters are very likely to change. Therefore it makes sense to keep them on a separate board. PA -> Interface -> LPF board -> Interface back to mainboard -> Antenna How does the system know which board is plugged in? It should be able to query somehow to determine the frequency range. How can this be done easily? Allow the board to provide some data to read back to the master board describi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"
- moved on the sheet: C1, C5, D1, D2, D3, D4, J3, J4, R1, R2, R3, R7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

Commit message: Updates
Parts:
- removed L5: L, symbol Device:L
Other:
- added sheet PA Switched RF Choke (pa-switched-rf-choke.kicad_sch)
- note added: "ADD PULLUPS/PULLDOWNS FOR ALL IMPORTANT PINS REST OF PA ANTENNA MATCHING NETWORK OR ATU ADD/TEST AUDIO + ANTENNA CABLE DETECTION ADD MORE MOSFET SWITCHES ADD SOME KIND OF MULTIPLEXING? ADD OPTIONAL INTERFACE PCB - EASY MOUNTING AT RIGHT ANGLES ADD OPTIONAL SQUEAKER ADD TEST POINTS EITHER PREVENT RADIO POWERUP USING USB-SUPPLIED POWER (EG. 12V SUPPLY PRESENCE ENABLES 5V LINE) OR CONSIDER POWER LIM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"
- note added: "POWER AMPLIFIER CHOKE"
- note added: "SWITCHED BASED ON FREQUENCY BAND"
- note removed: "ADD PULLUPS/PULLDOWNS FOR ALL IMPORTANT PINS CLASS E INDUCTOR FOR PA / ATS ANTENNA MATCHING NETWORK OR ATU ADD/TEST AUDIO+ANTENNA CABLE DETECTION ADD MORE MOSFET SWITCHES ADD SOME KIND OF MULTIPLEXING? ADD OPTIONAL INTERFACE PCB - EASY MOUNTING AT RIGHT ANGLES ADD TEST POINTS EITHER PREVENT RADIO POWERUP USING USB-SUPPLIED POWER (EG. 12V SUPPLY PRESENCE ENABLES 5V LINE) OR CONSIDER POWER LIMITS O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"
- note removed: "DIFFICULT TO ACHIEVE WITH OBSERVED SMT PRODUCTS: - HIGH DCR AND LOW ACCURACY ON HIGH I INDUCTORS. - LOW I ON HIGH SRF LOW DCR HIGH ACCURACY INDUCTORS. SOLUTION: SERIES-PARALLEL CONFIGURATION."
- note removed: "OPERATION ON ALL FREQUENCIES. SOLE OPERATION ON 70CM (430 MHz) TO 160M (1.8 MHz)."
- note removed: "PRIMARY RF CHOKE INDUCTOR"
- note removed: "SECONDARY/ TERTIARY SWITCHABLE RF CHOKE INDUCTORS"
- note removed: "SRF > 1.2GHz HIGH Q (50+) DCR <=0.1"
Changed lines of the file:
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@@
 	(polyline
 		(pts
-			(xy 343.535 125.095) (xy 343.535 144.145)
-		)
-		(stroke
-			(width 0)
-			(type default)
-		)
-	)
-	(polyline
-		(pts
 			(xy 21.59 25.4) (xy 21.59 96.52)
 		)
@@
 		)
 	)
-	(polyline
-		(pts
-			(xy 339.725 144.145) (xy 343.535 144.145)
-		)
-		(stroke
-			(width 0)
-			(type default)
-		)
-	)
 	(wire
 		(pts
@@
 		)
 	)
+	(polyline
+		(pts
+			(xy 304.546 108.458) (xy 304.8 108.458)
+		)
+		(stroke
+			(width 0)
+			(type default)
+		)
+	)
 	(wire
 		(pts
@@
 	(wire
 		(pts
-			(xy 314.96 128.27) (xy 314.96 147.32)
-		)
-		(stroke
-			(width 0)
-			(type default)
-		)
-	)
-	(wire
-		(pts
 			(xy 43.18 132.08) (xy 43.18 133.35)
 		)
@@
 		)
 	)
+	(polyline
+		(pts
+			(xy 304.8 180.34) (xy 354.076 180.34)
+		)
+		(stroke
+			(width 0)
+			(type default)
+		)
+	)
 	(wire
 		(pts
@@
 	(polyline
 		(pts
-			(xy 339.725 125.095) (xy 343.535 125.095)
-		)
-		(stroke
-			(width 0)
-			(type default)
-		)
-	)
-	(polyline
-		(pts
 			(xy 165.1 25.4) (xy 125.73 25.4)
 		)
@@
 		)
 	)
+	(polyline
+		(pts
+			(xy 354.076 108.458) (xy 354.076 180.34)
+		)
+		(stroke
+			(width 0)
+			(type default)
+		)
+	)
 	(wire
 		(pts
@@
 		)
 	)
+	(polyline
+		(pts
+			(xy 304.8 108.458) (xy 354.076 108.458)
+		)
+		(stroke
+			(width 0)
+			(type default)
+		)
+	)
 	(wire
 		(pts
@@
 		)
 	)
-	(text "SRF > 1.2GHz\nHIGH Q (50+)\nDCR <=0.1"
-		(exclude_from_sim no)
-		(at 322.072 141.224 0)
-		(effects
-			(font
-				(size 1.27 1.27)
-			)
-			(justify left)
-		)
-	)
 	(text "NB. IN A CLASS E\nRF POWER AMPLIFIER\nTHE PA-DRAIN FLOWS\nINWARD WHEN ENABLED\nAND IS SUNK AT THE\nMOSFET SOURCE PINS."
 		(exclude_from_sim no)
@@
 		)
 	)
-	(text "PRIMARY\nRF CHOKE\nINDUCTOR"
-		(exclude_from_sim no)
-		(at 322.072 122.428 0)
-		(effects
-			(font
-				(size 1.27 1.27)
-				(thickness 0.254)
-				(bold yes)
-			)
-			(justify left)
-		)
-	)
-	(text "SECONDARY/\nTERTIARY\nSWITCHABLE\nRF CHOKE\nINDUCTORS"
-		(exclude_from_sim no)
-		(at 322.326 152.146 0)
-		(effects
-			(font
-				(size 1.27 1.27)
-				(thickness 0.254)
-				(bold yes)
-			)
-			(justify left)
-		)
-	)
 	(text "DRAIN"
 		(exclude_from_sim no)
@@
 		)
 	)
-	(text "OPERATION ON\nALL FREQUENCIES.\nSOLE OPERATION\nON 70CM (430 MHz)\nTO 160M (1.8 MHz)."
-		(exclude_from_sim no)
-		(at 322.072 131.572 0)
-		(effects
-			(font
-				(size 1.27 1.27)
-			)
-			(justify left)
-		)
-	)
 	(text "USED FOR\nFIRMWARE\nUPLOADS"
 		(exclude_from_sim no)
@@
 		)
 	)
-	(text "ADD PULLUPS/PULLDOWNS FOR ALL IMPORTANT PINS\nCLASS E INDUCTOR FOR PA / ATS\nANTENNA MATCHING NETWORK OR ATU\nADD/TEST AUDIO+ANTENNA CABLE DETECTION\nADD MORE MOSFET SWITCHES\nADD SOME KIND OF MULTIPLEXING?\nADD OPTIONAL INTERFACE PCB - EASY MOUNTING AT RIGHT ANGLES\nADD TEST POINTS\nEITHER PREVENT RADIO POWERUP USING USB-SUPPLIED POWER (EG. 12V SUPPLY PRESENCE ENABLES 5V LINE) OR CONSIDER POWER LIMITS OF USB2 SUPPLIES"
+	(text "ADD PULLUPS/PULLDOWNS FOR ALL IMPORTANT PINS\nREST OF PA\nANTENNA MATCHING NETWORK OR ATU\nADD/TEST AUDIO + ANTENNA CABLE DETECTION\nADD MORE MOSFET SWITCHES\nADD SOME KIND OF MULTIPLEXING?\nADD OPTIONAL INTERFACE PCB - EASY MOUNTING AT RIGHT ANGLES\nADD OPTIONAL SQUEAKER\nADD TEST POINTS\nEITHER PREVENT RADIO POWERUP USING USB-SUPPLIED POWER (EG. 12V SUPPLY PRESENCE ENABLES 5V LINE) OR CONSIDER POWER LIMITS OF USB2 SUPPLIES\nOPTION FOR SUBSYSTEM POWER METERING"
 		(exclude_from_sim no)
-		(at 269.748 -30.48 0)
+		(at 268.732 -38.862 0)
 		(effects
 			(font
@@
 		)
 	)
+	(text "SWITCHED BASED ON FREQUENCY BAND"
+		(exclude_from_sim no)
+		(at 324.104 144.78 0)
+		(effects
+			(font
+				(size 1.27 1.27)
+			)
+		)
+	)
 	(text "400kHz"
 		(exclude_from_sim no)
@@
 		)
 	)
-	(text "DIFFICULT TO ACHIEVE WITH\nOBSERVED SMT PRODUCTS:\n - HIGH DCR AND LOW ACCURACY\n   ON HIGH I INDUCTORS.\n - LOW I ON HIGH SRF LOW DCR\n   HIGH ACCURACY INDUCTORS.\n\nSOLUTION: SERIES-PARALLEL\n          CONFIGURATION."
+	(text "POWER AMPLIFIER CHOKE"
 		(exclude_from_sim no)
-		(at 346.202 135.255 0)
+		(at 322.326 141.732 0)
 		(effects
 			(font
 				(size 1.27 1.27)
+				(thickness 0.254)
+				(bold yes)
 			)
-			(justify left)
 		)
 	)
@@
 		)
 	)
+	(global_label "PA-DRAIN"
+		(shape output)
+		(at 339.09 165.1 0)
+		(fields_autoplaced yes)
+		(effects
+			(font
+				(size 1.27 1.27)
+			)
+			(justify left)
+		)
+		(property "Intersheetrefs" "${INTERSHEET_REFS}"
+			(at 351.5701 165.1 0)
+			(effects
+				(font
+					(size 1.27 1.27)
+				)
+				(justify left)
+				(hide yes)
+			)
+		)
+	)
 	(global_label "BM5-ENABLE"
 		(shape input)
@@
 	(global_label "PA-12V"
 		(shape input)
-		(at 314.96 120.65 90)
+		(at 307.34 164.465 180)
 		(fields_autoplaced yes)
 		(effects
@@
 				(size 1.27 1.27)
 			)
-			(justify left)
+			(justify right)
 		)
 		(property "Intersheetrefs" "${INTERSHEET_REFS}"
-			(at 314.96 110.2262 90)
+			(at 296.9162 164.465 0)
 			(effects
 				(font
 					(size 1.27 1.27)
 				)
-				(justify left)
+				(justify right)
 				(hide yes)
 			)
@@
 	)
 	(symbol
-		(lib_id "Device:L")
-		(at 314.96 124.46 0)
-		(unit 1)
-		(exclude_from_sim no)
-		(in_bom yes)
-		(on_board yes)
-		(dnp no)
-		(fields_autoplaced yes)
-		(property "Reference" "L5"
-			(at 316.23 123.1899 0)
-			(effects
-				(font
-					(size 1.27 1.27)
-				)
-				(justify left)
-			)
-		)
-		(property "Value" "L"
-			(at 316.23 125.7299 0)
-			(effects
-				(font
-					(size 1.27 1.27)
-				)
-				(justify left)
-			)
-		)
-		(property "Footprint" ""
-			(at 314.96 124.46 0)
-			(effects
-				(font
-					(size 1.27 1.27)
-				)
-				(hide yes)
-			)
-		)
-		(property "Datasheet" "~"
-			(at 314.96 124.46 0)
-			(effects
-				(font
-					(size 1.27 1.27)
-				)
-				(hide yes)
-			)
-		)
-		(property "Description" "Inductor"
-			(at 314.96 124.46 0)
-			(effects
-				(font
-					(size 1.27 1.27)
-				)
-				(hide yes)
-			)
-		)
-		(pin "2"
-		)
-		(pin "1"
-		)
-		(instances
-			(project ""
-				(path "/c3abf330-1856-4368-a03b-0e6191ae29a9"
-					(reference "L5")
-					(unit 1)
-				)
-			)
-		)
-	)
-	(symbol
 		(lib_id "Connector_Generic:Conn_01x04")
 		(at 229.87 87.63 0)
@@
 				)
 			)
+		)
+	)
+	(sheet
+		(at 307.34 149.86)
+		(size 31.75 22.225)
+		(fields_autoplaced yes)
+		(stroke
+			(width 0.1524)
+			(type solid)
+		)
+		(fill
+			(color 0 0 0 0.0000)
+		)
+		(property "Sheetname" "PA Switched RF Choke"
+			(at 307.34 149.1484 0)
+			(effects
+				(font
+					(size 1.27 1.27)
+				)
+				(justify left bottom)
+			)
+		)
+		(property "Sheetfile" "pa-switched-rf-choke.kicad_sch"
+			(at 307.34 172.6696 0)
+			(effects
+				(font
+					(size 1.27 1.27)
+				)
+				(justify left top)
+			)
+		)
+		(pin "GND" input
+			(at 307.34 169.545 180)
+			(effects
+				(font
+					(size 1.27 1.27)
+				)
+				(justify left)
+			)
+		)
+		(pin "24V" input
+			(at 307.34 167.005 180)
+			(effects
+				(font
+					(size 1.27 1.27)
+				)
+				(justify left)
+			)
+		)
+		(pin "5V" input
+			(at 307.34 161.925 180)
+			(effects
+				(font
+					(size 1.27 1.27)
+				)
+				(justify left)
+			)
+		)
+		(pin "50UH-ENABLE-WHEN-LOW" input
+			(at 307.34 154.305 180)
+			(effects
+				(font
+					(size 1.27 1.27)
+				)
+				(justify left)
+			)
+		)
+		(pin "10UH-ENABLE-WHEN-LOW" input
+			(at 307.34 151.765 180)
+			(effects
+				(font
+					(size 1.27 1.27)
+				)
+				(justify left)
+			)
+		)
+		(pin "100UH-ENABLE-WHEN-LOW" input
+			(at 307.34 156.845 180)
+			(effects
+				(font
+					(size 1.27 1.27)
+				)
+				(justify left)
+			)
+		)
+		(pin "PA-DRAIN" output
+			(at 339.09 165.1 0)
+			(effects
+				(font
+					(size 1.27 1.27)
+				)
+				(justify right)
+			)
+		)
+		(instances
+			(project "adxi"
+				(path "/c3abf330-1856-4368-a03b-0e6191ae29a9"
+					(page "15")
+				)
+			)

Commit message: More outputs, etc
Parts:
- added L141: 220uH, symbol Device:L
Connections:
- net SPI-MOSI: now reaches A1.14 (D11)
- net SPI-SS-OUTPUTS: now reaches A1.15 (D12)
- net SPI-SCK: now reaches A1.16 (D13)
- no-connect marks 10 -> 16
Other:
- sheet PA Switched RF Choke renamed PA Switched Resonator
- added sheet Digital output expansion (spi-gpio-output.kicad_sch)
- sheet PA Switched Resonator: file pa-switched-rf-choke.kicad_sch -> pa-switched-resonator.kicad_sch
- sheet PA Switched Resonator ports: added 12PF-ENABLE-WHEN-LOW, 150PF-ENABLE-WHEN-LOW, 15PF-ENABLE-WHEN-LOW, 20PF-ENABLE-WHEN-LOW, 5.6NF-ENABLE-WHEN-LOW, 6.8PF-ENABLE-WHEN-LOW, 68NF-ENABLE-WHEN-LOW, 82PF-ENABLE-WHEN-LOW; removed none
- note added: "BONUS BLINKENLIGHTS"
- note added: "For effective power supply noise filtering, a design guideline is to use ferrite beads at about 20% of their rated DC current."
- note added: "MCU AND OUTPUT EXPANSION"
- note added: "POWER AMPLIFIER SWITCHED RESONATOR"
- note added: "RF CHOKE"
- note added: "RULE OF THUMB: "OPERATE SWR <4" "SURVIVE SWR <10""
- note added: "SHARED ACROSS ALL FREQUENCY BANDS. SRF > 140MHz"
- note added: "THIS ONE SHOULD BE POSSIBLE TO HARD WIRE IF REQUIRED"
- note added: "TRANSMIT POWER CONTROL"
- note removed: "MCU"
- note removed: "POWER AMPLIFIER CHOKE"
- moved on the sheet: A1, C24, C25, C26, C27, C28, C29, J20, Q2, R13, R14, R15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
