File: kicad-pcbs/adxi/adxi.kicad_sch (KiCad schematic)
At the start: 111 parts, among them J1 FROM-PC-SPK, J10 BANDMODULE3-ANT, J11 BANDMODULE4-ANT, J12 BANDMODULE3-PA, J13 BANDMODULE4-PA, J14 BANDMODULE5-ANT, J15 BANDMODULE6-ANT, J16 BANDMODULE5-PA, J17 BANDMODULE6-PA, J18 MMCX, J19 IPEX-1, J2 TO-PC-MIC, J20 LCD-2004, J3 BNC, J4 SMA, J5 12V SUPPLY, J6 BANDMODULE1-ANT, J7 BANDMODULE1-PA, J8 BANDMODULE2-ANT, J9 BANDMODULE2-PA, Q1 MMBF170, Q2 HY1904C2, U1 CD2003, U2 L7812, U3 74ACT244, U4 Si5351A-B-GT

Commit message: Pluggable PAs
Parts:
- added L161, L162, L163, L164, L165, L166, L167, L168, L169, L170, L171, L172, L173, L174, L175, L176, L177, L178, L179, L180, L181, L182, L183, L184, L185, L186, L187, L188, L189, L190, L191, L192, L193, L194, L195, L196, L197, L198, L199, L200, L201, L202, L203, L204, L205, L206, L207, L208, L209, L210, L211, L212, L213, L214, L215, L216, L217, L218, L219, L220, L221, L222, L223, L224, L225: 470nH, Inductor_SMD:L_1008_2520Metric, symbol Device:L
- L160: value L -> 470nH; footprint (none) -> Inductor_SMD:L_1008_2520Metric; LCSC Part # (none) -> C316369; MPN (none) -> SPH252012HR47MT; Manufacturer (none) -> Sunlord
Connections:
- net at FB2.1, L143.1, L156.1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: now also L162.1
- net at C39.1, C40.1, C41.1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: now also L194.2, L225.2
- net at L160.2: now also L161.1
- new net: L212.2, L213.1
- new net: L213.2, L214.1
- new net: L176.2, L177.1
- new net: L177.2, L178.1
- new net: L196.2, L197.1
- new net: L197.2, L198.1
- new net: L222.2, L223.1
- new net: L223.2, L224.1
- new net: L163.2, L164.1
- new net: L164.2, L165.1
- new net: L181.2, L182.1
- new net: L182.2, L183.1
- new net: L171.2, L172.1
- new net: L172.2, L173.1
- new net: L188.2, L189.1
- new net: L189.2, L190.1
- new net: L169.2, L170.1
- new net: L170.2, L171.1
- new net: L214.2, L215.1
- new net: L215.2, L216.1
- new net: L195.2, L196.1
- new net: L161.2, L195.1
- new net: L184.2, L185.1
- new net: L185.2, L186.1
- new net: L166.2, L167.1
- new net: L167.2, L168.1
- new net: L162.2, L163.1
- new net: L198.2, L199.1
- new net: L199.2, L200.1
- new net: L211.2, L212.1
- new net: L183.2, L184.1
- new net: L216.2, L217.1
- new net: L217.2, L218.1
- new net: L174.2, L175.1
- new net: L175.2, L176.1
- new net: L202.2, L203.1
- new net: L203.2, L204.1
- new net: L180.2, L181.1
- new net: L165.2, L166.1
- new net: L224.2, L225.1
- new net: L178.2, L179.1
- new net: L179.2, L180.1
- new net: L204.2, L205.1
- new net: L192.2, L193.1
- new net: L193.2, L194.1
- new net: L220.2, L221.1
- new net: L221.2, L222.1
- new net: L200.2, L201.1
- new net: L201.2, L202.1
- new net: L207.2, L208.1
- new net: L208.2, L209.1
- new net: L205.2, L206.1
- new net: L206.2, L207.1
- new net: L187.2, L188.1
- new net: L210.2, L211.1
- new net: L168.2, L169.1
- new net: L219.2, L220.1
- new net: L190.2, L191.1
- new net: L173.2, L174.1
- new net: L186.2, L187.1
- new net: L209.2, L210.1
- new net: L191.2, L192.1
- new net: L218.2, L219.1
Other:
- note added: "2x (33 x 0.47uH = 15.51uH @ 1.188Ω) = 7.755μH @ 0.594Ω SRF=170MHz I>3A"
- note added: "=Sokal's 'C1' to be calculated"
- note added: "ALL ARE SWITCHED BASED ON FREQUENCY AND NOMINALLY ADJACENT. IT LIKELY MAKES SENSE TO CREATE A UNIFORM INTERFACE AND PHYSICAL MODULE."
- note added: "PA-DRAIN"
- note added: "PA-SUPPLY"
- note added: "RFC-GND"
- note added: "xΩ xuH >xmA SRF>xMHz"
- note removed: "For 2200m through 160m bands (135 kHz - 2 MHz): Inductance: 100-470 μH (series combination may be necessary) Current rating: 100-500 mA (application dependent) Self-resonant frequency (SRF): Above 2 MHz Package size: 1008 (2520 metric) or larger DCR: As low as possible, typically <1 Ω Recommendations: Use multiple high-value SMD inductors in series Consider ferrite core SMD inductors for higher i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"
- note removed: "For 60m through 2m bands (5 MHz - 144 MHz): Inductance: 1-10 μH Current rating: 100-500 mA (application dependent) Self-resonant frequency (SRF): Above 150 MHz Q factor: >50 at operating frequencies Package size: 0805 (2012 metric) or 0603 (1608 metric) DCR: <0.5 Ω Recommendations: Use multi-layer or wire-wound SMD inductors for better Q factor Consider series combination of smaller value inducto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"
- moved on the sheet: L141, L142, L143, L144, L145, L146, L147, L148, L149, L150, L151, L152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

Commit message: Rationalize
Parts:
- removed J10: BANDMODULE3-ANT, Connector_PinSocket_2.54mm:PinSocket_1x07_P2.54mm_Vertical, symbol Connector_Generic:Conn_01x07
- removed J11: BANDMODULE4-ANT, Connector_PinSocket_2.54mm:PinSocket_1x07_P2.54mm_Vertical, symbol Connector_Generic:Conn_01x07
- removed J12: BANDMODULE3-PA, Connector_PinSocket_2.54mm:PinSocket_1x07_P2.54mm_Vertical, symbol Connector_Generic:Conn_01x07
- removed J13: BANDMODULE4-PA, Connector_PinSocket_2.54mm:PinSocket_1x07_P2.54mm_Vertical, symbol Connector_Generic:Conn_01x07
- removed J14: BANDMODULE5-ANT, Connector_PinSocket_2.54mm:PinSocket_1x07_P2.54mm_Vertical, symbol Connector_Generic:Conn_01x07
- removed J15: BANDMODULE6-ANT, Connector_PinSocket_2.54mm:PinSocket_1x07_P2.54mm_Vertical, symbol Connector_Generic:Conn_01x07
- removed J16: BANDMODULE5-PA, Connector_PinSocket_2.54mm:PinSocket_1x07_P2.54mm_Vertical, symbol Connector_Generic:Conn_01x07
- removed J17: BANDMODULE6-PA, Connector_PinSocket_2.54mm:PinSocket_1x07_P2.54mm_Vertical, symbol Connector_Generic:Conn_01x07
- removed J6: BANDMODULE1-ANT, Connector_PinSocket_2.54mm:PinSocket_1x07_P2.54mm_Vertical, symbol Connector_Generic:Conn_01x07
- removed J7: BANDMODULE1-PA, Connector_PinSocket_2.54mm:PinSocket_1x07_P2.54mm_Vertical, symbol Connector_Generic:Conn_01x07
- removed J8: BANDMODULE2-ANT, Connector_PinSocket_2.54mm:PinSocket_1x07_P2.54mm_Vertical, symbol Connector_Generic:Conn_01x07
- removed J9: BANDMODULE2-PA, Connector_PinSocket_2.54mm:PinSocket_1x07_P2.54mm_Vertical, symbol Connector_Generic:Conn_01x07
- renumbered C8 to C10, C9 to C11, C10 to C12, C11 to C13, C12 to C14, C13 to C15, C14 to C16, C15 to C17, C16 to C18, C17 to C19, C18 to C20, C19 to C21, C20 to C22, C21 to C23, C22 to C24, C23 to C25, C24 to C26, C25 to C27, C26 to C28, C43 to C29, C42 to C30, C41 to C31, C27 to C32, C40 to C33, C39 to C34, C38 to C35, C28 to C7, C7 to C8, C29 to C9, D34 to D8, J19 to J3, J3 to J4, J18 to J5, J4 to J6, J5 to J7, J20 to J8, L141 to L10, L145 to L11, L148 to L12, L151 to L13, L154 to L14, L142 to L15, L146 to L16, L149 to L17, L152 to L18, L155 to L19, L156 to L20, L157 to L21, L158 to L22, L159 to L23, L162 to L24, L163 to L25, L164 to L26, L165 to L27, L166 to L28, L167 to L29, L168 to L30, L169 to L31, L170 to L32, L171 to L33, L172 to L34, L173 to L35, L174 to L36, L175 to L37, L176 to L38, L177 to L39, L178 to L40, L179 to L41, L180 to L42, L181 to L43, L182 to L44, L183 to L45, L184 to L46, L185 to L47, L186 to L48, L187 to L49, L143 to L5, L188 to L50, L189 to L51, L190 to L52, L191 to L53, L192 to L54, L193 to L55, L194 to L56, L160 to L57, L161 to L58, L195 to L59, L144 to L6, L196 to L60, L197 to L61, L198 to L62, L199 to L63, L200 to L64, L201 to L65, L202 to L66, L203 to L67, L204 to L68, L205 to L69, L147 to L7, L206 to L70, L207 to L71, L208 to L72, L209 to L73, L210 to L74, L211 to L75, L212 to L76, L213 to L77, L214 to L78, L215 to L79, L150 to L8, L216 to L80, L217 to L81, L218 to L82, L219 to L83, L220 to L84, L221 to L85, L222 to L86, L223 to L87, L224 to L88, L225 to L89, L153 to L9, R8 to R10, R9 to R11, R10 to R12, R11 to R13, R12 to R14, R13 to R15, R14 to R4, R15 to R5, R4 to R6, R5 to R7, R6 to R8, R7 to R9, U4 to U1, U1 to U2, U2 to U3, U3 to U4
Other:
- removed sheet BM1-SWITCH-ANT
- removed sheet BM1-SWITCH-PA
- removed sheet BM2-SWITCH-ANT
- removed sheet BM2-SWITCH-PA
- removed sheet BM3-SWITCH-ANT
- removed sheet BM3-SWITCH-PA
- removed sheet BM4-SWITCH-ANT
- removed sheet BM4-SWITCH-PA
- removed sheet BM5-SWITCH-ANT
- removed sheet BM5-SWITCH-PA
- removed sheet BM6-SWITCH-ANT
- removed sheet BM6-SWITCH-PA5
- note added: "ANTENNA CONNECTION"
- note added: "BATTERIES"
- note added: "DC INPUT"
- note added: "LPF IN HERE"
- note added: "MAIN BOARD"
- note added: "PA / LPF"
- note added: "PA/LPF INTERFACE"
- note added: "POTENTIAL PHYSICAL LAYER ARCHITECTURES UNDER 'TIFFIN' PROPOSAL"
- note added: "POWER INTERFACE"
- note added: "SCREEN"
- note added: "THIRD PARTY CHARGE CONTROL MODULE"
- note added: "THIRD PARTY SCREEN MODULE"
- note added: "USBC/USB-PD DC INPUT"

Commit message: Significant updates
Parts:
- removed J3: IPEX-1, symbol Connector:Conn_Coaxial_Small
- removed J5: MMCX, Connector_Coaxial:MMCX_Molex_73415-1471_Vertical, symbol Connector:Conn_Coaxial_Small
- removed J6: SMA, Connector_Coaxial:SMA_Amphenol_901-144_Vertical, symbol Connector:Conn_Coaxial_Small
- added C44, C45: 10uF, Capacitor_SMD:C_1206_3216Metric, symbol Device:C_Small
- added D24, D25: 1N4148WS, Diode_SMD:D_SOD-323, symbol Diode:1N4148WS
- added FB3: 100mΩ/3A, Capacitor_SMD:C_1206_3216Metric, symbol Device:FerriteBead_Small
- added J3: USBC, symbol Connector:USB_C_Receptacle
- added J5: USB_A, Connector_USB:USB_Mini-B_Wuerth_65100516121_Horizontal, symbol Connector:USB_A
- added R77: R_Small_US, symbol Device:R_Small_US
- added R78: 5.1K, Resistor_SMD:R_0805_2012Metric, symbol Device:R_Small_US
- added R79, R80, R81, R82, R83, R84: 100K, Resistor_SMD:R_1206_3216Metric, symbol Device:R_Small_US
- added U7: TUSB321, Package_DFN_QFN:Texas_X2QFN-12_1.6x1.6mm_P0.4mm, symbol Interface_USB:TUSB321
- added U8: MT3608, Package_TO_SOT_SMD:SOT-23-6, symbol Regulator_Switching:MT3608
- J7: value 12V SUPPLY -> 12-24V SUPPLY
Connections:
- net ANTENNA is gone; now on net ANTENNA-A: J4.1 (In)
- net ANTENNA-B: now also J4.2 (Ext)
- net GND: now also C44.1, C45.1, J3.A1 (GND), J3.A12 (GND), J3.B1 (GND), J3.B12 (GND), J3.S1 (SHIELD), J5.4 (GND), J5.5 (Shield), R78.2, U7.10 (GND), U7.4 (PORT), U8.2 (GND); no longer J4.2 (Ext)
- net HOST-FSK-INPUT: no longer C8.2, R12.2
- net RECEIVED-AUDIO: no longer C4.2
- net VIN-DIRTY: now reaches FB1.1, J7.1
- net VIN-COMMON: now reaches C18.1, C20.1, C23.2, C25.2, L4.1
- net VIN-COMMON: now also D24.2 (A), D25.2 (A); no longer D7.2 (A2), FB1.2
- net VIN: now reaches L4.2, U3.1 (IN)
- new net: R84.1, U7.3 (CURRENT_MODE)
- new net: R83.2, R84.2
- new net: C8.2, R12.2
- new net: R81.1, R82.2
- new net: R79.1, R81.2
- new net: R78.1, R80.1, U8.3 (FB)
- new net: R77.2, U7.5 (VBUS_DET)
- new net: FB3.1, U7.12 (VDD)
- new net: R82.1, R83.1
- new net IFAULT-WHEN-LOW: U7.6 (~{VCONN_FAULT})
- new net IMODE1: U7.7 (OUT1)
- new net IMODE2: U7.8 (OUT2)
- new net USB-A-D+: J5.3 (D+)
- new net USB-A-D-: J5.2 (D-)
- new net USB-A-VBUS: J5.1 (VBUS)
- new net USB-C-CC1: J3.A5 (CC1), U7.1 (CC1)
- new net USB-C-CC2: J3.B5 (CC2), U7.2 (CC2)
- new net USB-C-USB2-D+: J3.A6 (D+), J3.B6 (D+)
- new net USB-C-USB2-D-: J3.A7 (D-), J3.B7 (D-)
- new net USB-C-VBUS: J3.A4 (VBUS), J3.A9 (VBUS), J3.B4 (VBUS), J3.B9 (VBUS), R77.1
- new net VDD-USBC-CLEAN: FB3.2, R79.2, U8.4 (EN), U8.5 (IN)
- new net VIN-CLAMPED: D25.1 (K), D7.2 (A2), FB1.2
- new net VIN-USBC: C44.2, C45.2, D24.1 (K), R80.2, U8.1 (SW)
- no-connect marks 16 -> 28
Other:
- note added: "- Needs footprint"
- note added: "- Needs to be selected SL2.1s (C2684433) @ $0.20 - Needs footprint"
- note added: "12V 0.5A NOMINAL"
- note added: "12V-24V NOMINAL"
- note added: "12V-36V NOMINAL"
- note added: "500K RESISTANCE TO REQUEST 5V @ 1.5A"
- note added: "5V 1.5A NOMINAL"
- note added: "ADD PULLUPS/PULLDOWNS FOR ALL IMPORTANT PINS REST OF PA ANTENNA MATCHING NETWORK OR ATU ADD/TEST ANTENNA CABLE DETECTION ADD OPTIONAL SQUEAKER ADD TEST POINTS"
- note added: "BOOST IC IN > 3V OUT <= 28V"
- note added: "CM108 AUDIO"
- note added: "EMI SOURCE"
- note added: "EXPECTED TO GENERATE NOISE AT A VARIABLE SWITCHING FREQUENCY BETWEEN 0.9-1.1MHZ WHICH FALLS BETWEEN THE 160M AND 630M AMATEUR RADIO BANDS."
- note added: "FEEDBACK VOLTAGE 0.6V MEANS 12V:0.6V SO 19:1 RATIO OF RESISTANCE"
- note added: "HOST USBC POWER AND DATA CONNECTION"
- note added: "MCU CONNECTION"
- note added: "ONBOARD USB2 HUB"
- note added: "SET TO UFP MODE (POWER CONSUMER)"
- note added: "SIDEBAND UTILITY PINS (UNUSED)"
- note added: "THESE INDICATE DETECTED CURRENT MODE TO MCU"
- note added: "USB PD LINES"
- note added: "USB2.0 DATA PINS"
- note added: "USB3.1 DATA PINS"
- note removed: "ADD PULLUPS/PULLDOWNS FOR ALL IMPORTANT PINS REST OF PA ANTENNA MATCHING NETWORK OR ATU ADD/TEST AUDIO + ANTENNA CABLE DETECTION ADD MORE MOSFET SWITCHES ADD SOME KIND OF MULTIPLEXING? ADD OPTIONAL INTERFACE PCB - EASY MOUNTING AT RIGHT ANGLES ADD OPTIONAL SQUEAKER ADD TEST POINTS EITHER PREVENT RADIO POWERUP USING USB-SUPPLIED POWER (EG. 12V SUPPLY PRESENCE ENABLES 5V LINE) OR CONSIDER POWER LIM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"
- moved on the sheet: A1, C10, C11, C12, C13, C14, C15, C16, C17, C18, C19, C20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

Commit message: Toward one USB cable
Parts:
- added C46, C47: 33pF, Capacitor_SMD:C_0603_1608Metric, symbol Device:C_Small
- added R76: 1K, Resistor_SMD:R_1206_3216Metric, symbol Device:R_Small_US
- added R85, R86: 5.1K, Resistor_SMD:R_0805_2012Metric, symbol Device:R_Small_US
- added R87, R88, R89, R90: 22, Resistor_SMD:R_0805_2012Metric, symbol Device:R_Small_US
- added U10: CM108B, Package_QFP:LQFP-48_7x7mm_P0.5mm, symbol adxi-symbols:CM108B
- added U11: 93C46, Package_SO:TSSOP-8_4.4x3mm_P0.65mm, symbol Memory_EEPROM:93CxxA
- added U9: SL2.1s, symbol adxi-symbols:SL2.1s
- added Y1: 12MHz, Crystal:Crystal_SMD_3225-4Pin_3.2x2.5mm, symbol Device:Crystal_GND24
Connections:
- net USB-A-VBUS is gone; now on net 5V: J5.1 (VBUS)
- net 3.3V: now also R86.1, U9.9 (VDD33)
- net 5V: now also U11.8 (VCC), U9.7 (VDD5)
- net GND: now also C46.2, C47.2, R85.2, U10.33 (AVSS), U10.36 (DVSS), U11.5 (GND), U9.8 (VSS), Y1.2, Y1.4
- net HOST-FSK-INPUT: now also U10.30 (LOL), U10.32 (LOR)
- net RECEIVED-AUDIO: now also U10.27 (MCIN)
- net USB-A-D+: now also U9.2 (DP2)
- net USB-A-D-: now also U9.1 (DM2)
- net USB-C-USB2-D+: now also R90.2, U9.6 (UDP); no longer J3.A6 (D+), J3.B6 (D+)
- net USB-C-USB2-D-: now also R89.2, U9.5 (UDM); no longer J3.A7 (D-), J3.B7 (D-)
- new net: J3.A7 (D-), J3.B7 (D-), R89.1
- new net: C46.1, U9.12 (XIN), Y1.1
- new net: C47.1, U9.11 (XOUT), Y1.3
- new net: R88.1, U10.41 (USBDP)
- new net: R76.2, R85.1
- new net: U10.5 (CS), U11.1 (CS)
- new net: U10.4 (SK), U11.2 (SCLK)
- new net: U10.3 (DW), U11.3 (DI)
- new net: U10.2 (DR), U11.4 (DO)
- new net: R87.1, U10.42 (USBDM)
- new net: J3.A6 (D+), J3.B6 (D+), R90.1
- new net 1.8V: R76.1, R86.2, U9.10 (VDD18)
- new net USB-CM108-D+: R88.2, U9.4 (DP1)
- new net USB-CM108-D-: R87.2, U9.3 (DM1)
- no-connect marks 28 -> 32
Other:
- note added: ".."
- note added: "3.3V TO 1.8V VOLTAGE DIVIDER"
- note added: "5.1K"
- note added: "6.1K"
- note added: "EEPROM POSSIBLY NOT REQ'D"
- note added: "EXTERNAL 5V"
- note added: "LOAD CAPACITANCE VALUES CALCULATED BASED UPON CL=20pF"
- note added: "MAY NEED PULLUPS OR 3.3V"
- note added: "MISSING INDUCTOR"
- note added: "MISSING RESISTOR VALUE"
- note added: "ONBOARD USB2.0 4 PORT HUB"
- note added: "POSSIBLE TO USE THIS OUTPUT TO TEST THE FILTER CONFIGURATION? COULD ALSO GENERATE 12MHz OSCILLATION REQUIRED FOR THE USB HUB."
- note added: "SEE doc/audio-summing"
- note removed: "- Needs footprint"
- note removed: "- Needs to be selected SL2.1s (C2684433) @ $0.20 - Needs footprint"
- note removed: "CM108 AUDIO"
- note removed: "ONBOARD USB2 HUB"
- note removed: "POSSIBLE TO USE THIS OUTPUT TO TEST THE FILTER CONFIGURATION?"

Commit message: USB work
Parts:
- removed C2, C3: 100nF, Capacitor_SMD:C_0805_2012Metric, symbol Device:C_Small
- removed C4: 470nF, symbol Device:C_Small
- removed C6, C8: 10nF, symbol Device:C_Small
- removed J1: FROM-PC-SPK, Connector_Audio:Jack_3.5mm_CUI_SJ1-3525N_Horizontal, symbol Connector_Audio:AudioJack3
- removed J2: TO-PC-MIC, Connector_Audio:Jack_3.5mm_CUI_SJ1-3525N_Horizontal, symbol Connector_Audio:AudioJack3
- removed R12, R8: 10K, Resistor_SMD:R_1206_3216Metric, symbol Device:R_Small_US
- removed R6: 1M, symbol Device:R_Small_US
- removed R7: 4.7K, symbol Device:R_Small_US
- added C48, C49, C51, C53, C58: 100nF, Capacitor_SMD:C_0603_1608Metric, symbol Device:C_Small
- added C50, C52, C54, C59: 10uF, Capacitor_SMD:C_0603_1608Metric, symbol Device:C_Small
- added C55: 1uF, symbol Device:C_Small
- added C56: 100nF, symbol Device:C_Small
- added C57: 10nF, symbol Device:C_Small
- added R91, R92, R93, R94, R95: 10K, Resistor_SMD:R_0402_1005Metric, symbol Device:R_Small_US
- J3: footprint (none) -> adxi-footprints:TYPE-C-SMD_C9900025773; LCSC Part # (none) -> C5156605; MPN (none) -> TYPE-C 24P QT 143; Manufacturer (none) -> Shou Han
- J5: value USB_A -> USB2 Type-A; footprint Connector_USB:USB_Mini-B_Wuerth_65100516121_Horizontal -> adxi-footprints:USB-A-SMD_10.0-QTJ6.3; LCSC Part # C2688795 -> C404966; MPN KH-MINI-SMT-5P-Cu -> 10.0 QTJ6.3; Manufacturer Shenzhen Kinghelm Elec -> Shou Han
- U9: footprint (none) -> adxi-footprints:SSOP-16_L4.6-W2.6-P0.53-LS4.0-BL
Connections:
- net 1.8V: now also C49.1
- net 3.3V: now also U10.7 (PWRSEL), U11.8 (VCC), C48.1, C50.1, C58.1, C59.1, R91.1, R92.1, R93.1, R94.1, R95.1
- net 5V: now also U10.29 (AVDD), U10.34 (AVDD), U10.35 (DVDD), C51.1, C52.1, C55.2, C56.1, C57.1; no longer U11.8 (VCC)
- net GND: now also U10.10 (MODE), U10.14 (DVSS), U10.22 (ADSEL), U10.23 (TEST), U10.24 (AVSS), U10.38 (MSEL), C48.2, C49.2, C50.2, C51.2, C52.2, C53.2, C54.2, C55.1, C56.2, C57.2, C58.2, C59.2
- net LEDO: now reaches U10.12 (LEDO)
- net MUTE-PLAYBACK-WHEN-LOW: now reaches U10.18 (MUTEP)
- net MUTE-PLAYBACK-WHEN-LOW: now also R92.2
- net LEDR: now reaches U10.21 (LEDR)
- net at U10.26 (VREF): now also C53.1, C54.1
- net VOLUME-UP-BUTTON-WHEN-LOW: now reaches U10.39 (VOLUP)
- net VOLUME-UP-BUTTON-WHEN-LOW: now also R95.2
- net PDSW: now reaches U10.40 (PDSW)
- net PDSW: now also R93.2
- net VOLDN: now reaches U10.48 (VOLDN)
- net VOLDN: now also R94.2
- net MUTE-RECORDING-WHEN-LOW: now reaches U10.6 (MUTER)
- net MUTE-RECORDING-WHEN-LOW: now also R91.2
- no-connect marks 32 -> 43
Other:
- note added: ""100mA""
- note added: ""3V MICROPHONE BIAS DRIVE""
- note added: ""AA PATH DISABLED""
- note added: ""INTERNAL ADC""
- note added: ""NORMAL OPERATION""
- note added: "10K IS CHOSEN TO CONSERVE POWER SINCE THE REACTION TIME IS NON-CRITICAL."
- note added: "ADXI"
- note added: "IGNORE I2S"
- note added: "IGNORE SPDIF"
- note added: "ONBOARD USB2.0 AUDIO DONGLE"
- note added: "REC. ENABLED "HEADSET MODE""
- note added: "REQUIRES 3.3V LEVEL CONVERSION"
- note added: "SEE doc/usb-audio"
- note added: "SEE doc/usb-hub"
- note added: "SELECTED DESIGN (INITIAL FOCUS)"
- note added: "THESE ARE PULLED DOWN TO THEIR "ACTIVE LOW" STATES BY THE SPI GPIO EXPANSION SYSTEM."
- note added: "VK2DIY"
- note removed: "AUDIO INPUT FROM COMPUTER"
- note removed: "AUDIO OUTPUT TO COMPUTER"
- note removed: "Audio interface consists of a Speaker input from PC sound card which is actually an input to Arduino nano analog comparator for tone frequency detection and sampling. Before inputting signal to analog comparator of Arduino it passes through a band pass filter which has an audio band pass frequency range of 500 Hz to 3500 Hz."
- note removed: "BAND PASS FILTER (CLAIM: "500Hz-3.5KHz")"
- note removed: "HOST AUDIO INTERFACE"
- note removed: "MAY NEED PULLUPS OR 3.3V"
- moved on the sheet: C46, C47, R87, R88, U10, U11, U9, Y1

Commit message: Another model
Parts:
- added D26: 1N4148WS, Diode_SMD:D_SOD-323, symbol Diode:1N4148WS
- added FB4, FB5: 100mΩ/3A, Capacitor_SMD:C_1206_3216Metric, symbol Device:FerriteBead_Small
- added L226: 22uH, adxi-footprints:IND-SMD_L10.8-W10.0, symbol Device:L
- added R100, R12, R6, R7, R8, R96, R97, R98, R99: 1K, Resistor_SMD:R_0603_1608Metric, symbol Device:R_Small_US
- U8: value MT3608 -> MT3608B; LCSC Part # (none) -> C19189893; MPN (none) -> MT3608B; Manufacturer (none) -> Xi'an Aerosemi Tech
Connections:
- net GND: now also R100.1, R8.1, R97.1
- net IFAULT-WHEN-LOW: now also A1.9 (D6)
- net IMODE1: now also A1.7 (D4)
- net IMODE2: now also A1.8 (D5)
- net SPI-MOSI: now also R6.1
- net SPI-SCK: now also R98.1
- net SPI-SS-OUTPUTS: now also R12.1
- net USB-C-CC1: now also FB4.2; no longer U7.1 (CC1)
- net USB-C-CC2: now also FB5.2; no longer U7.2 (CC2)
- net VDD-USBC-CLEAN: now also L226.2
- net VIN-CLAMPED: now also D25.2 (A); no longer D25.1 (K)
- net VIN-COMMON: now also D24.1 (K), D25.1 (K); no longer D24.2 (A), D25.2 (A)
- net VIN-USBC: now also D24.2 (A), D26.1 (K); no longer D24.1 (K), U8.1 (SW)
- new net: R96.1, R97.2
- new net: R100.2, R99.1
- new net: FB5.1, U7.2 (CC2)
- new net: FB4.1, U7.1 (CC1)
- new net: D26.2 (A), L226.1, U8.1 (SW)
- new net: R7.1, R8.2
- new net SPI-MOSI-3.3V: R6.2, R7.2
- new net SPI-SCK-3.3V: R98.2, R99.2
- new net SPI-SS-OUTPUTS-3.3V: R12.2, R96.2
Other:
- note added: "= UFP MODE (POWER CONSUMER)"
- note added: "BOOST IC VIN = 5V VOUT = 12V"
- note added: "NOISE AT F=0.9-1.2MHZ"
- note added: "OUTPUT EXPANSION"
- note added: "SEE docs/power-supply"
- note added: "SEE docs/spi-level-conversion"
- note added: "SPI LEVEL CONVERSION 5V TO 3.3V"
- note removed: "BOOST IC IN > 3V OUT <= 28V"
- note removed: "EXPECTED TO GENERATE NOISE AT A VARIABLE SWITCHING FREQUENCY BETWEEN 0.9-1.1MHZ WHICH FALLS BETWEEN THE 160M AND 630M AMATEUR RADIO BANDS."
- note removed: "MISSING INDUCTOR"
- note removed: "SET TO UFP MODE (POWER CONSUMER)"
- note removed: "THIS ONE SHOULD BE POSSIBLE TO HARD WIRE IF REQUIRED"
- moved on the sheet: C18, C20, C23, C25, C44, C45, C58, C59, D24, D25, D7, FB1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

Commit message: Updates
Parts:
- removed FB3, FB4, FB5: 100mΩ/3A, Capacitor_SMD:C_1206_3216Metric, symbol Device:FerriteBead_Small
- added FB6, FB7, FB8: 100mΩ/3A, Capacitor_SMD:C_1206_3216Metric, symbol Device:FerriteBead_Small
- added TP1: 12V, TestPoint:TestPoint_Plated_Hole_D2.0mm, symbol Connector:TestPoint
- added TP10: 3.3V, TestPoint:TestPoint_Plated_Hole_D2.0mm, symbol Connector:TestPoint
- added TP11: RFC-GND, TestPoint:TestPoint_Plated_Hole_D2.0mm, symbol Connector:TestPoint
- added TP12: PA-SUPPLY, TestPoint:TestPoint_Plated_Hole_D2.0mm, symbol Connector:TestPoint
- added TP13: PA-DRAIN, TestPoint:TestPoint_Plated_Hole_D2.0mm, symbol Connector:TestPoint
- added TP2: VIN-COM, TestPoint:TestPoint_Plated_Hole_D2.0mm, symbol Connector:TestPoint
- added TP3: VIN-USBC, TestPoint:TestPoint_Plated_Hole_D2.0mm, symbol Connector:TestPoint
- added TP4: VDD-USBC, TestPoint:TestPoint_Plated_Hole_D2.0mm, symbol Connector:TestPoint
- added TP5: VIN-CLAMPED, TestPoint:TestPoint_Plated_Hole_D2.0mm, symbol Connector:TestPoint
- added TP6: USBCVB, TestPoint:TestPoint_Plated_Hole_D2.0mm, symbol Connector:TestPoint
- added TP7: FPWR, TestPoint:TestPoint_Plated_Hole_D2.0mm, symbol Connector:TestPoint
- added TP8: RPWR, TestPoint:TestPoint_Plated_Hole_D2.0mm, symbol Connector:TestPoint
- added TP9: 5V, TestPoint:TestPoint_Plated_Hole_D2.0mm, symbol Connector:TestPoint
- R77: value R_Small_US -> 909K; footprint (none) -> Resistor_SMD:R_1206_3216Metric; LCSC Part # (none) -> C323176; MPN (none) -> RS-06K9093FT; Manufacturer (none) -> Fenghua
Connections:
- net 12V: now also TP1.1
- net 3.3V: now also TP10.1
- net 5V: now also TP9.1
- net ANTENNA-A: now also TP12.1
- net FORWARD-POWER: now also TP7.1
- net PA Switched Resonator/PA-DRAIN: now also TP13.1
- net REVERSE-POWER: now also TP8.1
- net USB-C-CC1: now also U7.1 (CC1), FB7.2; no longer J3.A5 (CC1)
- net USB-C-CC2: now also U7.2 (CC2), FB8.2; no longer J3.B5 (CC2)
- net USB-C-VBUS: now also FB6.2; no longer J3.A4 (VBUS), J3.A9 (VBUS), J3.B4 (VBUS), J3.B9 (VBUS)
- net VDD-USBC-CLEAN: now also U7.12 (VDD), TP4.1
- net VIN-CLAMPED: now also TP5.1
- net VIN-COMMON: now also TP2.1
- net VIN-USBC: now also TP3.1
- net at C29.1, C30.1, C31.1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: now also TP11.1
- net USBCVB: now reaches R77.2, U7.5 (VBUS_DET)
- net USBCVB: now also TP6.1
- new net: FB7.1, J3.A5 (CC1)
- new net: FB8.1, J3.B5 (CC2)
- new net: FB6.1, J3.A4 (VBUS), J3.A9 (VBUS), J3.B4 (VBUS), J3.B9 (VBUS)
Other:
- note added: "ADD PULLUPS/PULLDOWNS REST OF PA ANTENNA MATCHING NETWORK OR ATU ADD/TEST ANTENNA CABLE DETECTION ADD OPTIONAL SQUEAKER ADD TEST POINTS"
- note added: "F=0.9-1.2MHz (1.2MHz NOMINAL)"
- note added: "HARMONICS 180-240kHz 225-300kHz 300-400kHz 450-600kHz 600-800kHz 1.8-2.4MHz 2.7-3.6MHz 3.6-4.8MHz 4.5-6MHz"
- note added: "TEST POINTS"
- note added: "USB BUS 5V SUPPLY"
- note removed: "ADD PULLUPS/PULLDOWNS FOR ALL IMPORTANT PINS REST OF PA ANTENNA MATCHING NETWORK OR ATU ADD/TEST ANTENNA CABLE DETECTION ADD OPTIONAL SQUEAKER ADD TEST POINTS"
- note removed: "EXTERNAL 5V"
- note removed: "MISSING RESISTOR VALUE"
- note removed: "NOISE AT F=0.9-1.2MHZ"
- moved on the sheet: C1, C18, C20, C23, C25, C44, C45, C5, C7, C9, D1, D2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
