File: kicad-pcbs/adxi/adxi.kicad_sch (KiCad schematic)
At the start: 223 parts, among them J3 USBC, J4 BNC, J5 USB2 Type-A, J7 12-24V SUPPLY, J8 LCD-2004, Q1 MMBF170, Q2 HY1904C2, U1 Si5351A-B-GT, U10 CM108B, U11 93C46, U2 CD2003, U3 L7812, U4 74ACT244, U7 TUSB321, U8 MT3608B, U9 SL2.1s, Y1 12MHz

Commit message: Update
Parts:
- removed FB2: 100mΩ/3A, Capacitor_SMD:C_1206_3216Metric, symbol Device:FerriteBead_Small
- removed J4: BNC, Connector_Coaxial:BNC_TEConnectivity_1478204_Vertical, symbol Connector:Conn_Coaxial
- removed J8: LCD-2004, Connector_PinHeader_2.54mm:PinHeader_1x04_P2.54mm_Vertical, symbol Connector_Generic:Conn_01x04
- removed L10, L11, L12, L13, L14, L15, L16, L17, L18, L19: 18nH, Inductor_SMD:L_1210_3225Metric, symbol Device:L
- removed L20, L21, L22, L23: 100uH, Inductor_SMD:L_Cenker_CKCS8040, symbol Device:L
- removed L24, L25, L26, L27, L28, L29, L30, L31, L32, L33, L34, L35, L36, L37, L38, L39, L40, L41, L42, L43, L44, L45, L46, L47, L48, L49, L50, L51, L52, L53, L54, L55, L56, L57, L58, L59, L60, L61, L62, L63, L64, L65, L66, L67, L68, L69, L70, L71, L72, L73, L74, L75, L76, L77, L78, L79, L80, L81, L82, L83, L84, L85, L86, L87, L88, L89: 470nH, Inductor_SMD:L_1008_2520Metric, symbol Device:L
- removed L5, L6, L7, L8, L9: 33nH, Inductor_SMD:L_1210_3225Metric, symbol Device:L
- removed R79, R81, R82, R83, R84: 100K, Resistor_SMD:R_1206_3216Metric, symbol Device:R_Small_US
- removed U11: 93C46, Package_SO:TSSOP-8_4.4x3mm_P0.65mm, symbol Memory_EEPROM:93CxxA
- added C36: 18pF, Capacitor_SMD:C_0402_1005Metric, symbol Device:C_Small
- added D10, D11: BZT52C5V6, Diode_SMD:D_SOD-123, symbol Device:D_Zener
- added R101, R102: 1K, Resistor_SMD:R_0603_1608Metric, symbol Device:R_Small_US
- added R20, R21: 10K, Resistor_SMD:R_1206_3216Metric, symbol Device:R_Small_US
- added R22, R23: 1K, Resistor_SMD:R_1206_3216Metric, symbol Device:R_Small_US
- added Y2: 25MHz, Crystal:Crystal_SMD_3225-4Pin_3.2x2.5mm, symbol Device:Crystal_GND24
- C35: value C_Small -> 18pF; footprint (none) -> Capacitor_SMD:C_0402_1005Metric; LCSC Part # (none) -> C1549; MPN (none) -> 0402CG180J500NT; Manufacturer (none) -> Fenghua
- U1: value Si5351A-B-GT -> SI5351A-B-GTR; LCSC Part # (none) -> C504891; MPN (none) -> SI5351A-B-GTR; Manufacturer (none) -> Skyworks
Connections:
- net LEDR is gone; now on net CM108B-LEDR: U10.21 (LEDR)
- net PA-OUTPUT is gone; now on net PA-DRAIN: R1.2, R9.2
- net PA-POWER-PWM is gone; now on net CM108B-LEDO: A1.6 (D3)
- net FORWARD-POWER: now also R22.1
- net GND: now also C35.2, C36.2, D10.1 (K), D11.1 (K), R20.1, R21.1, Y2.2, Y2.4
- net HOST-FSK-INPUT: now also R101.1, R102.1; no longer U10.30 (LOL), U10.32 (LOR)
- net IFAULT-WHEN-LOW: no longer A1.9 (D6)
- net PA-DRIVE-PWM: now also A1.12 (D9)
- net REVERSE-POWER: now also R23.1
- net at R11.2: now also R21.2; no longer D4.2 (A)
- net at R3.2: now also R20.2; no longer D2.2 (A)
- net Late Stage Interface/RFC-GND: now reaches C29.1, C30.1, C31.1, C33.1, C34.1, D8.2 (A), TP11.1
- net at U1.2 (XA): now also C36.1, Y2.3
- net at U1.3 (XB): now also C35.1, Y2.1
- net CM108B-LEDR: now reaches A1.5 (D2)
- net HOST-FSK-BIAS: now reaches U10.31 (LOBS)
- net ANTENNA-A renamed Late Stage Interface/PA-SUPPLY
- net Late Stage Interface/PA-SUPPLY: now also D10.2 (A); no longer C35.2
- net LEDO renamed CM108B-LEDO
- net PA Switched Resonator/PA-DRAIN renamed PA-DRAIN
- net PA-DRAIN: now also D11.2 (A); no longer C35.1
- net RECEIVED-DATA renamed RECEIVED-SIGNAL
- new net: R102.2, U10.30 (LOL)
- new net: D2.2 (A), R22.2
- new net: D4.2 (A), R23.2
- new net: R101.2, U10.32 (LOR)
- no-connect marks 43 -> 57
Other:
- sheet PA-POWER-PWM renamed PA Transmit Power Modulation
- removed sheet PA Switched Resonator
- added sheet Late Stage Interface (late-stage-interface.kicad_sch)
- added sheet pa-lpf-ant (pa-lpf-ant.kicad_sch)
- sheet Digital output expansion ports: added none; removed O-10, O-11, O-12, O-13, O-14, O-15, O-16, O-9
- note added: ""GOOD ENOUGH" FORWARD/REVERSE POWER AND SWR, ANTENNA ABSENCE OR BREAKAGE DETECTION. RULE OF THUMB: "OPERATE SWR <4" "SURVIVE SWR <10""
- note added: "(11K)"
- note added: "(20K)"
- note added: "0-12V NOMINAL"
- note added: "0-4.2V NOMINAL"
- note added: "3.3V OUTPUTS"
- note added: "5.6V CLAMP"
- note added: "ADD PULLUPS/PULLDOWNS ADD OPTIONAL SQUEAKER ADD TEST POINTS"
- note added: "CD2003GP IS A CLONE OF TA2003, ITSELF A PIN-COMPATIBLE UPGRADE TO TA8164. ONLY THE AM SECTION IS USED AS A DIRECT CONVERSION RECEIVER."
- note added: "EEPROM IS NOT SUPPORTED AS IT ONLY ALLOWS CUSTOM USB DEVICE IDENTIFICATION"
- note added: "For effective power supply noise filtering, a design guideline is to use ferrite beads at about 20% of their rated DC current. We anticipate ~0.425A peak which is ~14%."
- note added: "INTENTIONALLY WITHOUT PULLUP"
- note added: "LOAD CAPACITANCE VALUES CALCULATED BASED UPON CL=12pF"
- note added: "MCU MODULE"
- note added: "NOT USED IN SINK MODE (UFP)"
- note added: "OFF-BOARD IMPLEMENTATION OF FREQUENCY BAND SPECIFIC CIRCUITRY."
- note added: "PLUG ORIENTATION (UNUSED)"
- note added: "POSSIBLE TO USE THIS OUTPUT TO TEST THE FILTER CONFIGURATION?"
- note added: "SEE doc/filter-models/cd2003-supply-low-pass-filter"
- note added: "SEE doc/mcu"
- note added: "SEE doc/power-supply"
- note added: "SEE doc/spi-level-conversion"
- note added: "SEE doc/swr-and-power-metering"
- note added: "SPI BUS"
- note added: "TO SWR DETECTION"
- note added: "TRANSIENT PROTECTION"
- note added: "USB SOUND CHIPSET STATUS"
- note added: "USB-PD STATUS"
- note added: "USBC USB-PD/DC INPUT"
- note added: "USED FOR SAFETY PURPOSES TO ENSURE TRANSMIT POWER IS NOT APPLIED WHEN ANTENNA IS MISSING, AND FOR CALCULATION OF SWR AND TUNING."
- note removed: "0.8Ω 210nH 1A SRF=1800MHz"
- note removed: "1.16Ω 400uH >1A SRF=4000MHz"
- note removed: "160-2200M / 135kHz-2MHz"
- note removed: "2-60M / 5-144MHz"
- note removed: "2x (33 x 0.47uH = 15.51uH @ 1.188Ω) = 7.755μH @ 0.594Ω SRF=170MHz I>3A"
- note removed: "500K RESISTANCE TO REQUEST 5V @ 1.5A"
- note removed: "70CM / 450MHz"
- note removed: "=Sokal's 'C1' to be calculated"
- note removed: "ADD PULLUPS/PULLDOWNS REST OF PA ANTENNA MATCHING NETWORK OR ATU ADD/TEST ANTENNA CABLE DETECTION ADD OPTIONAL SQUEAKER ADD TEST POINTS"
- note removed: "ALL ARE SWITCHED BASED ON FREQUENCY AND NOMINALLY ADJACENT. IT LIKELY MAKES SENSE TO CREATE A UNIFORM INTERFACE AND PHYSICAL MODULE."
- note removed: "BONUS BLINKENLIGHTS"
- note removed: "CD2003GP is a clone of Toshiba TA2003. TA2003 is itself a pin-compatible upgrade to the earlier Toshiba TA8164. Only the AM section is used as a direct conversion receiver."
- note removed: "DESIGN GOAL: "GOOD ENOUGH" FORWARD AND REVERSE POWER AND SWR PLUS ANTENNA ABSENCE OR BREAKAGE DETECTION FOR SAFETY PURPOSES."
- note removed: "DISPLAY"
- note removed: "EEPROM POSSIBLY NOT REQ'D"
- note removed: "FOR SWR / SAFETY"
- note removed: "For effective power supply noise filtering, a design guideline is to use ferrite beads at about 20% of their rated DC current."
- note removed: "INPUTS FOR EXTERNAL CRYSTALS"
- note removed: "LPF IN HERE"
- note removed: "MCU AND OUTPUT EXPANSION"
- note removed: "OUTPUT EXPANSION"
- note removed: "PA-DRAIN"
- note removed: "PA-SUPPLY"
- note removed: "POSSIBLE TO USE THIS OUTPUT TO TEST THE FILTER CONFIGURATION? COULD ALSO GENERATE 12MHz OSCILLATION REQUIRED FOR THE USB HUB."
- note removed: "POWER AMPLIFIER SWITCHED RESONATOR"
- note removed: "PROTECTION"
- note removed: "RECOMMENDED 2x1K Si5351A PIN-ADJACENT PULLUPS"
- note removed: "REQUIRES 3.3V LEVEL CONVERSION"
- note removed: "RESISTIVE LOAD"
- note removed: "RF CHOKE"
- note removed: "RFC-GND"
- note removed: "RULE OF THUMB: "OPERATE SWR <4" "SURVIVE SWR <10""
- note removed: "SEE docs/power-supply"
- note removed: "SEE docs/spi-level-conversion"
- note removed: "SWITCHED BASED ON FREQUENCY BAND"
- note removed: "TRANSMIT POWER CONTROL"
- note removed: "USBC/USB-PD DC INPUT"
- note removed: "docs/filter-models/cd2003-supply-low-pass-filter"
- note removed: "xΩ xuH >xmA SRF>xMHz"
- moved on the sheet: A1, C1, C10, C11, C12, C13, C14, C15, C16, C17, C19, C21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
