File: kicad-pcbs/adxi/adxi.kicad_sch (KiCad schematic)
At the start: 151 parts, among them J3 USBC, J5 USB2 Type-A, Q1 MMBF170, Q2 HY1904C2, U1 SI5351A-B-GTR, U10 CM108B, U2 CD2003, U3 L7812, U4 74ACT244, U6 LMV358CDRG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

Commit message: Updates
Parts:
- removed C14, C18: 470uF, Capacitor_SMD:C_Elec_10x10.2, symbol Device:C_Polarized_Small
- removed C23: 100nF, Capacitor_SMD:C_0805_2012Metric, symbol Device:C_Small
- removed C25, C44, C45: 10uF, Capacitor_SMD:C_1206_3216Metric, symbol Device:C_Small
- removed C30: 1nF, Capacitor_SMD:C_0805_2012Metric, symbol Device:C_Small
- removed C31: 100pF, Capacitor_SMD:C_0603_1608Metric, symbol Device:C_Small
- removed C33: 10pF, Capacitor_SMD:C_0603_1608Metric, symbol Device:C_Small
- removed C34: 1pF, Capacitor_SMD:C_0402_1005Metric, symbol Device:C_Small
- removed D1, D3: 1N4148WS, Diode_SMD:D_SOD-323, symbol Diode:1N4148WS
- removed D11, D8: BZT52C5V6, Diode_SMD:D_SOD-123, symbol Device:D_Zener
- removed L4: 100uH, adxi-footprints:IND-SMD_L13.4-W12.6, symbol Device:L
- removed Q2: HY1904C2, adxi-footprints:DFN-8_L5.9-W5.2-P1.27-LS6.2-BL, symbol kicad-parts:HY1904C2
- removed TP3: VIN-USBC, TestPoint:TestPoint_THTPad_2.0x2.0mm_Drill1.0mm, symbol Connector:TestPoint
- added C22: 10uF, Capacitor_SMD:C_1206_3216Metric, symbol Device:C_Small
- added D1, D3: 1N5711, Diode_SMD:D_SOD-123, symbol Diode:1N5711
- added D7: 500mW 43V, Diode_SMD:D_SOD-123, symbol Device:D_Zener
- added U12: SI2304DDS-T1-GE3, adxi-footprints:SOT-23-3_L2.9-W1.6-P1.90-LS2.8-BR, symbol adxi-symbols:SI2304DDS-T1-GE3
- C1, C5: footprint Capacitor_SMD:C_1206_3216Metric -> Capacitor_SMD:C_1210_3225Metric; LCSC Part # C13585 -> C5156756; MPN CL31A106KBHNNNE -> FS32X106K101EGG; Manufacturer Samsung -> Prosperity
- C12, C20, C8: value 470uF -> 1000uF; LCSC Part # C107397 -> C3359; MPN RVE1E471M1010 -> RVT1C102M1010; Manufacturer Roqang -> Honor
- C29: value 22nF -> 100nF; footprint Capacitor_SMD:C_1206_3216Metric -> Capacitor_SMD:C_0805_2012Metric; LCSC Part # C97929 -> C28233; MPN GRM3195C1H223JA01D -> CL21B104KCFNNNE; Manfacturer (none) -> Samsung; Manufacturer Murata -> (none)
- D10: value BZT52C5V6 -> 500mW 43V; LCSC Part # C173406 -> C268628; MPN BZT52C5V6 -> MMSZ5260B; Manufacturer MDD -> Panjit
- L226: footprint adxi-footprints:IND-SMD_L10.8-W10.0 -> Inductor_SMD:L_Changjiang_FNR4030S; Alternatives C475917 (1040-220-M), C128694 (SMMS0630-220M), C497873 (YSP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 -> (none); LCSC Part # C182173 -> C167883; MPN SLO1040H220MTT -> FNR4030S220MT; Manufacturer Sunltech Tech -> Changjiang
- TP11: value RFC-GND -> GND
- TP12: value PA-SUPPLY -> L1-SUPPLY
Connections:
- net Late Stage Interface/RFC-GND is gone; now on net GND: C29.1, TP11.1
- net 12V: now also C20.1, C29.2, C22.2
- net GND: now also C22.1, D7.1 (K), U12.2 (S); no longer C29.2
- net RECEIVED-SIGNAL: now also D7.2 (A), U12.3 (D)
- net VIN: now also D26.1 (K), R80.2
- net at C1.2: now also D1.1 (K)
- net at R1.1: now also D1.2 (A)
- net at C32.1, R15.2: now also U12.1 (G)
- net at R9.1: now also D3.1 (K)
- net at C5.2: now also D3.2 (A)
- net Late Stage Interface/PA-SUPPLY renamed Late Stage Interface/L1-SUPPLY
- removed net VIN-USBC: C20.1, D26.1 (K), R80.2
Other:
- sheet Late Stage Interface ports: added GND, L1-SUPPLY; removed PA-SUPPLY, RFC-GND
- sheet PA Transmit Power Modulation: file nfet-highside-load-switch.kicad_sch -> nfet-highside-load-switch-v2-si2304dds.kicad_sch
- note added: "1.1"
- note added: "DIRECTS ALL TRANSIENT VOLTAGE OVER AROUND 43V TO GROUND."
- note added: "HIGH PASS FILTER"
- note added: "NB. IN A CLASS E RF POWER AMPLIFIER THE PA-DRAIN FLOWS INWARD WHEN ENABLED AND IS SUNK AT THE MOSFET SOURCE PINS. MOSFET IS SELECTED FOR LOW C(OSS) ("OUTPUT GATE CAPACITANCE")"
- note added: "PA+LPF=LSM INTERFACE"
- note added: "SIMPLIFIED POWER STAGE REDUCES COST AND CAPACITOR VOLTAGE RATING REQUIREMENTS"
- note added: "THE CAPACITOR BLOCKS DC, BUT ALLOWS AC TO DRIVE THE GATE. THE RESISTOR PROVIDES (1) A DC RETURN PATH FOR THE GATE. (2) IMPROVED STABILITY WITH ULTRA-LOW IMPEDANCE GROUND PATH FOR UNWANTED RF AC SIGNALS. (3) HELPS WITH GATE DISCHARGE. (4) PULLS GATE TO GND IN THE EVENT OF DRIVER FAILURE."
- note added: "THE USE OF 74AC INSTEAD OF THE 74HC SERIES IS DUE TO THE INCREASED OUTPUT CURRENT CAPACITY WHICH IS NECESSARY TO DRIVE THE HIGH FREQUENCY GATE AND OVERCOME CAPACITANCE."
- note removed: "12V-24V NOMINAL"
- note removed: "2A INDUCTOR TO SMOOTH ANY HIGH FREQUENCY NOISE STILL PRESENT"
- note removed: "NB. IN A CLASS E RF POWER AMPLIFIER THE PA-DRAIN FLOWS INWARD WHEN ENABLED AND IS SUNK AT THE MOSFET SOURCE PINS."
- note removed: "RF CHOKE AC GROUND DECOUPLING"
- note removed: "SMALLER VALUE CAPACITORS ARE TO BE POSITIONED CLOSER TO RF CHOKE"
- note removed: "TRANSIENT PROTECTION"
- moved on the sheet: C16, C21, C26, C27, C28, TP12, TP13, U3

Commit message: Updates
Parts:
- U8: Alternatives (none) -> C2833712 C78162 C22396393 C77805; Note (none) -> China version of original Olimex part. Very widely cloned, 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
Other:
- note added: "BOOST IC VIN = 5V VOUT = 12V I < 4A"
- note added: "CHOOSE 6.8-10uH LOW DCR INDUCTOR"
- note added: "CONSIDER ANY 5V LDO, LATER DISABLED"
- note added: "MISSING 100uF AND 100nF CAPS"
- note added: "MISSING 22uF CERAMIC LOW ESR X5R/X7R INPUT SIDE CAPACITANCE"
- note added: "MISSING 22uF CERAMIC LOW ESR X5R/X7R OUTPUT SIDE CAPACITANCE"
- note added: "MISSING 330nF INPUT BYPASS"
- note added: "MISSING 5.1Ω RIPPLE REJECTION SERIES RESISTOR"
- note added: "THESE SHOULD BE NEXT TO REGULATOR"
- note added: "WRONG TOPOLOGY! VDD MUST BE FED FROM VBUS BEFORE POWER-ON COMPLETE"
- note added: "X"
- note removed: "BOOST IC VIN = 5V VOUT = 12V"
Changed lines of the file:
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@@
 		)
 	)
+	(polyline
+		(pts
+			(xy 115.57 293.37) (xy 120.65 293.37)
+		)
+		(stroke
+			(width 0.2794)
+			(type default)
+			(color 255 0 255 1)
+		)
+	)
 	(wire
 		(pts
@@
 	(polyline
 		(pts
+			(xy 71.12 311.15) (xy 71.12 292.1)
+		)
+		(stroke
+			(width 0.2794)
+			(type default)
+			(color 255 0 255 1)
+		)
+	)
+	(polyline
+		(pts
 			(xy 188.595 88.9) (xy 188.595 138.43)
 		)
@@
 		)
 	)
+	(polyline
+		(pts
+			(xy 86.36 292.1) (xy 71.12 292.1)
+		)
+		(stroke
+			(width 0.2794)
+			(type default)
+			(color 255 0 255 1)
+		)
+	)
+	(polyline
+		(pts
+			(xy 86.36 292.1) (xy 86.36 294.005)
+		)
+		(stroke
+			(width 0.2794)
+			(type default)
+			(color 255 0 255 1)
+		)
+	)
 	(wire
 		(pts
@@
 		)
 	)
+	(polyline
+		(pts
+			(xy 100.33 285.115) (xy 103.505 285.115)
+		)
+		(stroke
+			(width 0.2794)
+			(type default)
+			(color 255 0 255 1)
+		)
+	)
 	(wire
 		(pts
@@
 		)
 	)
+	(text "X"
+		(exclude_from_sim no)
+		(at 106.934 254.508 0)
+		(effects
+			(font
+				(size 3.81 3.81)
+				(thickness 0.254)
+				(bold yes)
+				(color 255 0 0 1)
+			)
+			(justify left top)
+		)
+	)
 	(text "BATTERIES"
 		(exclude_from_sim no)
@@
 		)
 	)
+	(text "WRONG TOPOLOGY!\nVDD MUST BE FED\nFROM VBUS BEFORE\nPOWER-ON COMPLETE"
+		(exclude_from_sim no)
+		(at 84.582 247.396 0)
+		(effects
+			(font
+				(size 1.27 1.27)
+				(thickness 0.254)
+				(bold yes)
+				(color 255 0 255 1)
+			)
+			(justify left top)
+		)
+	)
 	(text "REC. ENABLED \"HEADSET MODE\""
 		(exclude_from_sim no)
@@
 	(text "5V 1.5A NOMINAL"
 		(exclude_from_sim no)
-		(at 70.104 255.016 0)
+		(at 120.904 284.48 90)
 		(effects
 			(font
@@
 		)
 	)
+	(text "MISSING 22uF\nCERAMIC LOW\nESR X5R/X7R\nOUTPUT SIDE\nCAPACITANCE"
+		(exclude_from_sim no)
+		(at 69.85 301.244 0)
+		(effects
+			(font
+				(size 1.27 1.27)
+				(thickness 0.254)
+				(bold yes)
+				(color 255 0 255 1)
+			)
+			(justify right top)
+		)
+	)
 	(text "PA/LPF INTERFACE"
 		(exclude_from_sim no)
@@
 		)
 	)
+	(text "MISSING 330nF\nINPUT BYPASS"
+		(exclude_from_sim no)
+		(at 45.72 338.328 0)
+		(effects
+			(font
+				(size 1.27 1.27)
+				(thickness 0.254)
+				(bold yes)
+				(color 255 0 255 1)
+			)
+			(justify right top)
+		)
+	)
 	(text "SPI LEVEL CONVERSION 5V TO 3.3V"
 		(exclude_from_sim no)
@@
 		)
 	)
+	(text "MISSING 22uF\nCERAMIC LOW\nESR X5R/X7R\nINPUT SIDE\nCAPACITANCE"
+		(exclude_from_sim no)
+		(at 121.158 289.814 0)
+		(effects
+			(font
+				(size 1.27 1.27)
+				(thickness 0.254)
+				(bold yes)
+				(color 255 0 255 1)
+			)
+			(justify left top)
+		)
+	)
 	(text "USB PD\nLINES"
 		(exclude_from_sim no)
@@
 	(text "SEE doc/power-supply"
 		(exclude_from_sim no)
-		(at 111.506 364.49 0)
+		(at 110.49 365.506 0)
 		(effects
 			(font
@@
 		)
 	)
+	(text "CONSIDER ANY\n5V LDO, LATER\nDISABLED"
+		(exclude_from_sim no)
+		(at 110.49 248.158 0)
+		(effects
+			(font
+				(size 1.27 1.27)
+				(thickness 0.254)
+				(bold yes)
+				(color 255 0 255 1)
+			)
+			(justify left top)
+		)
+	)
 	(text "\"100mA\""
 		(exclude_from_sim no)
@@
 		)
 	)
+	(text "THESE SHOULD BE\nNEXT TO REGULATOR"
+		(exclude_from_sim no)
+		(at 110.236 359.918 0)
+		(effects
+			(font
+				(size 1.27 1.27)
+				(thickness 0.254)
+				(bold yes)
+				(color 255 0 255 1)
+			)
+			(justify top)
+		)
+	)
 	(text "THIRD PARTY\nSCREEN MODULE"
 		(exclude_from_sim no)
@@
 	(text "12V 0.5A NOMINAL"
 		(exclude_from_sim no)
-		(at 72.39 293.116 0)
+		(at 49.022 293.116 0)
 		(effects
 			(font
@@
 		)
 	)
-	(text "BOOST IC\nVIN = 5V\nVOUT = 12V"
+	(text "BOOST IC\nVIN = 5V\nVOUT = 12V\nI < 4A"
 		(exclude_from_sim no)
-		(at 109.728 309.626 0)
+		(at 110.49 310.896 0)
 		(effects
 			(font
@@
 		)
 	)
+	(text "MISSING 100uF\nAND 100nF CAPS"
+		(exclude_from_sim no)
+		(at 81.788 251.46 0)
+		(effects
+			(font
+				(size 1.27 1.27)
+				(thickness 0.254)
+				(bold yes)
+				(color 255 0 255 1)
+			)
+			(justify right top)
+		)
+	)
 	(text "THIRD PARTY CHARGE\nCONTROL MODULE"
 		(exclude_from_sim no)
@@
 		)
 	)
+	(text "MISSING 5.1Ω\nRIPPLE REJECTION\nSERIES RESISTOR"
+		(exclude_from_sim no)
+		(at 45.72 329.184 0)
+		(effects
+			(font
+				(size 1.27 1.27)
+				(thickness 0.254)
+				(bold yes)
+				(color 255 0 255 1)
+			)
+			(justify right top)
+		)
+	)
 	(text "ONBOARD USB2.0 4 PORT HUB"
 		(exclude_from_sim no)
@@
 		)
 	)
+	(text "CHOOSE 6.8-10uH\nLOW DCR INDUCTOR"
+		(exclude_from_sim no)
+		(at 99.568 283.972 0)
+		(effects
+			(font
+				(size 1.27 1.27)
+				(thickness 0.254)
+				(bold yes)
+				(color 255 0 255 1)
+			)
+			(justify right top)
+		)
+	)
 	(text "BATTERIES"
 		(exclude_from_sim no)
@@
 			)
 		)
-		(property "Datasheet" "https://www.olimex.com/Products/Breadboarding/BB-PWR-3608/resources/MT3608.pdf"
+		(property "Datasheet" "https://wmsc.lcsc.com/wmsc/upload/file/pdf/v2/lcsc/2311081139_XI-AN-Aerosemi-Tech-MT3608B_C19189893.pdf"
 			(at 113.03 285.75 0)
 			(effects
@@
 			)
 		)
-		(property "Alternatives" ""
+		(property "Alternatives" "C2833712 C78162 C22396393 C77805"
+			(at 106.68 297.18 0)
+			(effects
+				(font
+					(size 1.27 1.27)
+				)
+				(hide yes)
+			)
+		)
+		(property "Note" "China version of original Olimex part. Very widely cloned, identical clones from many manufacturers."
 			(at 106.68 297.18 0)
 			(effects
