File: kicad-pcbs/adxi/adxi.kicad_pcb (KiCad board)
At the start: 2 copper layers, 134.7 x 56.7 mm, 124 parts, among them J1 FROM-PC-SPK, J2 TO-PC-MIC, J3 12V SUPPLY, J4 Conn_Coaxial, J5 Conn_Coaxial_Small, Q1 MMBF170, Q2 MMBF170, Q3 MMBF170, Q4 MMBF170, U1 CD2003, U2 Si5351A-B-GT, U3 74ACT244

Commit message: LPFs, footprints, component selection, switching
Parts:
- removed the D1 at (148.4, 103.6)
- removed the D11 at (187.0, 71.0)
- removed the D15 at (191.1, 76.7)
- removed the D16 at (180.2, 92.5)
- removed the D17 at (194.2, 96.9)
- removed the D3 at (156.2, 103.6)
- removed the D4 at (160.3, 103.6)
- removed the D5 at (169.3, 103.6)
- removed the D9 at (164.0, 80.2)
- removed the L3 at (187.4, 82.2)
- removed the L3 at (187.4, 76.3)
- removed the L4 at (176.1, 72.9)
- removed the L5 at (187.4, 73.5)
- removed the L5 at (187.4, 79.2)
- removed the Q1 at (165.4, 95.8)
- removed the R11 at (148.4, 101.5)
- removed the R12 at (152.3, 101.5)
- removed the R14 at (160.3, 101.5)
- removed the R26 at (181.5, 105.3)
- removed R5: 10K, Resistor_SMD:R_1206_3216Metric
- added C30: 10pF, Capacitor_SMD:C_1206_3216Metric, F.Cu at (404.6, 92.7)
- added C31: 10pF, Capacitor_SMD:C_1206_3216Metric, F.Cu at (404.6, 96.1)
- added C32: 1pF, Capacitor_SMD:C_1206_3216Metric, F.Cu at (404.6, 99.4)
- added C59: 33pF, Capacitor_SMD:C_1206_3216Metric, F.Cu at (642.5, 107.5)
- added C60: 33pF, Capacitor_SMD:C_1206_3216Metric, F.Cu at (642.5, 110.9)
- added C61: 33pF, Capacitor_SMD:C_1206_3216Metric, F.Cu at (637.1, 105.3)
- added C62: 1pF, Capacitor_SMD:C_1206_3216Metric, F.Cu at (637.1, 108.6)
- added C63: 33pF, Capacitor_SMD:C_1206_3216Metric, F.Cu at (637.1, 112.0)
- added C64: 1pF, Capacitor_SMD:C_1206_3216Metric, F.Cu at (385.2, -12.1)
- added C65: 10pF, Capacitor_SMD:C_1206_3216Metric, F.Cu at (385.2, -8.71)
- added C66: 1pF, Capacitor_SMD:C_1206_3216Metric, F.Cu at (385.2, -5.36)
- added C67: 1pF, Capacitor_SMD:C_1206_3216Metric, F.Cu at (385.2, -2.01)
- added C68: 1pF, Capacitor_SMD:C_1206_3216Metric, F.Cu at (385.2, 1.34)
- added C69: 1pF, Capacitor_SMD:C_1206_3216Metric, F.Cu at (365.6, -28.8)
- added C70: 33pF, Capacitor_SMD:C_1206_3216Metric, F.Cu at (365.6, -25.4)
- added C71: 33pF, Capacitor_SMD:C_1206_3216Metric, F.Cu at (365.6, -22.1)
- added C72: 33pF, Capacitor_SMD:C_1206_3216Metric, F.Cu at (365.6, -18.7)
- added C73: 1pF, Capacitor_SMD:C_1206_3216Metric, F.Cu at (365.6, -15.4)
- added C74: 10pF, Capacitor_SMD:C_1206_3216Metric, F.Cu at (365.6, -12.0)
- added C75: 10pF, Capacitor_SMD:C_1206_3216Metric, F.Cu at (365.6, -8.68)
- added C76: 10pF, Capacitor_SMD:C_1206_3216Metric, F.Cu at (365.6, -5.33)
- added C77: 10pF, Capacitor_SMD:C_1206_3216Metric, F.Cu at (365.6, -1.98)
- added C78: 1pF, Capacitor_SMD:C_1206_3216Metric, F.Cu at (522.1, -54.9)
- added C79: 1pF, Capacitor_SMD:C_1206_3216Metric, F.Cu at (534.1, -54.9)
- added C80: 1pF, Capacitor_SMD:C_1206_3216Metric, F.Cu at (389.3, 7.80)
- added C81: 1pF, Capacitor_SMD:C_1206_3216Metric, F.Cu at (534.1, -51.6)
- added C82: 1pF, Capacitor_SMD:C_1206_3216Metric, F.Cu at (389.3, 11.2)
- added C83: 1pF, Capacitor_SMD:C_1206_3216Metric, F.Cu at (389.3, 14.5)
- added C84: 1pF, Capacitor_SMD:C_1206_3216Metric, F.Cu at (534.1, -48.2)
- added C85: 1pF, Capacitor_SMD:C_1206_3216Metric, F.Cu at (534.1, -44.9)
- added D19: 13V 5W, Diode_SMD:D_0603_1608Metric, F.Cu at (409.5, 92.3)
- added D20: 13V 5W, Diode_SMD:D_0603_1608Metric, F.Cu at (409.5, 94.9)
- added D21: 13V 5W, Diode_SMD:D_0603_1608Metric, F.Cu at (364.3, 97.7)
- added D22: 13V 5W, Diode_SMD:D_0603_1608Metric, F.Cu at (364.3, 100.3)
- added D23: 13V 5W, Diode_SMD:D_0603_1608Metric, F.Cu at (479.2, 102.8)
- added D24: 13V 5W, Diode_SMD:D_0603_1608Metric, F.Cu at (479.2, 105.4)
- added D25: 13V 5W, Diode_SMD:D_0603_1608Metric, F.Cu at (550.8, -5.23)
- added D26: 13V 5W, Diode_SMD:D_0603_1608Metric, F.Cu at (550.8, -2.64)
- added D27: 13V 5W, Diode_SMD:D_0603_1608Metric, F.Cu at (696.3, 48.5)
- added D31: 13V 5W, Diode_SMD:D_0603_1608Metric, F.Cu at (556.3, 102.0)
- added D32: 13V 5W, Diode_SMD:D_0603_1608Metric, F.Cu at (576.8, 108.2)
- added D33: 13V 5W, Diode_SMD:D_0603_1608Metric, F.Cu at (576.8, 100.5)
- added D34: 13V 5W, Diode_SMD:D_0603_1608Metric, F.Cu at (576.8, 103.1)
- added D35: 13V 5W, Diode_SMD:D_0603_1608Metric, F.Cu at (636.3, 94.5)
- added D36: 13V 5W, Diode_SMD:D_0603_1608Metric, F.Cu at (636.3, 97.1)
- added D37: 13V 5W, Diode_SMD:D_0603_1608Metric, F.Cu at (636.3, 99.7)
- added D38: 13V 5W, Diode_SMD:D_0603_1608Metric, F.Cu at (636.3, 102.3)
- added D39: BZT52C12, Diode_SMD:D_SOD-123, F.Cu at (397.9, 12.5)
- added D40: 13V 5W, Diode_SMD:D_0603_1608Metric, F.Cu at (390.1, -4.94)
- added D41: 13V 5W, Diode_SMD:D_0603_1608Metric, F.Cu at (390.1, -2.35)
- added D42: 13V 5W, Diode_SMD:D_0603_1608Metric, F.Cu at (390.1, 0.24)
- added D43: 13V 5W, Diode_SMD:D_0603_1608Metric, F.Cu at (390.1, 2.83)
- added D44: BZT52C12, Diode_SMD:D_SOD-123, F.Cu at (409.6, -12.1)
- added D45: BZT52C12, Diode_SMD:D_SOD-123, F.Cu at (604.8, 69.4)
- added D46: 13V 5W, Diode_SMD:D_0603_1608Metric, F.Cu at (370.4, -16.6)
- added D47: 13V 5W, Diode_SMD:D_0603_1608Metric, F.Cu at (370.4, -14.0)
- added D48: 13V 5W, Diode_SMD:D_0603_1608Metric, F.Cu at (370.4, -11.4)
- added D49: 13V 5W, Diode_SMD:D_0603_1608Metric, F.Cu at (370.4, -8.84)
- added D50: BZT52C12, Diode_SMD:D_SOD-123, F.Cu at (522.3, 142.1)
- added D51: BZT52C12, Diode_SMD:D_SOD-123, F.Cu at (519.7, 68.8)
- added D52: 13V 5W, Diode_SMD:D_0603_1608Metric, F.Cu at (384.5, 7.42)
- added D53: 13V 5W, Diode_SMD:D_0603_1608Metric, F.Cu at (384.5, 10.0)
- added D54: 13V 5W, Diode_SMD:D_0603_1608Metric, F.Cu at (384.5, 12.6)
- added D55: 13V 5W, Diode_SMD:D_0603_1608Metric, F.Cu at (384.5, 15.2)
- added D56: BZT52C12, Diode_SMD:D_SOD-123, F.Cu at (523.7, -64.9)
- added D57: BZT52C12, Diode_SMD:D_SOD-123, F.Cu at (539.8, -64.9)
- added D58: 13V 5W, Diode_SMD:D_0603_1608Metric, F.Cu at (491.2, -55.3)
- added D59: 13V 5W, Diode_SMD:D_0603_1608Metric, F.Cu at (491.2, -52.7)
- added D60: 13V 5W, Diode_SMD:D_0603_1608Metric, F.Cu at (491.2, -50.1)
- added D61: 13V 5W, Diode_SMD:D_0603_1608Metric, F.Cu at (491.2, -47.5)
- added D62: BZT52C12, Diode_SMD:D_SOD-123, F.Cu at (507.7, -81.6)
- added D63: BZT52C12, Diode_SMD:D_SOD-123, F.Cu at (539.8, -81.6)
- added D64: 13V 5W, Diode_SMD:D_0603_1608Metric, F.Cu at (517.2, -55.3)
- added D65: 13V 5W, Diode_SMD:D_0603_1608Metric, F.Cu at (517.2, -52.7)
- added D66: 13V 5W, Diode_SMD:D_0603_1608Metric, F.Cu at (517.2, -50.1)
- added D67: 13V 5W, Diode_SMD:D_0603_1608Metric, F.Cu at (517.2, -47.5)
- added D68: BZT52C12, Diode_SMD:D_SOD-123, F.Cu at (507.7, -98.3)
- added D69: BZT52C12, Diode_SMD:D_SOD-123, F.Cu at (491.6, -64.9)
- added D70: 13V 5W, Diode_SMD:D_0603_1608Metric, F.Cu at (539.0, -55.3)
- added D71: 13V 5W, Diode_SMD:D_0603_1608Metric, F.Cu at (539.0, -52.7)
- added D72: 13V 5W, Diode_SMD:D_0603_1608Metric, F.Cu at (539.0, -50.1)
- added D73: 13V 5W, Diode_SMD:D_0603_1608Metric, F.Cu at (539.0, -47.5)
- added D74: BZT52C12, Diode_SMD:D_SOD-123, F.Cu at (507.7, -64.9)
- added D75: BZT52C12, Diode_SMD:D_SOD-123, F.Cu at (523.7, -81.6)
- added D76: 13V 5W, Diode_SMD:D_0603_1608Metric, F.Cu at (485.1, -55.3)
- added D77: 13V 5W, Diode_SMD:D_0603_1608Metric, F.Cu at (485.1, -52.7)
- added D78: 13V 5W, Diode_SMD:D_0603_1608Metric, F.Cu at (485.1, -50.1)
- added D79: 13V 5W, Diode_SMD:D_0603_1608Metric, F.Cu at (485.1, -47.5)
- added D80: BZT52C12, Diode_SMD:D_SOD-123, F.Cu at (539.8, -98.3)
- added D81: BZT52C12, Diode_SMD:D_SOD-123, F.Cu at (491.6, -98.3)
- added D82: 13V 5W, Diode_SMD:D_0603_1608Metric, F.Cu at (501.2, -55.3)
- added D83: 13V 5W, Diode_SMD:D_0603_1608Metric, F.Cu at (501.2, -52.7)
- added D84: 13V 5W, Diode_SMD:D_0603_1608Metric, F.Cu at (501.2, -50.1)
- added D85: 13V 5W, Diode_SMD:D_0603_1608Metric, F.Cu at (501.2, -47.5)
- added D86: BZT52C12, Diode_SMD:D_SOD-123, F.Cu at (523.7, -98.3)
- added D87: BZT52C12, Diode_SMD:D_SOD-123, F.Cu at (491.6, -81.6)
- added D88: 13V 5W, Diode_SMD:D_0603_1608Metric, F.Cu at (507.2, -55.3)
- added D89: 13V 5W, Diode_SMD:D_0603_1608Metric, F.Cu at (507.2, -52.7)
- added D90: 13V 5W, Diode_SMD:D_0603_1608Metric, F.Cu at (507.2, -50.1)
- added D91: 13V 5W, Diode_SMD:D_0603_1608Metric, F.Cu at (507.2, -47.5)
- added L11: 470nH, Inductor_SMD:L_1008_2520Metric, F.Cu at (647.8, 97.7)
- added L12: 2.2uH, adxi-footprints:L_Chilisin_NLC252018-2.92x2.50x2.20, F.Cu at (647.8, 101.5)
- added L13: 4.7uH ±5%, Inductor_SMD:L_1210_3225Metric, F.Cu at (632.3, 94.5)
- added L14: 720nH, Inductor_SMD:L_1008_2520Metric, F.Cu at (632.3, 97.0)
- added L15: 720nH, Inductor_SMD:L_1008_2520Metric, F.Cu at (632.3, 99.5)
- added L16: 15nH ±2%, Inductor_SMD:L_0603_1608Metric, F.Cu at (632.3, 102.0)
- added L17: 15nH ±2%, Inductor_SMD:L_0603_1608Metric, F.Cu at (632.3, 104.5)
- added L18: 15nH ±2%, Inductor_SMD:L_0603_1608Metric, F.Cu at (632.3, 107.0)
- added L19: 15nH ±2%, Inductor_SMD:L_0603_1608Metric, F.Cu at (632.3, 109.6)
- added L20: 15nH ±2%, Inductor_SMD:L_0603_1608Metric, F.Cu at (632.3, 112.1)
- added L21: 15nH ±2%, Inductor_SMD:L_0603_1608Metric, F.Cu at (632.3, 114.6)
- added L22: 15nH ±2%, Inductor_SMD:L_0603_1608Metric, F.Cu at (390.5, -11.9)
- added L23: 15nH ±2%, Inductor_SMD:L_0603_1608Metric, F.Cu at (390.5, -8.11)
- added L24: 15nH ±2%, Inductor_SMD:L_0603_1608Metric, F.Cu at (370.4, -29.2)
- added L25: 15nH ±2%, Inductor_SMD:L_0603_1608Metric, F.Cu at (370.4, -26.7)
- added L26: 15nH ±2%, Inductor_SMD:L_0603_1608Metric, F.Cu at (370.4, -24.2)
- added L27: 15nH ±2%, Inductor_SMD:L_0603_1608Metric, F.Cu at (370.4, -21.7)
- added L28: 15nH ±2%, Inductor_SMD:L_0603_1608Metric, F.Cu at (370.4, -19.2)
- added L29: 15nH ±2%, Inductor_SMD:L_0603_1608Metric, F.Cu at (374.4, -29.2)
- added L30: 220nH, Inductor_SMD:L_0805_2012Metric, F.Cu at (374.4, -26.7)
- added L31: 220nH, Inductor_SMD:L_0805_2012Metric, F.Cu at (374.4, -24.2)
- added L32: 390nH, Inductor_SMD:L_1008_2520Metric, F.Cu at (374.4, -21.7)
- added L33: 470nH, Inductor_SMD:L_1008_2520Metric, F.Cu at (374.4, -19.2)
- added L34: 470nH, Inductor_SMD:L_1008_2520Metric, F.Cu at (378.4, -29.2)
- added L5: 120, Inductor_SMD:L_1008_2520Metric, F.Cu at (409.9, 98.1)
- added L8: 100nH, Inductor_SMD:L_1008_2520Metric, F.Cu at (646.8, 107.0)
- added Q10: HY1904C2, kicad-parts:HY1904C2, F.Cu at (399.8, 138.1)
- added Q11: 2N7002, Package_TO_SOT_SMD:SOT-23, F.Cu at (407.7, 70.6)
- added Q12: HY1904C2, kicad-parts:HY1904C2, F.Cu at (403.7, 59.6)
- added Q13: 2N7002, Package_TO_SOT_SMD:SOT-23, F.Cu at (487.1, 134.5)
- added Q14: HY1904C2, kicad-parts:HY1904C2, F.Cu at (484.0, 140.5)
- added Q15: 2N7002, Package_TO_SOT_SMD:SOT-23, F.Cu at (473.5, 71.2)
- added Q16: HY1904C2, kicad-parts:HY1904C2, F.Cu at (480.6, 71.5)
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- renumbered C26 to C1, C10 to C13, C22 to C14, C29 to C16, C30 to C18, C21 to C19, C1 to C2, C31 to C21, C11 to C22, C32 to C23, C5 to C3, C25 to C5, D21 to D1, D23 to D2, D22 to D3, D24 to D4, D6 to D5, D7 to D6, D18 to D7, J3 to J5, L12 to L1, L11 to L2, L2 to L3, L8 to L4, Q4 to Q1, R21 to R1, R3 to R10, R8 to R11, R16 to R12, R10 to R14, R9 to R15, R23 to R2, R17 to R3, R2 to R6, R22 to R7, R24 to R8, R18 to R9, U2 to U4
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Connections:
- net CARRIER renamed TX-CLK
- net FSK renamed HOST-FSK-INPUT
- A1 pad 12: LED-WSPR -> unconnected-(A1-D9-Pad12)
- A1 pad 13: LED-JS8 -> unconnected-(A1-D10-Pad13)
- A1 pad 14: LED-FT4 -> unconnected-(A1-D11-Pad14)
- A1 pad 15: LED-FT8 -> unconnected-(A1-D12-Pad15)
- A1 pad 16: LED-TX -> unconnected-(A1-D13-Pad16)
- A1 pad 5: SWITCH-1-UP -> unconnected-(A1-D2-Pad5)
- A1 pad 6: SWITCH-2-DOWN -> PA-POWER-PWM
- A1 pad 7: SWITCH-3-TRANSMIT -> unconnected-(A1-D4-Pad7)
- A1 pad 8: GND -> unconnected-(A1-D5-Pad8)
- A1 pad 9: GND -> unconnected-(A1-D6-Pad9)
- C16 pad 1: 12V -> Net-(D7-A2)
- C18 pad 1: 12V -> Net-(D7-A2)
- C21 pad 1: 12V -> GND
- C21 pad 2: GND -> Net-(D7-A2)
- C23 pad 1: 12V -> GND
- C23 pad 2: GND -> Net-(D7-A2)
- C33 pad 1: 80M-LPF-OUT -> 10M-LPF-OUT
- C34 pad 1: 80M-LPF-OUT -> 10M-LPF-OUT
- C35 pad 1: 80M-LPF-OUT -> 10M-LPF-OUT
- C36 pad 1: 80M-LPF-OUT -> 10M-LPF-OUT
- C37 pad 1: 40M-LPF-OUT -> 10M-LPF-OUT
- C38 pad 1: 40M-LPF-OUT -> 10M-LPF-OUT
- C39 pad 1: 40M-LPF-OUT -> 2M-LPF-OUT
- C40 pad 1: 40M-LPF-OUT -> 2M-LPF-OUT
- C41 pad 1: 40M-LPF-OUT -> 2M-LPF-OUT
- C42 pad 1: 40M-LPF-OUT -> 2M-LPF-OUT
- C43 pad 1: 40M-LPF-OUT -> 20M-LPF-OUT
- C45 pad 1: 10M-LPF-OUT -> 20M-LPF-OUT
- C46 pad 1: 10M-LPF-OUT -> 20M-LPF-OUT
- C49 pad 1: 10M-LPF-OUT -> Net-(C49-Pad1)
- C50 pad 1: 10M-LPF-OUT -> 40M-LPF-OUT
- C50 pad 2: GND -> Net-(C49-Pad1)
- C51 pad 1: 10M-LPF-OUT -> Net-(C49-Pad1)
- C52 pad 1: 10M-LPF-OUT -> Net-(C49-Pad1)
- C53 pad 1: 10M-LPF-OUT -> Net-(C49-Pad1)
- C54 pad 1: 10M-LPF-OUT -> 80M-LPF-OUT
- C54 pad 2: GND -> Net-(C54-Pad2)
- C55 pad 1: 10M-LPF-OUT -> GND
- C55 pad 2: GND -> Net-(C54-Pad2)
- C56 pad 1: 2M-LPF-OUT -> 15M-LPF-OUT
- C57 pad 1: 2M-LPF-OUT -> 15M-LPF-OUT
- C58 pad 1: 2M-LPF-OUT -> unconnected-(C58-Pad1)
- C58 pad 2: GND -> unconnected-(C58-Pad2)
- D10 pad 1: GND -> Net-(D10-K)
- D10 pad 2: 10M-LPF-IN -> 2M-LPF-OUT
- D11 pad 1: GND -> Net-(D11-K)
- D11 pad 2: Net-(D2-A) (its old number) -> 10M-LPF-IN
- D12 pad 1: GND -> Net-(D12-K)
- D12 pad 2: 40M-LPF-IN -> 10M-LPF-OUT
- D13 pad 1: GND -> Net-(D13-K)
- D13 pad 2: 80M-LPF-IN -> 20M-LPF-IN
- D14 pad 1: GND -> Net-(D14-K)
- D14 pad 2: 10M-LPF-OUT -> 20M-LPF-OUT
- D15 pad 1: GND -> Net-(D15-K)
- D15 pad 2: Net-(D19-A) -> 40M-LPF-IN
- D16 pad 1: GND -> Net-(D16-K)
- D16 pad 2: Net-(D20-A) -> 40M-LPF-OUT
- D17 pad 1: GND -> Net-(D17-K)
- D17 pad 2: Net-(D25-A) -> 80M-LPF-IN
- D18 pad 1: GND -> Net-(D18-K)
- D18 pad 2: Net-(D26-A) -> 80M-LPF-OUT
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Routing:
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Other:
- board text added: "15M"
- board text added: "30M"
- board text added: "60M"
- board text added: "FILTER"
- board text added: "IN"
- board text added: "OUT"
- board text added: "adxi"
- board text added: "github.com/vk2diy/adxi"
- board text removed: "FT4"
- board text removed: "FT8"
- board text removed: "JS8"
- board text removed: "MODE"
- board text removed: "TX"
- board text removed: "WSPR"

Commit message: Updates
Parts:
- removed C30, C31, C43, C44, C49, C51, C52, C53, C65, C74, C75, C76, C77: 10pF, Capacitor_SMD:C_1206_3216Metric
- removed C32, C33, C34, C35, C36, C37, C38, C42, C45, C46, C47, C48, C62, C64, C66, C67, C68, C69, C73, C78, C79, C80, C81, C82, C83, C84, C85: 1pF, Capacitor_SMD:C_1206_3216Metric
- removed C39, C40, C41, C56, C57, C58, C59, C60, C61, C63, C70, C71, C72: 33pF, Capacitor_SMD:C_1206_3216Metric
- removed C50: 8.2pF, Capacitor_SMD:C_1206_3216Metric
- removed C54: 820pF C0G 5% 1206, Capacitor_SMD:C_1206_3216Metric
- removed C55: 2.7nF C0G 5% 1206, Capacitor_SMD:C_1206_3216Metric
- removed D20, D21, D22, D23, D24, D25, D26, D27, D28, D29, D30, D31, D32, D33, D34, D35, D36, D37, D38, D40, D41, D42, D43, D46, D47, D48, D49, D52, D53, D54, D55, D58, D59, D60, D61, D64, D65, D66, D67, D70, D71, D72, D73, D76, D77, D78, D79, D82, D83, D84, D85, D88, D89, D90, D91: 13V 5W, Diode_SMD:D_0603_1608Metric
- removed D39, D44, D45, D50, D51, D56, D57, D62, D63, D68, D69, D74, D75, D80, D81, D86, D87: BZT52C12, Diode_SMD:D_SOD-123
- removed L10, L8, L9: 100nH, Inductor_SMD:L_1008_2520Metric
- removed L11, L33, L34: 470nH, Inductor_SMD:L_1008_2520Metric
- removed L12: 2.2uH, adxi-footprints:L_Chilisin_NLC252018-2.92x2.50x2.20
- removed L13: 4.7uH ±5%, Inductor_SMD:L_1210_3225Metric
- removed L14, L15: 720nH, Inductor_SMD:L_1008_2520Metric
- removed L16, L17, L18, L19, L20, L21, L22, L23, L24, L25, L26, L27, L28, L29: 15nH ±2%, Inductor_SMD:L_0603_1608Metric
- removed L30, L31: 220nH, Inductor_SMD:L_0805_2012Metric
- removed L32: 390nH, Inductor_SMD:L_1008_2520Metric
- removed L5, L6, L7: 120, Inductor_SMD:L_1008_2520Metric
- removed Q27, Q29, Q31, Q33, Q35, Q37, Q39, Q41, Q43, Q45, Q47, Q49, Q51, Q53, Q55, Q57: 2N7002, Package_TO_SOT_SMD:SOT-23
- removed Q28, Q30, Q32, Q34, Q36, Q38, Q40, Q42, Q44, Q46, Q48, Q50, Q52, Q54, Q56, Q58: HY1904C2, kicad-parts:HY1904C2
- removed R100, R103, R104, R107, R108, R111, R112, R115, R116, R119, R120, R123, R124, R127, R64, R67, R68, R71, R72, R75, R76, R79, R80, R83, R84, R87, R88, R91, R92, R95, R96, R99: 1K 0.25W, Resistor_SMD:R_1206_3216Metric
- removed R101, R102, R105, R106, R109, R110, R113, R114, R117, R118, R121, R122, R125, R126, R65, R66, R69, R70, R73, R74, R77, R78, R81, R82, R85, R86, R89, R90, R93, R94, R97, R98: 6.8K 0.25W, Resistor_SMD:R_1206_3216Metric
- added D98: BZT52C12, Diode_SMD:D_SOD-123, F.Cu at (112.6, 37.4)
- added J10: BANDMODULE3-ANT, Connector_PinSocket_2.54mm:PinSocket_1x07_P2.54mm_Vertical, F.Cu at (52.7, 76.5)
- added J11: BANDMODULE4-ANT, Connector_PinSocket_2.54mm:PinSocket_1x07_P2.54mm_Vertical, B.Cu at (45.3, 43.7)
- added J12: BANDMODULE3-PA, Connector_PinSocket_2.54mm:PinSocket_1x07_P2.54mm_Vertical, F.Cu at (123.1, 76.6)
- added J13: BANDMODULE4-PA, Connector_PinSocket_2.54mm:PinSocket_1x07_P2.54mm_Vertical, B.Cu at (116.2, 43.5)
- added J14: BANDMODULE5-ANT, Connector_PinSocket_2.54mm:PinSocket_1x07_P2.54mm_Vertical, B.Cu at (44.9, 66.6)
- added J15: BANDMODULE6-ANT, Connector_PinSocket_2.54mm:PinSocket_1x07_P2.54mm_Vertical, B.Cu at (45.2, 89.6)
- added J16: BANDMODULE5-PA, Connector_PinSocket_2.54mm:PinSocket_1x07_P2.54mm_Vertical, B.Cu at (115.5, 67.1)
- added J17: BANDMODULE6-PA, Connector_PinSocket_2.54mm:PinSocket_1x07_P2.54mm_Vertical, B.Cu at (115.8, 89.2)
- added J18: MMCX, Connector_Coaxial:MMCX_Molex_73415-1471_Vertical, F.Cu at (30.4, 42.4)
- added J20: LCD-2004, Connector_PinHeader_2.54mm:PinHeader_1x04_P2.54mm_Vertical, F.Cu at (32.5, 108.5)
- added J6: BANDMODULE1-ANT, Connector_PinSocket_2.54mm:PinSocket_1x07_P2.54mm_Vertical, F.Cu at (52.9, 30.6)
- added J7: BANDMODULE1-PA, Connector_PinSocket_2.54mm:PinSocket_1x07_P2.54mm_Vertical, F.Cu at (123.1, 30.6)
- added J8: BANDMODULE2-ANT, Connector_PinSocket_2.54mm:PinSocket_1x07_P2.54mm_Vertical, F.Cu at (52.7, 53.5)
- added J9: BANDMODULE2-PA, Connector_PinSocket_2.54mm:PinSocket_1x07_P2.54mm_Vertical, F.Cu at (123.3, 53.8)
- added Q63: 2N7002, Package_TO_SOT_SMD:SOT-23, F.Cu at (112.2, 41.5)
- added Q64: HY1904C2, kicad-parts:HY1904C2, F.Cu at (114.0, 32.4)
- added R136: 1K 0.25W, Resistor_SMD:R_1206_3216Metric, F.Cu at (106.9, 30.6)
- added R137: 6.8K 0.25W, Resistor_SMD:R_1206_3216Metric, F.Cu at (106.9, 33.9)
- added R138: 6.8K 0.25W, Resistor_SMD:R_1206_3216Metric, F.Cu at (106.9, 37.2)
- added R139: 1K 0.25W, Resistor_SMD:R_1206_3216Metric, F.Cu at (106.9, 40.5)
- D11, D12, D13, D16, D17, D18, Q10, Q11, Q12, Q13, Q14, Q19, Q20, Q21, Q22, Q23, Q24, Q9, R28, R29, R30, R31, R32, R33, R34, R35, R36, R37, R38, R39, R48, R49, R50, R51, R52, R53, R54, R55, R56, R57, R58, R59: moved to B.Cu
- D19: value 13V 5W -> BZT52C12; footprint Diode_SMD:D_0603_1608Metric -> Diode_SMD:D_SOD-123
- J1, J2: footprint Connector_Audio:Jack_3.5mm_CUI_SJ2-3593D-SMT_Horizontal -> Connector_Audio:Jack_3.5mm_CUI_SJ1-3525N_Horizontal
- moved D9 555.8 mm to (54.2, 95.1), turned to 180 degrees
- moved Q6 549.0 mm to (58.5, 90.6)
- moved Q22 548.4 mm to (103.6, 70.6), turned to 180 degrees
- moved D17 546.0 mm to (104.9, 75.6), turned to 180 degrees
- moved Q5 542.2 mm to (64.4, 94.6), turned to 180 degrees
- moved R23 542.2 mm to (59.2, 95.1)
- moved Q21 540.5 mm to (105.4, 79.7), turned to 180 degrees
- moved R56 536.7 mm to (102.9, 103.8)
- moved R22 536.7 mm to (64.8, 91.6)
- moved R21 536.5 mm to (64.8, 89.2)
- moved R20 536.1 mm to (64.1, 97.7), turned to 180 degrees
- moved D18 535.4 mm to (108.6, 97.1)
- moved R57 535.0 mm to (102.9, 100.5)
- moved R58 534.5 mm to (102.9, 97.3)
- moved R59 534.1 mm to (102.9, 94.0)
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Connections:
- net 10M-LPF-OUT renamed BM5-ANT
- net 20M-LPF-IN renamed BM6-ANT
- net 20M-LPF-OUT renamed BM2-PA
- net 2M-LPF-IN renamed BM2-ANT
- net 2M-LPF-OUT renamed BM1-ANT
- net 40M-LPF-IN renamed BM3-PA
- net 40M-LPF-OUT renamed BM4-PA
- net 60M-LPF-IN renamed BM3-ANT
- net 80M-LPF-IN renamed BM5-PA
- net 80M-LPF-OUT renamed BM6-PA
- D11 pad 2: 10M-LPF-IN -> BM4-ANT
- D19 pad 1: GND -> Net-(D19-K)
- D19 pad 2: 10M-LPF-IN -> PA-12V
- Q10 pad 1: 10M-LPF-IN -> BM4-ANT
- Q10 pad 2: 10M-LPF-IN -> BM4-ANT
- Q10 pad 3: 10M-LPF-IN -> BM4-ANT
- Q10 pad 5: PA-DRAIN -> ANTENNA
- Q10 pad 6: PA-DRAIN -> ANTENNA
- Q10 pad 7: PA-DRAIN -> ANTENNA
- Q10 pad 8: PA-DRAIN -> ANTENNA
- Q14 pad 5: PA-DRAIN -> ANTENNA
- Q14 pad 6: PA-DRAIN -> ANTENNA
- Q14 pad 7: PA-DRAIN -> ANTENNA
- Q14 pad 8: PA-DRAIN -> ANTENNA
- Q16 pad 5: ANTENNA -> PA-DRAIN
- Q16 pad 6: ANTENNA -> PA-DRAIN
- Q16 pad 7: ANTENNA -> PA-DRAIN
- Q16 pad 8: ANTENNA -> PA-DRAIN
- Q20 pad 5: ANTENNA -> PA-DRAIN
- Q20 pad 6: ANTENNA -> PA-DRAIN
- Q20 pad 7: ANTENNA -> PA-DRAIN
- Q20 pad 8: ANTENNA -> PA-DRAIN
- Q24 pad 5: ANTENNA -> PA-DRAIN
- Q24 pad 6: ANTENNA -> PA-DRAIN
- Q24 pad 7: ANTENNA -> PA-DRAIN
- Q24 pad 8: ANTENNA -> PA-DRAIN
- Q26 pad 1: 15M-LPF-IN -> PA-12V
- Q26 pad 2: 15M-LPF-IN -> PA-12V
- Q26 pad 3: 15M-LPF-IN -> PA-12V
- Q26 pad 4: Net-(D39-K) -> Net-(D19-K)
- Q26 pad 5: PA-DRAIN -> 12V
- Q26 pad 6: PA-DRAIN -> 12V
- Q26 pad 7: PA-DRAIN -> 12V
- Q26 pad 8: PA-DRAIN -> 12V
- Q4 pad 5: PA-DRAIN -> ANTENNA
- Q4 pad 6: PA-DRAIN -> ANTENNA
- Q4 pad 7: PA-DRAIN -> ANTENNA
- Q4 pad 8: PA-DRAIN -> ANTENNA
- Q6 pad 5: PA-DRAIN -> ANTENNA
- Q6 pad 6: PA-DRAIN -> ANTENNA
- Q6 pad 7: PA-DRAIN -> ANTENNA
- Q6 pad 8: PA-DRAIN -> ANTENNA
- R16 pad 2: 2M-LPF-ENABLE -> BM2-ENABLE
- R20 pad 2: 60M-LPF-ENABLE -> BM3-ENABLE
- R24 pad 2: 2M-LPF-ENABLE -> BM1-ENABLE
- R28 pad 2: 10M-LPF-ENABLE -> BM4-ENABLE
- R32 pad 2: 10M-LPF-ENABLE -> BM5-ENABLE
- R36 pad 2: 20M-LPF-ENABLE -> BM6-ENABLE
- R40 pad 2: 20M-LPF-ENABLE -> BM2-ENABLE
- R44 pad 2: 40M-LPF-ENABLE -> BM3-ENABLE
- R48 pad 2: 40M-LPF-ENABLE -> BM4-ENABLE
- R52 pad 2: 80M-LPF-ENABLE -> BM5-ENABLE
- R56 pad 2: 80M-LPF-ENABLE -> BM6-ENABLE
- R60 pad 2: 15M-LPF-ENABLE -> PA-DRIVE-PWM
- R61 pad 2: 12V -> 24V
- R62 pad 2: 12V -> 24V
- R63 pad 1: Net-(D39-K) -> Net-(D19-K)
Routing:
- net ANTENNA: track 0.00 -> 127.2 mm
- net BM3-ANT: track 0.00 -> 29.3 mm
- net HOST-FSK-INPUT: track 0.00 -> 23.0 mm
- net BM1-ANT: track 0.00 -> 21.2 mm
- net BM2-ANT: track 0.00 -> 20.3 mm
- net Net-(FB1-Pad1): track 15.2 -> 0.00 mm
- net Net-(D19-K): track 0.00 -> 12.6 mm, vias 0 -> 2
- net Net-(D7-A2): track 9.61 -> 0.00 mm
- net Net-(Q25-D): track 0.00 -> 8.05 mm
- net 24V: track 0.00 -> 6.41 mm
- net 12V: track 0.00 -> 6.25 mm
- net Net-(Q5-D): track 0.00 -> 5.49 mm
- net PA-12V: track 0.00 -> 4.97 mm
- net Net-(C2-Pad2): track 0.00 -> 4.43 mm
- net Net-(C2-Pad1): track 0.00 -> 3.57 mm
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- added copper zone on In1.Cu, net GND
Other:
- board size 134.7 x 56.7 mm -> 106.9 x 124.1 mm
- copper layers 2 -> 4
- board text added: "1"
- board text added: "2"
- board text added: "3"
- board text added: "4"
- board text added: "5"
- board text added: "6"
- board text added: "ANT"
- board text added: "BAND MODULE"
- board text added: "LCD"
- board text added: "MMCX"
- board text removed: "10M"
- board text removed: "15M"
- board text removed: "20M"
- board text removed: "2M"
- board text removed: "30M"
- board text removed: "40M"
- board text removed: "60M"
- board text removed: "80M"
- board text removed: "ANTENNA"
- board text removed: "FILTER"
- board text removed: "IN FROM PC"
- board text removed: "OUT TO PC"

Commit message: Updates
Parts:
- added L10: 3.3uH, Inductor_SMD:L_1008_2520Metric, F.Cu at (151.2, 29.8)
- added L11: 3.3uH, Inductor_SMD:L_1008_2520Metric, F.Cu at (151.2, 33.5)
- added L12: 3.3uH, Inductor_SMD:L_1008_2520Metric, F.Cu at (151.2, 37.2)
- added L13: 3.3uH, Inductor_SMD:L_1008_2520Metric, F.Cu at (151.2, 41.0)
- added L14: 3.3uH, Inductor_SMD:L_1008_2520Metric, F.Cu at (151.2, 44.8)
- added L15: 3.3uH, Inductor_SMD:L_1008_2520Metric, F.Cu at (151.2, 48.5)
- added L16: 3.3uH, Inductor_SMD:L_1008_2520Metric, F.Cu at (151.2, 52.2)
- added L17: 3.3uH, Inductor_SMD:L_1008_2520Metric, F.Cu at (151.2, 56.0)
- added L18: 3.3uH, Inductor_SMD:L_1008_2520Metric, F.Cu at (156.1, 29.8)
- added L19: 3.3uH, Inductor_SMD:L_1008_2520Metric, F.Cu at (156.1, 33.5)
- added L20: 3.3uH, Inductor_SMD:L_1008_2520Metric, F.Cu at (156.1, 37.2)
- added L21: 3.3uH, Inductor_SMD:L_1008_2520Metric, F.Cu at (156.1, 41.0)
- added L22: 3.3uH, Inductor_SMD:L_1008_2520Metric, F.Cu at (156.1, 44.8)
- added L23: 3.3uH, Inductor_SMD:L_1008_2520Metric, F.Cu at (156.1, 48.5)
- added L24: 3.3uH, Inductor_SMD:L_1008_2520Metric, F.Cu at (156.1, 52.2)
- added L25: 3.3uH, Inductor_SMD:L_1008_2520Metric, F.Cu at (156.1, 56.0)
- added L26: 3.3uH, Inductor_SMD:L_1008_2520Metric, F.Cu at (161.1, 29.8)
- added L27: 3.3uH, Inductor_SMD:L_1008_2520Metric, F.Cu at (161.1, 33.5)
- added L28: 3.3uH, Inductor_SMD:L_1008_2520Metric, F.Cu at (161.1, 37.2)
- added L29: 3.3uH, Inductor_SMD:L_1008_2520Metric, F.Cu at (161.1, 41.0)
- added L30: 3.3uH, Inductor_SMD:L_1008_2520Metric, F.Cu at (161.1, 44.8)
- added L31: 3.3uH, Inductor_SMD:L_1008_2520Metric, F.Cu at (161.1, 48.5)
- added L32: 3.3uH, Inductor_SMD:L_1008_2520Metric, F.Cu at (161.1, 52.2)
- added L33: 3.3uH, Inductor_SMD:L_1008_2520Metric, F.Cu at (161.1, 56.0)
- added L34: 3.3uH, Inductor_SMD:L_1008_2520Metric, F.Cu at (166.0, 29.8)
- added L35: 3.3uH, Inductor_SMD:L_1008_2520Metric, F.Cu at (166.0, 33.5)
- added L36: 3.3uH, Inductor_SMD:L_1008_2520Metric, F.Cu at (166.0, 37.2)
- added L44: 10uH, Inductor_SMD:L_1008_2520Metric, F.Cu at (166.0, 41.0)
- added L45: 10uH, Inductor_SMD:L_1008_2520Metric, F.Cu at (166.0, 44.8)
- added L46: 10uH, Inductor_SMD:L_1008_2520Metric, F.Cu at (166.0, 48.5)
- added L47: 10uH, Inductor_SMD:L_1008_2520Metric, F.Cu at (166.0, 52.2)
- added L48: 10uH, Inductor_SMD:L_1008_2520Metric, F.Cu at (166.0, 56.0)
- added L49: 10uH, Inductor_SMD:L_1008_2520Metric, F.Cu at (171.0, 29.8)
- added L50: 10uH, Inductor_SMD:L_1008_2520Metric, F.Cu at (171.0, 33.5)
- added L51: 10uH, Inductor_SMD:L_1008_2520Metric, F.Cu at (171.0, 37.2)
- added L52: 10uH, Inductor_SMD:L_1008_2520Metric, F.Cu at (171.0, 41.0)
- added L53: 10uH, Inductor_SMD:L_1008_2520Metric, F.Cu at (171.0, 44.8)
- added L54: 10uH, Inductor_SMD:L_1008_2520Metric, F.Cu at (171.0, 48.5)
- added L55: 10uH, Inductor_SMD:L_1008_2520Metric, F.Cu at (171.0, 52.2)
- added L56: 10uH, Inductor_SMD:L_1008_2520Metric, F.Cu at (171.0, 56.0)
- added L57: 10uH, Inductor_SMD:L_1008_2520Metric, F.Cu at (175.9, 29.8)
- added L58: 10uH, Inductor_SMD:L_1008_2520Metric, F.Cu at (175.9, 33.5)
- added L59: 10uH, Inductor_SMD:L_1008_2520Metric, F.Cu at (175.9, 37.2)
- added L6: 100uH, Inductor_SMD:L_0805_2012Metric, F.Cu at (180.7, 29.2)
- added L60: 10uH, Inductor_SMD:L_1008_2520Metric, F.Cu at (175.9, 41.0)
- added L61: 10uH, Inductor_SMD:L_1008_2520Metric, F.Cu at (175.9, 44.8)
- added L62: 10uH, Inductor_SMD:L_1008_2520Metric, F.Cu at (175.9, 48.5)
- added L63: 10uH, Inductor_SMD:L_1008_2520Metric, F.Cu at (175.9, 52.2)
- added L7: 100uH, Inductor_SMD:L_0805_2012Metric, F.Cu at (180.7, 32.0)
- added L8: 100uH, Inductor_SMD:L_0805_2012Metric, F.Cu at (180.7, 34.8)
- added L9: 100uH, Inductor_SMD:L_0805_2012Metric, F.Cu at (180.7, 37.5)
Other:
- board text added: "BISCUIT BOX"
- board text added: "CHINA BOX"
- board text added: "SCREEN"

Commit message: More outputs, etc
Parts:
- added C30: 6.8pF, Capacitor_SMD:C_1206_3216Metric, F.Cu at (202.6, 157.3)
- added C31: 12pF, Capacitor_SMD:C_1206_3216Metric, F.Cu at (206.0, 157.3)
- added C32: 15pF, Capacitor_SMD:C_1206_3216Metric, F.Cu at (209.3, 157.3)
- added C33: 20pF, Capacitor_SMD:C_1206_3216Metric, F.Cu at (212.7, 157.3)
- added C34: 5.6nF, Capacitor_SMD:C_1206_3216Metric, F.Cu at (216.0, 157.3)
- added C35: 68nF, Capacitor_SMD:C_1206_3216Metric, F.Cu at (219.4, 157.3)
- added C36: 82pF, Capacitor_SMD:C_1206_3216Metric, F.Cu at (222.7, 157.3)
- added C37: 150pF, Capacitor_SMD:C_1206_3216Metric, F.Cu at (226.1, 157.3)
- added D20: BZT52C12, Diode_SMD:D_SOD-123, F.Cu at (247.8, 103.5)
- added D21: BZT52C12, Diode_SMD:D_SOD-123, F.Cu at (247.8, 70.1)
- added D22: BZT52C12, Diode_SMD:D_SOD-123, F.Cu at (208.6, 120.8)
- added D23: BZT52C12, Diode_SMD:D_SOD-123, F.Cu at (263.8, 86.8)
- added D24: BZT52C12, Diode_SMD:D_SOD-123, F.Cu at (208.6, 137.5)
- added D25: BZT52C12, Diode_SMD:D_SOD-123, F.Cu at (263.8, 70.1)
- added D26: BZT52C12, Diode_SMD:D_SOD-123, F.Cu at (240.7, 120.8)
- added D27: BZT52C12, Diode_SMD:D_SOD-123, F.Cu at (192.5, 137.5)
- added D28: BZT52C12, Diode_SMD:D_SOD-123, F.Cu at (192.5, 120.8)
- added D29: BZT52C12, Diode_SMD:D_SOD-123, F.Cu at (240.7, 137.5)
- added D30: BZT52C12, Diode_SMD:D_SOD-123, F.Cu at (224.7, 137.5)
- added D31: BZT52C12, Diode_SMD:D_SOD-123, F.Cu at (247.8, 86.8)
- added D32: BZT52C12, Diode_SMD:D_SOD-123, F.Cu at (263.8, 103.5)
- added D33: BZT52C12, Diode_SMD:D_SOD-123, F.Cu at (224.7, 120.8)
- added L100: 100nH, Inductor_SMD:L_1008_2520Metric, F.Cu at (211.2, 86.0)
- added L101: 100nH, Inductor_SMD:L_1008_2520Metric, F.Cu at (211.2, 89.8)
- added L102: 100nH, Inductor_SMD:L_1008_2520Metric, F.Cu at (211.2, 93.5)
- added L103: 100nH, Inductor_SMD:L_1008_2520Metric, F.Cu at (211.2, 97.3)
- added L104: 100nH, Inductor_SMD:L_1008_2520Metric, F.Cu at (211.2, 101.0)
- added L105: 100nH, Inductor_SMD:L_1008_2520Metric, F.Cu at (211.2, 104.8)
- added L106: 100nH, Inductor_SMD:L_1008_2520Metric, F.Cu at (211.2, 108.5)
- added L107: 100nH, Inductor_SMD:L_1008_2520Metric, F.Cu at (216.2, 63.5)
- added L108: 100nH, Inductor_SMD:L_1008_2520Metric, F.Cu at (216.2, 67.3)
- added L109: 100nH, Inductor_SMD:L_1008_2520Metric, F.Cu at (216.2, 71.0)
- added L110: 100nH, Inductor_SMD:L_1008_2520Metric, F.Cu at (216.2, 74.8)
- added L111: 100nH, Inductor_SMD:L_1008_2520Metric, F.Cu at (216.2, 78.5)
- added L112: 100nH, Inductor_SMD:L_1008_2520Metric, F.Cu at (216.2, 82.3)
- added L113: 100nH, Inductor_SMD:L_1008_2520Metric, F.Cu at (216.2, 86.0)
- added L114: 100nH, Inductor_SMD:L_1008_2520Metric, F.Cu at (216.2, 89.8)
- added L115: 100nH, Inductor_SMD:L_1008_2520Metric, F.Cu at (216.2, 93.5)
- added L116: 100nH, Inductor_SMD:L_1008_2520Metric, F.Cu at (216.2, 97.3)
- added L117: 100nH, Inductor_SMD:L_1008_2520Metric, F.Cu at (216.2, 101.0)
- added L118: 100nH, Inductor_SMD:L_1008_2520Metric, F.Cu at (216.2, 104.8)
- added L119: 100nH, Inductor_SMD:L_1008_2520Metric, F.Cu at (216.2, 108.5)
- added L120: 100nH, Inductor_SMD:L_1008_2520Metric, F.Cu at (221.1, 63.5)
- added L121: 100nH, Inductor_SMD:L_1008_2520Metric, F.Cu at (221.1, 67.3)
- added L122: 100nH, Inductor_SMD:L_1008_2520Metric, F.Cu at (221.1, 71.0)
- added L123: 100nH, Inductor_SMD:L_1008_2520Metric, F.Cu at (221.1, 74.8)
- added L124: 100nH, Inductor_SMD:L_1008_2520Metric, F.Cu at (221.1, 78.5)
- added L125: 100nH, Inductor_SMD:L_1008_2520Metric, F.Cu at (221.1, 82.3)
- added L126: 100nH, Inductor_SMD:L_1008_2520Metric, F.Cu at (221.1, 86.0)
- added L127: 100nH, Inductor_SMD:L_1008_2520Metric, F.Cu at (221.1, 89.8)
- added L128: 100nH, Inductor_SMD:L_1008_2520Metric, F.Cu at (221.1, 93.5)
- added L129: 100uH, Inductor_SMD:L_0805_2012Metric, F.Cu at (225.9, 63.0)
- added L130: 100uH, Inductor_SMD:L_0805_2012Metric, F.Cu at (225.9, 65.8)
- added L131: 100uH, Inductor_SMD:L_0805_2012Metric, F.Cu at (225.9, 68.5)
- added L132: 100uH, Inductor_SMD:L_0805_2012Metric, F.Cu at (225.9, 71.3)
- added L133: 100uH, Inductor_SMD:L_0805_2012Metric, F.Cu at (230.4, 63.0)
- added L134: 100uH, Inductor_SMD:L_0805_2012Metric, F.Cu at (230.4, 65.8)
- added L135: 100uH, Inductor_SMD:L_0805_2012Metric, F.Cu at (230.4, 68.5)
- added L136: 100uH, Inductor_SMD:L_0805_2012Metric, F.Cu at (230.4, 71.3)
- added L137: 100uH, Inductor_SMD:L_0805_2012Metric, F.Cu at (235.0, 63.0)
- added L138: 100uH, Inductor_SMD:L_0805_2012Metric, F.Cu at (235.0, 65.8)
- added L139: 100uH, Inductor_SMD:L_0805_2012Metric, F.Cu at (235.0, 68.5)
- added L140: 100uH, Inductor_SMD:L_0805_2012Metric, F.Cu at (235.0, 71.3)
- added L37: 100nH, Inductor_SMD:L_1008_2520Metric, F.Cu at (196.4, 71.0)
- added L38: 100nH, Inductor_SMD:L_1008_2520Metric, F.Cu at (196.4, 74.8)
- added L39: 100nH, Inductor_SMD:L_1008_2520Metric, F.Cu at (196.4, 78.5)
- added L40: 100nH, Inductor_SMD:L_1008_2520Metric, F.Cu at (196.4, 82.3)
- added L41: 100nH, Inductor_SMD:L_1008_2520Metric, F.Cu at (196.4, 86.0)
- added L42: 100nH, Inductor_SMD:L_1008_2520Metric, F.Cu at (196.4, 89.8)
- added L43: 100nH, Inductor_SMD:L_1008_2520Metric, F.Cu at (196.4, 93.5)
- added L5: 100nH, Inductor_SMD:L_1008_2520Metric, F.Cu at (186.5, 63.5)
- added L64: 100nH, Inductor_SMD:L_1008_2520Metric, F.Cu at (196.4, 97.3)
- added L65: 100nH, Inductor_SMD:L_1008_2520Metric, F.Cu at (196.4, 101.0)
- added L66: 100nH, Inductor_SMD:L_1008_2520Metric, F.Cu at (196.4, 104.8)
- added L67: 100nH, Inductor_SMD:L_1008_2520Metric, F.Cu at (196.4, 108.5)
- added L68: 100nH, Inductor_SMD:L_1008_2520Metric, F.Cu at (201.3, 63.5)
- added L69: 100nH, Inductor_SMD:L_1008_2520Metric, F.Cu at (201.3, 67.3)
- added L70: 100nH, Inductor_SMD:L_1008_2520Metric, F.Cu at (201.3, 71.0)
- added L71: 100nH, Inductor_SMD:L_1008_2520Metric, F.Cu at (201.3, 74.8)
- added L72: 100nH, Inductor_SMD:L_1008_2520Metric, F.Cu at (201.3, 78.5)
- added L73: 100nH, Inductor_SMD:L_1008_2520Metric, F.Cu at (201.3, 82.3)
- added L74: 100nH, Inductor_SMD:L_1008_2520Metric, F.Cu at (201.3, 86.0)
- added L75: 100nH, Inductor_SMD:L_1008_2520Metric, F.Cu at (201.3, 89.8)
- added L76: 100nH, Inductor_SMD:L_1008_2520Metric, F.Cu at (201.3, 93.5)
- added L77: 100nH, Inductor_SMD:L_1008_2520Metric, F.Cu at (201.3, 97.3)
- added L78: 100nH, Inductor_SMD:L_1008_2520Metric, F.Cu at (201.3, 101.0)
- added L79: 100nH, Inductor_SMD:L_1008_2520Metric, F.Cu at (201.3, 104.8)
- added L80: 100nH, Inductor_SMD:L_1008_2520Metric, F.Cu at (201.3, 108.5)
- added L81: 100nH, Inductor_SMD:L_1008_2520Metric, F.Cu at (206.3, 63.5)
- added L82: 100nH, Inductor_SMD:L_1008_2520Metric, F.Cu at (206.3, 67.3)
- added L83: 100nH, Inductor_SMD:L_1008_2520Metric, F.Cu at (206.3, 71.0)
- added L84: 100nH, Inductor_SMD:L_1008_2520Metric, F.Cu at (206.3, 74.8)
- added L85: 100nH, Inductor_SMD:L_1008_2520Metric, F.Cu at (206.3, 78.5)
- added L86: 100nH, Inductor_SMD:L_1008_2520Metric, F.Cu at (206.3, 82.3)
- added L87: 100nH, Inductor_SMD:L_1008_2520Metric, F.Cu at (206.3, 86.0)
- added L88: 100nH, Inductor_SMD:L_1008_2520Metric, F.Cu at (206.3, 89.8)
- added L89: 100nH, Inductor_SMD:L_1008_2520Metric, F.Cu at (206.3, 93.5)
- added L90: 100nH, Inductor_SMD:L_1008_2520Metric, F.Cu at (206.3, 97.3)
- added L91: 100nH, Inductor_SMD:L_1008_2520Metric, F.Cu at (206.3, 101.0)
- added L92: 100nH, Inductor_SMD:L_1008_2520Metric, F.Cu at (206.3, 104.8)
- added L93: 100nH, Inductor_SMD:L_1008_2520Metric, F.Cu at (206.3, 108.5)
- added L94: 100nH, Inductor_SMD:L_1008_2520Metric, F.Cu at (211.2, 63.5)
- added L95: 100nH, Inductor_SMD:L_1008_2520Metric, F.Cu at (211.2, 67.3)
- added L96: 100nH, Inductor_SMD:L_1008_2520Metric, F.Cu at (211.2, 71.0)
- added L97: 100nH, Inductor_SMD:L_1008_2520Metric, F.Cu at (211.2, 74.8)
- added L98: 100nH, Inductor_SMD:L_1008_2520Metric, F.Cu at (211.2, 78.5)
- added L99: 100nH, Inductor_SMD:L_1008_2520Metric, F.Cu at (211.2, 82.3)
- added Q27: 2N7002, Package_TO_SOT_SMD:SOT-23, F.Cu at (247.3, 107.6)
- added Q28: HY1904C2, kicad-parts:HY1904C2, F.Cu at (249.1, 98.5)
- added Q29: 2N7002, Package_TO_SOT_SMD:SOT-23, F.Cu at (247.3, 74.2)
- added Q30: HY1904C2, kicad-parts:HY1904C2, F.Cu at (249.1, 65.1)
- added Q31: 2N7002, Package_TO_SOT_SMD:SOT-23, F.Cu at (208.1, 124.9)
- added Q32: HY1904C2, kicad-parts:HY1904C2, F.Cu at (209.9, 115.8)
- added Q33: 2N7002, Package_TO_SOT_SMD:SOT-23, F.Cu at (263.4, 90.9)
- added Q34: HY1904C2, kicad-parts:HY1904C2, F.Cu at (265.2, 81.8)
- added Q35: 2N7002, Package_TO_SOT_SMD:SOT-23, F.Cu at (208.1, 141.6)
- added Q36: HY1904C2, kicad-parts:HY1904C2, F.Cu at (209.9, 132.5)
- added Q37: 2N7002, Package_TO_SOT_SMD:SOT-23, F.Cu at (263.4, 74.2)
- added Q38: HY1904C2, kicad-parts:HY1904C2, F.Cu at (265.2, 65.1)
- added Q39: 2N7002, Package_TO_SOT_SMD:SOT-23, F.Cu at (240.2, 124.9)
- added Q40: HY1904C2, kicad-parts:HY1904C2, F.Cu at (242.0, 115.8)
- added Q41: 2N7002, Package_TO_SOT_SMD:SOT-23, F.Cu at (192.1, 141.6)
- added Q42: HY1904C2, kicad-parts:HY1904C2, F.Cu at (193.8, 132.5)
- added Q43: 2N7002, Package_TO_SOT_SMD:SOT-23, F.Cu at (192.1, 124.9)
- added Q44: HY1904C2, kicad-parts:HY1904C2, F.Cu at (193.8, 115.8)
- added Q45: 2N7002, Package_TO_SOT_SMD:SOT-23, F.Cu at (240.2, 141.6)
- added Q46: HY1904C2, kicad-parts:HY1904C2, F.Cu at (242.0, 132.5)
- added Q47: 2N7002, Package_TO_SOT_SMD:SOT-23, F.Cu at (224.2, 141.6)
- added Q48: HY1904C2, kicad-parts:HY1904C2, F.Cu at (226.0, 132.5)
- added Q49: 2N7002, Package_TO_SOT_SMD:SOT-23, F.Cu at (247.3, 90.9)
- added Q50: HY1904C2, kicad-parts:HY1904C2, F.Cu at (249.1, 81.8)
- added Q51: 2N7002, Package_TO_SOT_SMD:SOT-23, F.Cu at (263.4, 107.6)
- added Q52: HY1904C2, kicad-parts:HY1904C2, F.Cu at (265.2, 98.5)
- added Q53: 2N7002, Package_TO_SOT_SMD:SOT-23, F.Cu at (224.2, 124.9)
- added Q54: HY1904C2, kicad-parts:HY1904C2, F.Cu at (226.0, 115.8)
- added R100: 1K 0.25W, Resistor_SMD:R_1206_3216Metric, F.Cu at (235.0, 130.8)
- added R101: 6.8K 0.25W, Resistor_SMD:R_1206_3216Metric, F.Cu at (235.0, 134.1)
- added R102: 6.8K 0.25W, Resistor_SMD:R_1206_3216Metric, F.Cu at (235.0, 137.3)
- added R103: 1K 0.25W, Resistor_SMD:R_1206_3216Metric, F.Cu at (235.0, 140.6)
- added R104: 1K 0.25W, Resistor_SMD:R_1206_3216Metric, F.Cu at (218.9, 130.8)
- added R105: 6.8K 0.25W, Resistor_SMD:R_1206_3216Metric, F.Cu at (218.9, 134.1)
- added R106: 6.8K 0.25W, Resistor_SMD:R_1206_3216Metric, F.Cu at (218.9, 137.3)
- added R107: 1K 0.25W, Resistor_SMD:R_1206_3216Metric, F.Cu at (218.9, 140.6)
- added R108: 1K 0.25W, Resistor_SMD:R_1206_3216Metric, F.Cu at (242.1, 80.0)
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Connections:
- net /PA Switched RF Choke/L-100UH-A renamed /PA Switched Resonator/L-100UH-A
- net /PA Switched RF Choke/L-100UH-B renamed Net-(L131-Pad2)
- net /PA Switched RF Choke/L-50UH-A renamed /PA Switched Resonator/L-50UH-A
- net /PA Switched RF Choke/L-50UH-B renamed /PA Switched Resonator/L-50UH-B
- L10 pad 1: Net-(L10-Pad1) -> /PA Switched Resonator/L-10UH-A
- L11 pad 1: Net-(L10-Pad2) -> /PA Switched Resonator/L-10UH-A
- L11 pad 2: Net-(L11-Pad2) -> Net-(L10-Pad2)
- L12 pad 1: Net-(L11-Pad2) -> /PA Switched Resonator/L-10UH-A
- L12 pad 2: Net-(L12-Pad2) -> Net-(L10-Pad2)
- L13 pad 1: Net-(L12-Pad2) -> Net-(L10-Pad2)
- L14 pad 1: /PA Switched RF Choke/L-10UH-A -> Net-(L10-Pad2)
- L14 pad 2: Net-(L14-Pad2) -> Net-(L13-Pad2)
- L15 pad 1: /PA Switched RF Choke/L-10UH-A -> Net-(L10-Pad2)
- L15 pad 2: Net-(L14-Pad2) -> Net-(L13-Pad2)
- L16 pad 1: /PA Switched RF Choke/L-10UH-A -> Net-(L10-Pad2)
- L16 pad 2: Net-(L14-Pad2) -> Net-(L13-Pad2)
- L17 pad 1: Net-(L14-Pad2) -> Net-(L10-Pad2)
- L17 pad 2: Net-(L17-Pad2) -> Net-(L13-Pad2)
- L18 pad 1: Net-(L14-Pad2) -> Net-(L13-Pad2)
- L18 pad 2: Net-(L17-Pad2) -> Net-(L18-Pad2)
- L19 pad 1: Net-(L14-Pad2) -> Net-(L13-Pad2)
- L19 pad 2: Net-(L17-Pad2) -> Net-(L18-Pad2)
- L20 pad 1: Net-(L17-Pad2) -> Net-(L13-Pad2)
- L20 pad 2: Net-(L10-Pad1) -> Net-(L18-Pad2)
- L21 pad 1: Net-(L17-Pad2) -> Net-(L13-Pad2)
- L21 pad 2: Net-(L10-Pad1) -> Net-(L18-Pad2)
- L22 pad 1: Net-(L17-Pad2) -> Net-(L13-Pad2)
- L22 pad 2: Net-(L10-Pad1) -> Net-(L18-Pad2)
- L23 pad 1: Net-(L13-Pad2) -> Net-(L18-Pad2)
- L24 pad 1: Net-(L23-Pad2) -> Net-(L18-Pad2)
- L24 pad 2: /PA Switched RF Choke/L-10UH-B -> Net-(L23-Pad2)
- L25 pad 1: Net-(L10-Pad1) -> Net-(L18-Pad2)
- L25 pad 2: Net-(L10-Pad2) -> Net-(L23-Pad2)
- L26 pad 1: Net-(L10-Pad2) -> Net-(L18-Pad2)
- L26 pad 2: Net-(L11-Pad2) -> Net-(L23-Pad2)
- L27 pad 1: Net-(L11-Pad2) -> Net-(L18-Pad2)
- L27 pad 2: Net-(L12-Pad2) -> Net-(L23-Pad2)
- L28 pad 1: Net-(L12-Pad2) -> Net-(L23-Pad2)
- L28 pad 2: Net-(L13-Pad2) -> Net-(L28-Pad2)
- L29 pad 1: Net-(L13-Pad2) -> Net-(L23-Pad2)
- L29 pad 2: Net-(L23-Pad2) -> Net-(L28-Pad2)
- L30 pad 2: /PA Switched RF Choke/L-10UH-B -> Net-(L28-Pad2)
- L31 pad 1: Net-(L10-Pad1) -> Net-(L23-Pad2)
- L31 pad 2: Net-(L10-Pad2) -> Net-(L28-Pad2)
- L32 pad 1: Net-(L10-Pad2) -> Net-(L23-Pad2)
- L32 pad 2: Net-(L11-Pad2) -> Net-(L28-Pad2)
- L33 pad 1: Net-(L11-Pad2) -> Net-(L28-Pad2)
- L33 pad 2: Net-(L12-Pad2) -> Net-(L33-Pad2)
- L34 pad 1: Net-(L12-Pad2) -> Net-(L28-Pad2)
- L34 pad 2: Net-(L13-Pad2) -> Net-(L33-Pad2)
- L35 pad 1: Net-(L13-Pad2) -> Net-(L28-Pad2)
- L35 pad 2: Net-(L23-Pad2) -> Net-(L33-Pad2)
- L36 pad 1: Net-(L23-Pad2) -> Net-(L28-Pad2)
- L36 pad 2: /PA Switched RF Choke/L-10UH-B -> Net-(L33-Pad2)
Other:
- board text added: "5 TIER CHINESE TIFFIN LUNCH BOX"
- board text added: "ATU/ANT OUT LPF/SWR DISPLAY PA/RF CHOKE MCU/TIMING PSU"
- board text added: "POTENTIAL TIERS:"
- board text added: "https://duckduckgo.com/?q=hellema+spiced+cookies+tin"
- board text added: "https://www.aliexpress.com/item/1005006756495960.html https://www.aliexpress.com/item/1005006075889043.html"
- board text added: "https://www.aliexpress.com/item/1005006978580242.html"
