File: kicad-pcbs/adxi/adxi.kicad_pcb (KiCad board)
At the start: 4 copper layers, 106.9 x 124.1 mm, 396 parts, among them J1 FROM-PC-SPK, J10 BANDMODULE3-ANT, J11 BANDMODULE4-ANT, J12 BANDMODULE3-PA, J13 BANDMODULE4-PA, J14 BANDMODULE5-ANT, J15 BANDMODULE6-ANT, J16 BANDMODULE5-PA, J17 BANDMODULE6-PA, J18 MMCX, J2 TO-PC-MIC, J20 LCD-2004, J3 BNC, J4 SMA, J5 12V SUPPLY, J6 BANDMODULE1-ANT, J7 BANDMODULE1-PA, J8 BANDMODULE2-ANT, J9 BANDMODULE2-PA, Q1 MMBF170, Q10 HY1904C2, Q11 2N7002, Q12 HY1904C2, Q13 2N7002, Q14 HY1904C2, Q15 2N7002, Q16 HY1904C2, Q17 2N7002, Q18 HY1904C2, Q19 2N7002, Q2 HY1904C2, Q20 HY1904C2, Q21 2N7002, Q22 HY1904C2, Q23 2N7002, Q24 HY1904C2, Q25 2N7002, Q26 HY1904C2, Q27 2N7002, Q28 HY1904C2, Q29 2N7002, Q3 2N7002, Q30 HY1904C2, Q31 2N7002, Q32 HY1904C2, Q33 2N7002, Q34 HY1904C2, Q35 2N7002, Q36 HY1904C2, Q37 2N7002, Q38 HY1904C2, Q39 2N7002, Q4 HY1904C2, Q40 HY1904C2, Q41 2N7002, Q42 HY1904C2, Q43 2N7002, Q44 HY1904C2, Q45 2N7002, Q46 HY1904C2, Q47 2N7002, Q48 HY1904C2, Q49 2N7002, Q5 2N7002, Q50 HY1904C2, Q51 2N7002, Q52 HY1904C2, Q53 2N7002, Q54 HY1904C2, Q6 HY1904C2, Q63 2N7002, Q64 HY1904C2, Q7 2N7002, Q8 HY1904C2, Q9 2N7002, U1 CD2003, U3 74ACT244, U4 Si5351A-B-GT

Commit message: Rationalize
Parts:
- removed the C16 at (65.2, 137.0)
- removed the C21 at (58.5, 141.3)
- removed the D10 at (64.6, 39.4)
- removed the D11 at (62.7, 49.2)
- removed the D12 at (59.7, 76.2)
- removed the D13 at (57.9, 98.7)
- removed the D14 at (104.9, 62.3)
- removed the D15 at (105.1, 81.3)
- removed the D16 at (105.2, 51.0)
- removed the D17 at (104.9, 75.6)
- removed the D18 at (108.6, 97.1)
- removed the D9 at (54.2, 95.1)
- removed D98: BZT52C12, Diode_SMD:D_SOD-123
- removed J10: BANDMODULE3-ANT, Connector_PinSocket_2.54mm:PinSocket_1x07_P2.54mm_Vertical
- removed J11: BANDMODULE4-ANT, Connector_PinSocket_2.54mm:PinSocket_1x07_P2.54mm_Vertical
- removed J12: BANDMODULE3-PA, Connector_PinSocket_2.54mm:PinSocket_1x07_P2.54mm_Vertical
- removed J13: BANDMODULE4-PA, Connector_PinSocket_2.54mm:PinSocket_1x07_P2.54mm_Vertical
- removed J14: BANDMODULE5-ANT, Connector_PinSocket_2.54mm:PinSocket_1x07_P2.54mm_Vertical
- removed J15: BANDMODULE6-ANT, Connector_PinSocket_2.54mm:PinSocket_1x07_P2.54mm_Vertical
- removed J16: BANDMODULE5-PA, Connector_PinSocket_2.54mm:PinSocket_1x07_P2.54mm_Vertical
- removed J17: BANDMODULE6-PA, Connector_PinSocket_2.54mm:PinSocket_1x07_P2.54mm_Vertical
- removed J20: LCD-2004, Connector_PinHeader_2.54mm:PinHeader_1x04_P2.54mm_Vertical
- removed the J5 at (39.3, 136.2)
- removed the J6 at (52.9, 30.6)
- removed J9: BANDMODULE2-PA, Connector_PinSocket_2.54mm:PinSocket_1x07_P2.54mm_Vertical
- removed the Q10 at (64.0, 54.2)
- removed the Q11 at (60.1, 80.3)
- removed the Q12 at (58.4, 71.2)
- removed the Q13 at (57.4, 94.7)
- removed the Q14 at (59.2, 103.7)
- removed the Q15 at (105.4, 58.2)
- removed the Q16 at (103.6, 67.3)
- removed the Q17 at (105.6, 77.2)
- removed the Q18 at (103.8, 86.3)
- removed the Q19 at (105.6, 55.1)
- removed the Q20 at (103.9, 46.0)
- removed the Q21 at (105.4, 79.7)
- removed the Q22 at (103.6, 70.6)
- removed the Q23 at (108.1, 93.0)
- removed the Q24 at (109.9, 102.1)
- removed the Q3 at (66.0, 55.6)
- removed the Q4 at (58.5, 67.7)
- removed the Q5 at (64.4, 94.6)
- removed the Q6 at (58.5, 90.6)
- removed Q63: 2N7002, Package_TO_SOT_SMD:SOT-23
- removed Q64: HY1904C2, kicad-parts:HY1904C2
- removed the Q7 at (64.2, 43.5)
- removed the Q8 at (57.9, 45.3)
- removed the Q9 at (62.2, 45.1)
- removed R136, R139: 1K 0.25W, Resistor_SMD:R_1206_3216Metric
- removed R137, R138: 6.8K 0.25W, Resistor_SMD:R_1206_3216Metric
- removed the R16 at (65.8, 69.3)
- removed the R17 at (65.8, 66.0)
- removed the R18 at (65.8, 62.8)
- removed the R19 at (65.8, 59.5)
- removed the R20 at (64.1, 97.7)
- removed the R21 at (64.8, 89.2)
- removed the R22 at (64.8, 91.6)
- removed the R23 at (59.2, 95.1)
- removed the R24 at (58.9, 32.7)
- removed the R25 at (58.9, 36.0)
- removed the R26 at (58.9, 39.2)
- removed the R27 at (65.2, 46.7)
- removed the R28 at (57.0, 56.0)
- removed the R29 at (57.0, 52.7)
- removed the R30 at (57.0, 49.4)
- removed the R31 at (57.0, 46.1)
- removed the R32 at (65.4, 69.4)
- removed the R33 at (65.4, 72.7)
- removed the R34 at (65.4, 76.0)
- removed the R35 at (65.4, 79.3)
- removed the R36 at (52.1, 105.5)
- removed the R37 at (52.1, 102.2)
- removed the R38 at (52.1, 98.9)
- removed the R39 at (52.1, 95.6)
- removed the R40 at (110.7, 69.0)
- removed the R41 at (110.7, 65.7)
- removed the R42 at (110.7, 62.5)
- removed the R43 at (110.7, 59.2)
- removed the R44 at (110.8, 88.0)
- removed the R45 at (110.8, 84.7)
- removed the R46 at (110.8, 81.5)
- removed the R47 at (110.8, 78.2)
- removed the R48 at (110.9, 44.2)
- removed the R49 at (110.9, 47.5)
- removed the R50 at (110.9, 50.8)
- removed the R51 at (110.9, 54.1)
- removed the R52 at (110.7, 68.9)
- removed the R53 at (110.7, 72.1)
- removed the R54 at (110.7, 75.4)
- removed the R55 at (110.7, 78.7)
- removed the R56 at (102.9, 103.8)
- removed the R57 at (102.9, 100.5)
- removed the R58 at (102.9, 97.3)
- removed the R59 at (102.9, 94.0)
- added C20: 470uF, Capacitor_SMD:C_Elec_10x10.2, F.Cu at (308.0, 20.1)
- added C25: 10uF, Capacitor_SMD:C_1206_3216Metric, F.Cu at (292.2, 32.1)
- added C29: 22nF, Capacitor_SMD:C_1206_3216Metric, F.Cu at (260.1, 22.1)
- added C30: 1nF, Capacitor_SMD:C_0805_2012Metric, F.Cu at (269.2, 25.3)
- added C31: 100pF, Capacitor_SMD:C_0603_1608Metric, F.Cu at (264.9, 25.1)
- added C33: 10pF, Capacitor_SMD:C_0603_1608Metric, F.Cu at (264.9, 27.6)
- added C34: 1pF, Capacitor_SMD:C_0402_1005Metric, F.Cu at (268.4, 27.8)
- added FB2: 100mΩ/3A, Capacitor_SMD:C_1206_3216Metric, F.Cu at (260.1, 25.5)
- added L10: 18nH, Inductor_SMD:L_1210_3225Metric, F.Cu at (260.1, 18.4)
- added L11: 18nH, Inductor_SMD:L_1210_3225Metric, F.Cu at (265.7, -2.70)
- added L12: 18nH, Inductor_SMD:L_1210_3225Metric, F.Cu at (265.7, 1.51)
- added L13: 18nH, Inductor_SMD:L_1210_3225Metric, F.Cu at (265.7, 5.72)
- added L14: 18nH, Inductor_SMD:L_1210_3225Metric, F.Cu at (265.7, 9.93)
- added L15: 18nH, Inductor_SMD:L_1210_3225Metric, F.Cu at (265.7, 14.1)
- added L16: 18nH, Inductor_SMD:L_1210_3225Metric, F.Cu at (265.7, 18.4)
- added L17: 18nH, Inductor_SMD:L_1210_3225Metric, F.Cu at (271.3, -2.70)
- added L18: 18nH, Inductor_SMD:L_1210_3225Metric, F.Cu at (271.3, 1.51)
- added L19: 18nH, Inductor_SMD:L_1210_3225Metric, F.Cu at (271.3, 5.72)
- added L20: 100uH, Inductor_SMD:L_Cenker_CKCS8040, F.Cu at (252.2, 0.01)
- added L21: 100uH, Inductor_SMD:L_Cenker_CKCS8040, F.Cu at (252.2, 9.65)
- added L22: 100uH, Inductor_SMD:L_Cenker_CKCS8040, F.Cu at (252.2, 19.3)
- added L23: 100uH, Inductor_SMD:L_Cenker_CKCS8040, F.Cu at (252.2, 28.9)
- added L24: 470nH, Inductor_SMD:L_1008_2520Metric, F.Cu at (220.0, -2.93)
- added L25: 470nH, Inductor_SMD:L_1008_2520Metric, F.Cu at (220.0, 0.82)
- added L26: 470nH, Inductor_SMD:L_1008_2520Metric, F.Cu at (220.0, 4.57)
- added L27: 470nH, Inductor_SMD:L_1008_2520Metric, F.Cu at (220.0, 8.32)
- added L28: 470nH, Inductor_SMD:L_1008_2520Metric, F.Cu at (220.0, 12.1)
- added L29: 470nH, Inductor_SMD:L_1008_2520Metric, F.Cu at (220.0, 15.8)
- added L30: 470nH, Inductor_SMD:L_1008_2520Metric, F.Cu at (220.0, 19.6)
- added L31: 470nH, Inductor_SMD:L_1008_2520Metric, F.Cu at (220.0, 23.3)
- added L32: 470nH, Inductor_SMD:L_1008_2520Metric, F.Cu at (220.0, 27.1)
- added L33: 470nH, Inductor_SMD:L_1008_2520Metric, F.Cu at (220.0, 30.8)
- added L34: 470nH, Inductor_SMD:L_1008_2520Metric, F.Cu at (220.0, 34.6)
- added L35: 470nH, Inductor_SMD:L_1008_2520Metric, F.Cu at (224.9, -2.93)
- added L36: 470nH, Inductor_SMD:L_1008_2520Metric, F.Cu at (224.9, 0.82)
- added L37: 470nH, Inductor_SMD:L_1008_2520Metric, F.Cu at (224.9, 4.57)
- added L38: 470nH, Inductor_SMD:L_1008_2520Metric, F.Cu at (224.9, 8.32)
- added L39: 470nH, Inductor_SMD:L_1008_2520Metric, F.Cu at (224.9, 12.1)
- added L40: 470nH, Inductor_SMD:L_1008_2520Metric, F.Cu at (224.9, 15.8)
- added L41: 470nH, Inductor_SMD:L_1008_2520Metric, F.Cu at (224.9, 19.6)
- added L42: 470nH, Inductor_SMD:L_1008_2520Metric, F.Cu at (224.9, 23.3)
- added L43: 470nH, Inductor_SMD:L_1008_2520Metric, F.Cu at (224.9, 27.1)
- added L44: 470nH, Inductor_SMD:L_1008_2520Metric, F.Cu at (224.9, 30.8)
- added L45: 470nH, Inductor_SMD:L_1008_2520Metric, F.Cu at (224.9, 34.6)
- added L46: 470nH, Inductor_SMD:L_1008_2520Metric, F.Cu at (229.9, -2.93)
- added L47: 470nH, Inductor_SMD:L_1008_2520Metric, F.Cu at (229.9, 0.82)
- added L48: 470nH, Inductor_SMD:L_1008_2520Metric, F.Cu at (229.9, 4.57)
- added L49: 470nH, Inductor_SMD:L_1008_2520Metric, F.Cu at (229.9, 8.32)
- added L5: 33nH, Inductor_SMD:L_1210_3225Metric, F.Cu at (260.1, -2.70)
- added L50: 470nH, Inductor_SMD:L_1008_2520Metric, F.Cu at (229.9, 12.1)
- added L51: 470nH, Inductor_SMD:L_1008_2520Metric, F.Cu at (229.9, 15.8)
- added L52: 470nH, Inductor_SMD:L_1008_2520Metric, F.Cu at (229.9, 19.6)
- added L53: 470nH, Inductor_SMD:L_1008_2520Metric, F.Cu at (229.9, 23.3)
- added L54: 470nH, Inductor_SMD:L_1008_2520Metric, F.Cu at (229.9, 27.1)
- added L55: 470nH, Inductor_SMD:L_1008_2520Metric, F.Cu at (229.9, 30.8)
- added L56: 470nH, Inductor_SMD:L_1008_2520Metric, F.Cu at (229.9, 34.6)
- added L57: 470nH, Inductor_SMD:L_1008_2520Metric, F.Cu at (234.8, -2.93)
- added L58: 470nH, Inductor_SMD:L_1008_2520Metric, F.Cu at (234.8, 0.82)
- added L59: 470nH, Inductor_SMD:L_1008_2520Metric, F.Cu at (234.8, 4.57)
- added L6: 33nH, Inductor_SMD:L_1210_3225Metric, F.Cu at (260.1, 1.51)
- added L60: 470nH, Inductor_SMD:L_1008_2520Metric, F.Cu at (234.8, 8.32)
- added L61: 470nH, Inductor_SMD:L_1008_2520Metric, F.Cu at (234.8, 12.1)
- added L62: 470nH, Inductor_SMD:L_1008_2520Metric, F.Cu at (234.8, 15.8)
- added L63: 470nH, Inductor_SMD:L_1008_2520Metric, F.Cu at (234.8, 19.6)
- added L64: 470nH, Inductor_SMD:L_1008_2520Metric, F.Cu at (234.8, 23.3)
- added L65: 470nH, Inductor_SMD:L_1008_2520Metric, F.Cu at (234.8, 27.1)
- added L66: 470nH, Inductor_SMD:L_1008_2520Metric, F.Cu at (234.8, 30.8)
- added L67: 470nH, Inductor_SMD:L_1008_2520Metric, F.Cu at (234.8, 34.6)
- added L68: 470nH, Inductor_SMD:L_1008_2520Metric, F.Cu at (239.8, -2.93)
- added L69: 470nH, Inductor_SMD:L_1008_2520Metric, F.Cu at (239.8, 0.82)
- added L7: 33nH, Inductor_SMD:L_1210_3225Metric, F.Cu at (260.1, 5.72)
- added L70: 470nH, Inductor_SMD:L_1008_2520Metric, F.Cu at (239.8, 4.57)
- added L71: 470nH, Inductor_SMD:L_1008_2520Metric, F.Cu at (239.8, 8.32)
- added L72: 470nH, Inductor_SMD:L_1008_2520Metric, F.Cu at (239.8, 12.1)
- added L73: 470nH, Inductor_SMD:L_1008_2520Metric, F.Cu at (239.8, 15.8)
- added L74: 470nH, Inductor_SMD:L_1008_2520Metric, F.Cu at (239.8, 19.6)
- added L75: 470nH, Inductor_SMD:L_1008_2520Metric, F.Cu at (239.8, 23.3)
- added L76: 470nH, Inductor_SMD:L_1008_2520Metric, F.Cu at (239.8, 27.1)
- added L77: 470nH, Inductor_SMD:L_1008_2520Metric, F.Cu at (239.8, 30.8)
- added L78: 470nH, Inductor_SMD:L_1008_2520Metric, F.Cu at (239.8, 34.6)
- added L79: 470nH, Inductor_SMD:L_1008_2520Metric, F.Cu at (244.8, -2.93)
- added L8: 33nH, Inductor_SMD:L_1210_3225Metric, F.Cu at (260.1, 9.93)
- added L80: 470nH, Inductor_SMD:L_1008_2520Metric, F.Cu at (244.8, 0.82)
- added L81: 470nH, Inductor_SMD:L_1008_2520Metric, F.Cu at (244.8, 4.57)
- added L82: 470nH, Inductor_SMD:L_1008_2520Metric, F.Cu at (244.8, 8.32)
- added L83: 470nH, Inductor_SMD:L_1008_2520Metric, F.Cu at (244.8, 12.1)
- added L84: 470nH, Inductor_SMD:L_1008_2520Metric, F.Cu at (244.8, 15.8)
- added L85: 470nH, Inductor_SMD:L_1008_2520Metric, F.Cu at (244.8, 19.6)
- added L86: 470nH, Inductor_SMD:L_1008_2520Metric, F.Cu at (244.8, 23.3)
- added L87: 470nH, Inductor_SMD:L_1008_2520Metric, F.Cu at (244.8, 27.1)
- added L88: 470nH, Inductor_SMD:L_1008_2520Metric, F.Cu at (244.8, 30.8)
- added L89: 470nH, Inductor_SMD:L_1008_2520Metric, F.Cu at (244.8, 34.6)
- added L9: 33nH, Inductor_SMD:L_1210_3225Metric, F.Cu at (260.1, 14.1)
- added U5: 74HC595, Package_SO:SOIC-16_3.9x9.9mm_P1.27mm, F.Cu at (221.8, 44.3)
- added U6: 74HC595, Package_SO:SOIC-16_3.9x9.9mm_P1.27mm, F.Cu at (230.2, 44.3)
- C23: value 10uF -> 100nF; footprint Capacitor_SMD:C_1206_3216Metric -> Capacitor_SMD:C_0805_2012Metric
- D8: value BZT52C12 -> BZT52C5V6
- J7: value BANDMODULE1-PA -> 12V SUPPLY; footprint Connector_PinSocket_2.54mm:PinSocket_1x07_P2.54mm_Vertical -> Connector_BarrelJack:BarrelJack_GCT_DCJ200-10-A_Horizontal
- J8: value BANDMODULE2-ANT -> LCD-2004; footprint Connector_PinSocket_2.54mm:PinSocket_1x07_P2.54mm_Vertical -> Connector_PinHeader_2.54mm:PinHeader_1x04_P2.54mm_Vertical
- moved D7 277.3 mm to (297.1, 34.8), turned to 0 degrees
- moved FB1 276.4 mm to (292.2, 35.5), turned to 0 degrees
- moved L4 267.8 mm to (292.6, 23.4), turned to 0 degrees
- moved C18 265.3 mm to (308.0, 8.28), turned to 0 degrees
- moved C23 246.0 mm to (297.3, 32.0)
- moved L3 238.0 mm to (292.6, 9.38), turned to 0 degrees
- moved J8 235.2 mm to (287.1, 32.8)
- moved D8 204.6 mm to (265.8, 22.1), turned to 0 degrees
- moved J7 182.9 mm to (306.0, 28.1)
- moved R5 83.1 mm to (114.3, 60.6)
- moved U1 83.1 mm to (108.6, 63.3)
- moved U4 83.1 mm to (100.6, 63.8)
- moved R4 83.1 mm to (113.1, 66.3)
- moved J4 50.6 mm to (79.0, 56.3)
- moved J5 50.6 mm to (75.8, 64.8)
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- renumbered C13 to C15, C14 to C16, C19 to C21, C20 to C22, C22 to C24, C30 to C36, C31 to C37, C32 to C38, C33 to C39, C34 to C40, C35 to C41, C36 to C42, C37 to C43, D20 to D10, D21 to D11, D22 to D12, D23 to D13, D24 to D14, D25 to D15, D26 to D16, D27 to D17, D28 to D18, D29 to D19, D30 to D20, D31 to D21, D32 to D22, D33 to D23, D19 to D9, J3 to J4, J18 to J5, J4 to J6, L5 to L100, L14 to L101, L19 to L102, L24 to L103, L29 to L104, L34 to L105, L39 to L106, L65 to L107, L70 to L108, L75 to L109, L10 to L110, L15 to L111, L20 to L112, L25 to L113, L30 to L114, L35 to L115, L40 to L116, L66 to L117, L71 to L118, L76 to L119, L11 to L120, L16 to L121, L21 to L122, L26 to L123, L31 to L124, L36 to L125, L41 to L126, L67 to L127, L72 to L128, L77 to L129, L12 to L130, L17 to L131, L22 to L132, L27 to L133, L32 to L134, L37 to L135, L43 to L136, L68 to L137, L73 to L138, L78 to L139, L79 to L140, L84 to L141, L89 to L142, L94 to L143, L99 to L144, L104 to L145, L109 to L146, L114 to L147, L119 to L148, L124 to L149, L80 to L150, L85 to L151, L90 to L152, L95 to L153, L100 to L154, L105 to L155, L110 to L156, L115 to L157, L120 to L158, L125 to L159, L81 to L160, L86 to L161, L91 to L162, L96 to L163, L101 to L164, L106 to L165, L111 to L166, L116 to L167, L121 to L168, L126 to L169, L82 to L170, L87 to L171, L92 to L172, L97 to L173, L102 to L174, L107 to L175, L112 to L176, L117 to L177, L122 to L178, L127 to L179, L83 to L180, L88 to L181, L93 to L182, L98 to L183, L103 to L184, L108 to L185, L113 to L186, L118 to L187, L123 to L188, L128 to L189, L44 to L190, L46 to L191, L48 to L192, L50 to L193, L52 to L194, L6 to L195, L7 to L196, L133 to L197, L134 to L198, L45 to L199, L47 to L200, L49 to L201, L51 to L202, L53 to L203, L9 to L204, L8 to L205, L135 to L206, L136 to L207, L54 to L208, L55 to L209, L56 to L210, L57 to L211, L58 to L212, L129 to L213, L131 to L214, L137 to L215, L138 to L216, L59 to L217, L60 to L218, L61 to L219, L62 to L220, L63 to L221, L130 to L222, L132 to L223, L139 to L224, L140 to L225, L42 to L90, L13 to L91, L18 to L92, L23 to L93, L28 to L94, L33 to L95, L38 to L96, L64 to L97, L69 to L98, L74 to L99, Q32 to Q10, Q33 to Q11, Q34 to Q12, Q35 to Q13, Q36 to Q14, Q37 to Q15, Q38 to Q16, Q39 to Q17, Q40 to Q18, Q41 to Q19, Q42 to Q20, Q43 to Q21, Q44 to Q22, Q45 to Q23, Q46 to Q24, Q47 to Q25, Q48 to Q26, Q49 to Q27, Q50 to Q28, Q51 to Q29, Q25 to Q3, Q52 to Q30, Q53 to Q31, Q54 to Q32, Q26 to Q4, Q27 to Q5, Q28 to Q6, Q29 to Q7, Q30 to Q8, Q31 to Q9, R8 to R10, R9 to R11, R10 to R12, R11 to R13, R12 to R14, R13 to R15, R60 to R16, R61 to R17, R62 to R18, R63 to R19, R64 to R20, R65 to R21, R66 to R22, R67 to R23, R68 to R24, R69 to R25, R70 to R26, R71 to R27, R72 to R28, R73 to R29, R74 to R30, R75 to R31, R76 to R32, R77 to R33, R78 to R34, R79 to R35, R80 to R36, R81 to R37, R82 to R38, R83 to R39, R14 to R4, R84 to R40, R85 to R41, R86 to R42, R87 to R43, R88 to R44, R89 to R45, R90 to R46, R91 to R47, R92 to R48, R93 to R49, R15 to R5, R94 to R50, R95 to R51, R96 to R52, R97 to R53, R98 to R54, R99 to R55, R100 to R56, R101 to R57, R102 to R58, R103 to R59, R104 to R60, R105 to R61, R106 to R62, R107 to R63, R108 to R64, R109 to R65, R110 to R66, R111 to R67, R112 to R68, R113 to R69, R114 to R70, R115 to R71, R116 to R72, R117 to R73, R118 to R74, R119 to R75, R6 to R8, R7 to R9, U4 to U1, U1 to U2, U3 to U4
Connections:
- net /PA Switched Resonator/PA-SUPPLY renamed ANTENNA-B
- net PA-12V renamed ANTENNA-A
- net PA-DRAIN renamed /PA Switched Resonator/PA-DRAIN
- A1 pad 14: unconnected-(A1-D11-Pad14) -> SPI-MOSI
- A1 pad 15: unconnected-(A1-D12-Pad15) -> SPI-SS-OUTPUTS
- A1 pad 16: unconnected-(A1-D13-Pad16) -> SPI-SCK
- D8 pad 1: Net-(D8-K) -> GND
- D8 pad 2: BM2-ANT -> Net-(D8-A)
- J7 pad 1: GND -> Net-(FB1-Pad1)
- J7 pad 2: BM1-PA -> GND
- J7 pad 3: GND -> (no net)
- J8 pad 2: BM2-ANT -> 3.3V
- J8 pad 3: GND -> I2C-SDA-3.3V
- J8 pad 4: BM2-ANT -> I2C-SCL-3.3V
Routing:
- net ANTENNA: track 127.2 -> 0.00 mm
- net GND: track 45.4 -> 2.44 mm
- net BM3-ANT: track 29.3 -> 0.00 mm
- net BM1-ANT: track 21.2 -> 0.00 mm
- net BM2-ANT: track 20.3 -> 0.00 mm
- net HOST-FSK-INPUT: track 23.0 -> 2.87 mm
- net Net-(Q5-D) (its old number): track 5.49 -> 0.00 mm
- net Net-(D5-A): track 8.49 -> 3.96 mm
- net Net-(C2-Pad2): track 4.43 -> 0.00 mm
- net 12V: track 6.25 -> 3.81 mm
- net Net-(C6-Pad2): track 2.74 -> 1.97 mm
- net unconnected-(A1-D9-Pad12): track 0.69 -> 0.00 mm
- net unconnected-(A1-D12-Pad15): track 0.51 -> 0.00 mm
- added copper zone on F.Cu, net (none)
- removed copper zone on In1.Cu, net GND
Other:
- board size 106.9 x 124.1 mm -> 128.7 x 130 mm
- board text removed: "1"
- board text removed: "2"
- board text removed: "3"
- board text removed: "4"
- board text removed: "5"
- board text removed: "6"
- board text removed: "BAND MODULE"
- board text removed: "LCD"

Commit message: Significant updates
Parts:
- removed C2, C3: 100nF, Capacitor_SMD:C_0805_2012Metric
- removed J1: FROM-PC-SPK, Connector_Audio:Jack_3.5mm_CUI_SJ1-3525N_Horizontal
- removed J2: TO-PC-MIC, Connector_Audio:Jack_3.5mm_CUI_SJ1-3525N_Horizontal
- removed J5: MMCX, Connector_Coaxial:MMCX_Molex_73415-1471_Vertical
- removed J6: SMA, Connector_Coaxial:SMA_Amphenol_901-144_Vertical
- removed R12, R8: 10K, Resistor_SMD:R_1206_3216Metric
- added C44: 10uF, Capacitor_SMD:C_1206_3216Metric, F.Cu at (307.4, 56.7)
- added C45: 10uF, Capacitor_SMD:C_1206_3216Metric, F.Cu at (304.9, 56.6)
- added D24: 1N4148WS, Diode_SMD:D_SOD-323, F.Cu at (302.7, 59.3)
- added D25: 1N4148WS, Diode_SMD:D_SOD-323, F.Cu at (302.6, 55.9)
- added FB3: 100mΩ/3A, Capacitor_SMD:C_1206_3216Metric, F.Cu at (309.9, 66.5)
- added R78: 5.1K, Resistor_SMD:R_0805_2012Metric, F.Cu at (307.3, 74.7)
- added R79: 100K, Resistor_SMD:R_1206_3216Metric, F.Cu at (306.1, 67.8)
- added R80: 100K, Resistor_SMD:R_1206_3216Metric, F.Cu at (306.8, 77.0)
- added R81: 100K, Resistor_SMD:R_1206_3216Metric, F.Cu at (306.1, 65.3)
- added R82: 100K, Resistor_SMD:R_1206_3216Metric, F.Cu at (306.1, 62.7)
- added R83: 100K, Resistor_SMD:R_1206_3216Metric, F.Cu at (306.1, 60.3)
- added R84: 100K, Resistor_SMD:R_1206_3216Metric, F.Cu at (309.9, 58.6)
- added U7: TUSB321, Package_DFN_QFN:Texas_X2QFN-12_1.6x1.6mm_P0.4mm, F.Cu at (310.1, 62.5)
- added U8: MT3608, Package_TO_SOT_SMD:SOT-23-6, F.Cu at (306.7, 71.4)
- J7: value 12V SUPPLY -> 12-24V SUPPLY
Connections:
- net Net-(FB1-Pad1) renamed /VIN-DIRTY
- net Net-(U3-IN) renamed /VIN
- C18 pad 1: Net-(D7-A2) -> /VIN-COMMON
- C20 pad 1: Net-(D7-A2) -> /VIN-COMMON
- C23 pad 2: Net-(D7-A2) -> /VIN-COMMON
- C25 pad 2: Net-(D7-A2) -> /VIN-COMMON
- D7 pad 2: Net-(D7-A2) -> /VIN-CLAMPED
- FB1 pad 2: Net-(D7-A2) -> /VIN-CLAMPED
- J4 pad 1: ANTENNA -> ANTENNA-A
- J4 pad 2: GND -> ANTENNA-B
- L4 pad 1: Net-(D7-A2) -> /VIN-COMMON
Routing:
- net Net-(C2-Pad1): track 3.57 -> 0.00 mm
- net HOST-FSK-INPUT: track 2.87 -> 0.00 mm
- net Net-(C6-Pad2): track 1.97 -> 0.00 mm
Other:
- board size 128.7 x 130 mm -> 129.7 x 130 mm
- board text added: "USB-C-PD"
- board text removed: "IN"
- board text removed: "OUT"
