File: kicad-pcbs/adxi/adxi.kicad_pcb (KiCad board)
At the start: 4 copper layers, 129.7 x 130 mm, 164 parts, among them J2 PA-SUPPLY, J3 USBC, J4 PA-DRAIN, J5 USB2 Type-A, J6 RFC-GND, Q1 MMBF170, Q2 HY1904C2, Q3 2N7002, Q4 HY1904C2, U1 SI5351A-B-GTR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

Commit message: Minor changes only
Parts:
- moved TP5 15.0 mm to (120.9, 155.0)
- moved TP7 12.9 mm to (135.8, 143.2)
- moved TP2 12.7 mm to (144.7, 129.7)
- moved TP8 11.7 mm to (139.7, 138.6)
- moved TP1 2.76 mm to (104.2, 161.7)
- moved TP15 0.69 mm to (110.1, 160.3)
Routing:
- net REVERSE-POWER: track 82.2 -> 94.8 mm
- net /VIN: track 23.9 -> 15.0 mm
- net FORWARD-POWER: track 94.6 -> 102.3 mm
- net 12V: track 145.3 -> 142.6 mm
Other:
- board text added: "COIL EXTRA CABLE LENGTH HERE AND ZIPTIE TO STANDOFF"
- board text added: "USB2 TYPE-A TO USB2 MINI TYPE-B CABLE"
- board text removed: "USB2 TYPE-A TO USB2-MINI CABLE"

Commit message: Minor silkscreen updates
Other:
- board text added: "USB CABLE ROUTE"
- board text added: "USB2 MINI TYPE-B"
- board text added: "USB2 TYPE-A"
- board text removed: "MCU USB"
- board text removed: "USB2 TYPE-A TO USB2 MINI TYPE-B CABLE"

Commit message: Updates
Parts:
- removed C14, C18: 470uF, Capacitor_SMD:C_Elec_10x10.2
- removed C23: 100nF, Capacitor_SMD:C_0805_2012Metric
- removed C25, C44, C45: 10uF, Capacitor_SMD:C_1206_3216Metric
- removed C30: 1nF, Capacitor_SMD:C_0805_2012Metric
- removed C31: 100pF, Capacitor_SMD:C_0603_1608Metric
- removed C33: 10pF, Capacitor_SMD:C_0603_1608Metric
- removed C34: 1pF, Capacitor_SMD:C_0402_1005Metric
- removed D11, D8: BZT52C5V6, Diode_SMD:D_SOD-123
- removed L4: 100uH, adxi-footprints:IND-SMD_L13.4-W12.6
- removed Q2, Q4: HY1904C2, adxi-footprints:DFN-8_L5.9-W5.2-P1.27-LS6.2-BL
- removed TP3: VIN-USBC, TestPoint:TestPoint_THTPad_2.0x2.0mm_Drill1.0mm
- added C22: 10uF, Capacitor_SMD:C_1206_3216Metric, F.Cu at (126.4, 114.4)
- added D7: 500mW 43V, Diode_SMD:D_SOD-123, F.Cu at (30.7, 107.0)
- added U11: SI2304DDS-T1-GE3, adxi-footprints:SOT-23-3_L2.9-W1.6-P1.90-LS2.8-BR, F.Cu at (131.0, 111.6)
- added U12: SI2304DDS-T1-GE3, adxi-footprints:SOT-23-3_L2.9-W1.6-P1.90-LS2.8-BR, F.Cu at (35.1, 109.3)
- C1, C5: footprint Capacitor_SMD:C_1206_3216Metric -> Capacitor_SMD:C_1210_3225Metric
- C12, C20, C8: value 470uF -> 1000uF
- C29: value 22nF -> 100nF; footprint Capacitor_SMD:C_1206_3216Metric -> Capacitor_SMD:C_0805_2012Metric
- D1, D3: value 1N4148WS -> 1N5711; footprint Diode_SMD:D_SOD-323 -> Diode_SMD:D_SOD-123
- D10: value BZT52C5V6 -> 500mW 43V
- J3, J5: moved to F.Cu
- J6: value RFC-GND -> RESERVED
- L226: footprint adxi-footprints:IND-SMD_L10.8-W10.0 -> Inductor_SMD:L_Changjiang_FNR4030S
- TP11: value RFC-GND -> GND
- TP12: value PA-SUPPLY -> L1-SUPPLY
- moved C29 83.1 mm to (111.2, 122.8), turned to 180 degrees
- moved J5 50.2 mm to (117.6, 147.2), turned to 135 degrees
- moved C8 31.3 mm to (103.8, 125.5), turned to 180 degrees
- moved TP13 28.3 mm to (123.0, 110.4), turned to 180 degrees
- moved TP11 24.2 mm to (126.3, 110.3)
- moved C20 18.2 mm to (103.8, 136.5), turned to 180 degrees
- moved TP5 14.7 mm to (133.1, 146.8)
- moved R98 10.6 mm to (88.6, 129.0), turned to 180 degrees
- moved R100 10.5 mm to (88.6, 125.6), turned to 0 degrees
- moved R99 10.0 mm to (88.6, 127.3), turned to 180 degrees
- moved C12 9.46 mm to (55.3, 116.2), turned to 90 degrees
- moved D26 9.01 mm to (67.1, 150.3), turned to 90 degrees
- moved D10 8.33 mm to (150.5, 110.9)
- moved D9 6.80 mm to (131.9, 116.6), turned to 90 degrees
- moved TP2 5.61 mm to (142.7, 134.9)
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Connections:
- net /Late Stage Interface/PA-SUPPLY renamed /Late Stage Interface/L1-SUPPLY
- C20 pad 1: /VIN-USBC -> 12V
- C29 pad 1: /Late Stage Interface/RFC-GND -> GND
- C29 pad 2: GND -> 12V
- D26 pad 1: /VIN-USBC -> /VIN
- J6 pad 1: /Late Stage Interface/RFC-GND -> GND
- J6 pad 2: /Late Stage Interface/RFC-GND -> GND
- J6 pad 3: /Late Stage Interface/RFC-GND -> GND
- J6 pad 4: /Late Stage Interface/RFC-GND -> GND
- R80 pad 2: /VIN-USBC -> /VIN
- TP11 pad 1: /Late Stage Interface/RFC-GND -> GND
Routing:
- net /VIN-USBC: track 152.1 -> 0.00 mm, vias 6 -> 0
- net /Late Stage Interface/RFC-GND: track 135.7 -> 0.00 mm
- net 12V: track 142.6 -> 59.6 mm, vias 7 -> 0
- net FORWARD-POWER: track 102.3 -> 41.6 mm, vias 3 -> 5
- net GND: track 181.9 -> 122.8 mm, vias 108 -> 83
- net /VIN: track 15.0 -> 72.4 mm, vias 0 -> 3
- net REVERSE-POWER: track 94.8 -> 44.5 mm, vias 2 -> 4
- net RECEIVED-SIGNAL: track 158.7 -> 118.1 mm, vias 1 -> 0
- net PA-DRIVE-PWM: track 105.2 -> 91.6 mm, vias 4 -> 3
- net SPI-SCK-3.3V: track 81.0 -> 68.1 mm
- net /Late Stage Interface/L1-SUPPLY: track 51.7 -> 62.5 mm
- net Net-(D9-K): track 15.4 -> 8.73 mm, vias 2 -> 0
- net I2C-SDA-3.3V: track 44.1 -> 37.7 mm
- net Net-(D5-K): track 67.3 -> 73.6 mm
- net SPI-SCK: track 2.75 -> 8.81 mm, vias 0 -> 1
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Other:
- outline, holes or cut-outs redrawn
- board text added: "1.2"
- board text added: "MECHANICAL FUNCTION: RESISTS INSERTION FORCES FOR ANTENNA CONNECTIONS MADE TO THE LATE STAGE MODULE WHICH IS PLUGGED IN ABOVE THIS BOARD."
- board text added: "RESERVED"
- board text added: "THIS IS THE CLASS-E POWER AMPLIFIER SWITCHED DRAIN FOR THE LATE STAGE MODULE POWER AMPLIFIER CIRCUITRY."
- board text added: "THIS IS THE DC FEED ORIGIN FOR THE LATE STAGE MODULE'S POWER AMPLIFIER CIRCUITRY."
- board text removed: "1.0"
- board text removed: "ANT"
- board text removed: "RFC-"
- board text removed: "RFC-GND"
- board text removed: "USBC VIN"

Commit message: final
Parts:
- moved TP2 11.6 mm to (147.5, 124.4)
- moved C12 4.31 mm to (55.6, 120.5)
- moved TP8 1.63 mm to (138.8, 140.0)
Routing:
- net USB-A-D-: track 40.6 -> 91.0 mm, vias 1 -> 2
- net USB-A-D+: track 41.9 -> 86.6 mm, vias 1 -> 2
- net GND: track 122.8 -> 161.4 mm, vias 83 -> 96
- net REVERSE-POWER: track 44.5 -> 82.6 mm, vias 4 -> 5
- net FORWARD-POWER: track 41.6 -> 75.8 mm, vias 5 -> 6
- net /VIN: track 72.4 -> 104.9 mm
- net PA-DRIVE-PWM: track 91.6 -> 66.2 mm, vias 3 -> 2
- net 12V: track 59.6 -> 83.6 mm, vias 0 -> 2
- net 5V: track 158.1 -> 179.7 mm, vias 6 -> 7
- net /Late Stage Interface/L1-SUPPLY: track 62.5 -> 56.5 mm
- net Net-(J3-D--PadA7): track 56.4 -> 53.6 mm, vias 4 -> 5
- net Net-(FB6-Pad1): track 13.1 -> 12.0 mm, vias 1 -> 0
- net Net-(J3-CC1): track 4.11 -> 3.28 mm, vias 1 -> 0
- net I2C-SCL-3.3V: track 45.2 -> 44.4 mm, vias 5 -> 4
- net Net-(J3-CC2): track 8.37 -> 7.58 mm, vias 1 -> 2
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Other:
- outline, holes or cut-outs redrawn
- board text added: "USB2 TYPE-A THROUGH TO MCU MODULE (MOUNTED BELOW)"
- board text removed: "USB2 TYPE-A"
