File: kicad-pcbs/adxi/pa-switched-resonator.kicad_sch (KiCad schematic)
At the start: 144 parts

Commit message: Rationalize
Parts:
- renumbered C30 to C36, C31 to C37, C32 to C38, C33 to C39, C34 to C40, C35 to C41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

Commit message: Update
Parts:
- renumbered C36 to C2, C37 to C3, C38 to C4, C39 to C6, C41 to C60, C42 to C61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
