File: kicad-pcbs/adxi/nfet-highside-load-switch.kicad_sch (KiCad schematic)
At the start: 7 parts, among them Q29 2N7002, Q30 HY1904C2

Commit message: Rationalize
Parts:
- renumbered D21 to D9, Q29 to Q3, Q30 to Q4, R68 to R16, R69 to R17, R70 to R18, R71 to R19

Commit message: More work, getting close now!
Parts:
- Q4: footprint kicad-parts:HY1904C2 -> kicad-6-parts:HY1904C2

Commit message: Simplify PSU, add 4xM3 mounting holes, silkscreen, better footprints
Parts:
- Q4: footprint kicad-6-parts:HY1904C2 -> adxi-footprints:DFN-8_L5.9-W5.2-P1.27-LS6.2-BL
Changed lines of the file:
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@@
 			)
 		)
-		(property "Footprint" "kicad-6-parts:HY1904C2"
+		(property "Footprint" "adxi-footprints:DFN-8_L5.9-W5.2-P1.27-LS6.2-BL"
 			(at 173.99 99.06 0)
 			(effects
