File: kicad-pcbs/adxi/nfet-highside-load-switch.kicad_sch (KiCad schematic)
At the start: 7 parts, among them Q3 2N7002, Q4 HY1904C2

Commit message: Fixed vias
Parts:
- Q3: LCSC Part # (none) -> C8545; MPN (none) -> 2N7002; Manufacturer (none) -> Changjing
Changed lines of the file:
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@@
 			)
 		)
-		(property "Description" ""
+		(property "Description" "60V 115mA 200mW 7.5Ω@10V,500mA 2.5V@250uA 1PCSNChannel SOT-23 MOSFETs ROHS"
 			(at 125.095 93.98 0)
 			(effects
+				(font
+					(size 1.27 1.27)
+				)
+				(hide yes)
+			)
+		)
+		(property "LCSC Part #" "C8545"
+			(at 125.095 93.98 0)
+			(effects
+				(font
+					(size 1.27 1.27)
+				)
+				(hide yes)
+			)
+		)
+		(property "MPN" "2N7002"
+			(at 125.095 93.98 0)
+			(effects
+				(font
+					(size 1.27 1.27)
+				)
+				(hide yes)
+			)
+		)
+		(property "Manufacturer" "Changjing"
+			(at 125.095 93.98 0)
+			(effects
