File: kicad-pcbs/adxi/late-stage-interface.kicad_sch (KiCad schematic)
At the start: 3 parts, among them J2 PA-SUPPLY, J4 PA-DRAIN, J6 RFC-GND

Commit message: Updates
Parts:
- J6: value RFC-GND -> RESERVED
Connections:
- net PA-SUPPLY renamed L1-SUPPLY
- net RFC-GND renamed GND
Other:
- note added: "THIS IS THE DC FEED ORIGIN FOR THE POWER AMPLIFIER CIRCUITRY."
- note added: "THIS IS THE MECHANICALLY SIGNIFICANT "THIRD LEG" OF THE LATE STAGE MODULE. IT IS IMPORTANT TO COUNTER THE FORCE OF THE ANTENNA INSERTION/REMOVAL. IN FUTURE SIGNALS MAY BE ADDED, FOR NOW ALL WILL BE LEFT AS GND TO REDUCE FLOATING CHARGES IN PROXIMITY TO THE POWER AMPLIFIER'S RESONATOR."
- note added: "THIS IS THE SIGNAL OUTPUT AND MOSFET DRAIN SWITCH INTERFACE."
