File: kicad-pcbs/adxi/spi-gpio-output.kicad_sch (KiCad schematic)
At the start: 2 parts, among them U5 74HC595

Commit message: USB work
Parts:
- renumbered U5 to U6
Changed lines of the file:
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@@
 			(project ""
 				(path "/c3abf330-1856-4368-a03b-0e6191ae29a9/78428e41-003b-411e-a951-46f73eeac9f7"
-					(reference "U?")
+					(reference "U5")
 					(unit 1)
 				)
@@
 		(on_board yes)
 		(dnp no)
-		(property "Reference" "U5"
+		(property "Reference" "U6"
 			(at 133.985 118.745 0)
 			(effects
@@
 			(project "adxi"
 				(path "/c3abf330-1856-4368-a03b-0e6191ae29a9/78428e41-003b-411e-a951-46f73eeac9f7"
-					(reference "U5")
+					(reference "U6")
 					(unit 1)
 				)

Commit message: Update
Parts:
- removed U6: 74HC595, Package_SO:SOIC-16_3.9x9.9mm_P1.27mm, symbol 74xx:74HC595
