File: kicad-pcbs/adxi-lsm-20m-30m-40m-1/adxi-lsm-20m-30m-40m-1.kicad_sch (KiCad schematic)
At the start: 54 parts, among them J1 ANT, J2 Conn_01x04, J3 Conn_01x04, J4 Conn_01x04

Commit message: 20m/30m/40m late stage module
Parts:
- added C1: 10pF, Capacitor_SMD:C_0603_1608Metric, symbol Device:C_Small
- added C10, C28, C31: 100pF, Capacitor_SMD:C_0805_2012Metric, symbol Device:C_Small
- added C15: 220pF, Capacitor_SMD:C_0805_2012Metric, symbol Device:C_Small
- added C26, C32: 470pF, Capacitor_SMD:C_0805_2012Metric, symbol Device:C_Small
- added C27: 1nF, Capacitor_SMD:C_1206_3216Metric, symbol Device:C_Small
- added C29: 12pF, Capacitor_SMD:C_0603_1608Metric, symbol Device:C_Small
- added C30: 68pF, Capacitor_SMD:C_0603_1608Metric, symbol Device:C_Small
- added C33, C9: 47pF, Capacitor_SMD:C_0805_2012Metric, symbol Device:C_Small
- added C5: 22pF, Capacitor_SMD:C_0805_2012Metric, symbol Device:C_Small
- added JP10: 100PF, Jumper:SolderJumper-2_P1.3mm_Open_RoundedPad1.0x1.5mm, symbol Jumper:SolderJumper_2_Open
- added JP11: 220PF, Jumper:SolderJumper-2_P1.3mm_Open_RoundedPad1.0x1.5mm, symbol Jumper:SolderJumper_2_Open
- added JP12: 470PF, Jumper:SolderJumper-2_P1.3mm_Open_RoundedPad1.0x1.5mm, symbol Jumper:SolderJumper_2_Open
- added JP13: 1NF, Jumper:SolderJumper-2_P1.3mm_Open_RoundedPad1.0x1.5mm, symbol Jumper:SolderJumper_2_Open
- added JP14: 0.15UH, Jumper:SolderJumper-2_P1.3mm_Open_RoundedPad1.0x1.5mm, symbol Jumper:SolderJumper_2_Open
- added JP15: 0.22UH, Jumper:SolderJumper-2_P1.3mm_Open_RoundedPad1.0x1.5mm, symbol Jumper:SolderJumper_2_Open
- added JP16: 0.47UH, Jumper:SolderJumper-2_P1.3mm_Open_RoundedPad1.0x1.5mm, symbol Jumper:SolderJumper_2_Open
- added JP17: 0.94UH, Connector_PinHeader_1.00mm:PinHeader_1x03_P1.00mm_Vertical, symbol Connector_Generic:Conn_01x03
- added JP18: 2.2UH, Connector_PinHeader_1.00mm:PinHeader_1x03_P1.00mm_Vertical, symbol Connector_Generic:Conn_01x03
- added JP19: 9.27UH, Connector_PinHeader_1.00mm:PinHeader_1x03_P1.00mm_Vertical, symbol Connector_Generic:Conn_01x03
- added JP20: 40M, Jumper:SolderJumper-2_P1.3mm_Open_RoundedPad1.0x1.5mm, symbol Jumper:SolderJumper_2_Open
- added JP21: 0.94UH., Jumper:SolderJumper-2_P1.3mm_Open_RoundedPad1.0x1.5mm, symbol Jumper:SolderJumper_2_Open
- added JP22: 2.2UH., Jumper:SolderJumper-2_P1.3mm_Open_RoundedPad1.0x1.5mm, symbol Jumper:SolderJumper_2_Open
- added JP23: 4.7UH., Jumper:SolderJumper-2_P1.3mm_Open_RoundedPad1.0x1.5mm, symbol Jumper:SolderJumper_2_Open
- added JP24: 9.27UH., Jumper:SolderJumper-2_P1.3mm_Open_RoundedPad1.0x1.5mm, symbol Jumper:SolderJumper_2_Open
- added JP25: 4.7UH, Connector_PinHeader_1.00mm:PinHeader_1x03_P1.00mm_Vertical, symbol Connector_Generic:Conn_01x03
- added JP26: 30M, Jumper:SolderJumper-2_P1.3mm_Open_RoundedPad1.0x1.5mm, symbol Jumper:SolderJumper_2_Open
- added JP27: 20M, Jumper:SolderJumper-2_P1.3mm_Open_RoundedPad1.0x1.5mm, symbol Jumper:SolderJumper_2_Open
- added JP7: 10PF, Jumper:SolderJumper-2_P1.3mm_Open_RoundedPad1.0x1.5mm, symbol Jumper:SolderJumper_2_Open
- added JP8: 22PF, Jumper:SolderJumper-2_P1.3mm_Open_RoundedPad1.0x1.5mm, symbol Jumper:SolderJumper_2_Open
- added JP9: 47PF, Jumper:SolderJumper-2_P1.3mm_Open_RoundedPad1.0x1.5mm, symbol Jumper:SolderJumper_2_Open
- added L25, L26, L27, L28, L29, L30, L31, L32, L33, L34, L35, L36, L37, L38, L39, L40, L41, L42, L43, L44, L45, L46, L47, L48, L49, L50, L51, L52, L53, L54, L55, L56, L57, L58, L61, L62, L63, L67, L72: 470nH, Inductor_SMD:L_1008_2520Metric, symbol Device:L
- added L59, L60: 220nH, Inductor_SMD:L_0805_2012Metric, symbol Device:L
- added L64, L65, L66, L68, L69, L70, L71: 2.2uH, adxi-footprints:L_Chilisin_NLC252018-2.92x2.50x2.20, symbol Device:L
- J2: value Conn_01x04 -> PA-DRAIN; footprint Connector_PinHeader_2.54mm:PinHeader_1x04_P2.54mm_Vertical -> Connector_PinSocket_2.54mm:PinSocket_1x04_P2.54mm_Vertical
- J3: value Conn_01x04 -> PA-SUPPLY; footprint Connector_PinHeader_2.54mm:PinHeader_1x04_P2.54mm_Vertical -> Connector_PinSocket_2.54mm:PinSocket_1x04_P2.54mm_Vertical
- J4: value Conn_01x04 -> RFC-GND; footprint Connector_PinHeader_2.54mm:PinHeader_1x04_P2.54mm_Vertical -> Connector_PinSocket_2.54mm:PinSocket_1x04_P2.54mm_Vertical
Connections:
- net GND: now also C1.2, C10.2, C15.2, C26.2, C27.2, C28.2, C29.2, C32.2, C33.2, C5.2, C9.2, L57.2, L58.2, L59.2, L60.2, L61.2
- net at J3.1 (Pin_1), J3.2 (Pin_2), J3.3 (Pin_3)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: now also JP20.2 (B), JP26.2 (B), JP27.2 (B), L25.1
- net at J2.1 (Pin_1), J2.2 (Pin_2), J2.3 (Pin_3)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: now also JP19.3 (Pin_3), JP24.2 (B); no longer J1.2 (Ext)
- new net: L50.2, L51.1
- new net: L51.2, L52.1
- new net: L45.2, L46.1
- new net: L46.2, L47.1
- new net: JP22.1 (A), L64.2
- new net: JP18.3 (Pin_3), JP22.2 (B), JP25.2 (Pin_2)
- new net: C29.1, C33.1, JP26.1 (A)
- new net: C26.1, JP12.2 (B)
- new net: L44.2, L45.1
- new net: C15.1, JP11.2 (B)
- new net: JP25.1 (Pin_1), L65.1, L67.1
- new net: JP19.2 (Pin_2), JP23.2 (B), JP25.3 (Pin_3)
- new net: JP19.1 (Pin_1), L68.1
- new net: L54.2, L55.1
- new net: L55.2, L56.1
- new net: L29.2, L30.1
- new net: L30.2, L31.1
- new net: J1.2 (Ext), JP10.1 (A), JP11.1 (A), JP12.1 (A), JP13.1 (A), JP14.1 (A), JP15.1 (A), JP16.1 (A), JP17.2 (Pin_2), JP7.1 (A), JP8.1 (A), JP9.1 (A)
- new net: C1.1, JP7.2 (B)
- new net: L69.2, L70.1
- new net: L70.2, L71.1
- new net: JP18.1 (Pin_1), L64.1
- new net: JP17.3 (Pin_3), JP18.2 (Pin_2), JP21.2 (B)
- new net: L34.2, L35.1
- new net: L35.2, L36.1
- new net: L48.2, L49.1
- new net: L49.2, L50.1
- new net: L68.2, L69.1
- new net: L56.2, L57.1
- new net: JP17.1 (Pin_1), L62.1
- new net: L62.2, L63.1
- new net: L65.2, L66.1
- new net: L42.2, L43.1
- new net: L43.2, L44.1
- new net: JP14.2 (B), L58.1, L59.1
- new net: L47.2, L48.1
- new net: L52.2, L53.1
- new net: L53.2, L54.1
- new net: C5.1, JP8.2 (B)
- new net: JP23.1 (A), L66.2, L67.2
- new net: L26.2, L27.1
- new net: L27.2, L28.1
- new net: C9.1, JP9.2 (B)
- new net: JP16.2 (B), L61.1
- new net: C31.2, C32.1
- new net: JP24.1 (A), L72.2
- new net: C31.1, JP20.1 (A)
- new net: C10.1, JP10.2 (B)
- new net: C27.1, JP13.2 (B)
- new net: L31.2, L32.1
- new net: L32.2, L33.1
- new net: L25.2, L26.1
- new net: C28.1, C30.2
- new net: C30.1, JP27.1 (A)
- new net: L28.2, L29.1
- new net: L36.2, L37.1
- new net: L37.2, L38.1
- new net: L39.2, L40.1
- new net: L40.2, L41.1
- new net: L41.2, L42.1
- new net: JP21.1 (A), L63.2
- new net: L38.2, L39.1
- new net: L33.2, L34.1
- new net: JP15.2 (B), L60.1
- new net: L71.2, L72.1
Other:
- note added: "2x (33 x 0.47uH = 15.51uH @ 1.188Ω) = 7.755μH @ 0.594Ω SRF=170MHz I>3A"
- note added: "=40.5pF"
- note added: "=59pF"
- note added: "=82.46pF"
- note added: "ANTENNA TUNING UNIT"
- note added: "C1 = 0.1836 ÷ (2π⋅f⋅R) where: f = Frequency (Hz) R = Resistance (Ω) - usually 50 20m (14MHz) = 41.8pF (we use 40.5pF) 30m (10MHz) = 58.5pF (we use 59pF) 40m (7MHz) = 83.6pF (we use 82.46pF)"
- note added: "C1 CAP"
- note added: "CAPACITANCE"
- note added: "INDUCTANCE"
- note added: "LARGE VALUES ARE IN SERIES."
- note added: "PARALELL ENABLE/DISABLE."
- note added: "RF CHOKE"
- note added: "SMALL VALUES ARE IN PARALLEL."
- note added: "SOKAL 'C1'"
- note added: "SOKAL 'C2'"
- note added: "SOKAL 'L1'"
- note added: "SOKAL 'L2'"
- note removed: "LPF CAPACITANCE"
- note removed: "LPF INDUCTANCE"
- note removed: "MISSING BITS: INTER-BOARD CONNECTORS, RF CHOKE = ?"
- moved on the sheet: C11, C12, C13, C14, C16, C17, C18, C19, C2, C20, C21, C22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

Commit message: Updates
Parts:
- removed C29: 12pF, Capacitor_SMD:C_0603_1608Metric, symbol Device:C_Small
- added C34: 20pF, Capacitor_SMD:C_1206_3216Metric, symbol Device:C_Small
- added JP28: 20M-D, Jumper:SolderJumper-2_P1.3mm_Open_RoundedPad1.0x1.5mm, symbol Jumper:SolderJumper_2_Open
- added JP29: 30M-D, Jumper:SolderJumper-2_P1.3mm_Open_RoundedPad1.0x1.5mm, symbol Jumper:SolderJumper_2_Open
- added JP30: 40M-D, Jumper:SolderJumper-2_P1.3mm_Open_RoundedPad1.0x1.5mm, symbol Jumper:SolderJumper_2_Open
- added JP31: 20M-A, Jumper:SolderJumper-2_P1.3mm_Open_RoundedPad1.0x1.5mm, symbol Jumper:SolderJumper_2_Open
- added JP32: 30M-A, Jumper:SolderJumper-2_P1.3mm_Open_RoundedPad1.0x1.5mm, symbol Jumper:SolderJumper_2_Open
- added JP33: 40M-A, Jumper:SolderJumper-2_P1.3mm_Open_RoundedPad1.0x1.5mm, symbol Jumper:SolderJumper_2_Open
- added JP34: 20M-E, Jumper:SolderJumper-2_P1.3mm_Open_RoundedPad1.0x1.5mm, symbol Jumper:SolderJumper_2_Open
- added JP35: 30M-E, Jumper:SolderJumper-2_P1.3mm_Open_RoundedPad1.0x1.5mm, symbol Jumper:SolderJumper_2_Open
- added JP36: 40M-E, Jumper:SolderJumper-2_P1.3mm_Open_RoundedPad1.0x1.5mm, symbol Jumper:SolderJumper_2_Open
- C1: footprint Capacitor_SMD:C_0603_1608Metric -> Capacitor_SMD:C_1206_3216Metric; LCSC Part # C1634 -> C377014; MPN CL10C100JB8NNNC -> TCC1206COG100J102DT; Manufacturer Samsung -> CCTC
- C5: value 22pF -> 12pF; footprint Capacitor_SMD:C_0805_2012Metric -> Capacitor_SMD:C_1206_3216Metric; LCSC Part # C1804 -> C1886; MPN CL21C220JBANNNC -> 1206CG120J500NT; Manufacturer Samsung -> Fenghua
- J4: value RFC-GND -> C1-GND
- JP1: value 20M-A -> 20M-F
- JP2: value 30M-A -> 30M-F
- JP20: value 40M -> 40M-C
- JP26: value 30M -> 30M-C
- JP27: value 20M -> 20M-C
- JP3: value 40M-A -> 40M-F
- JP6: value 40M-C -> 40M-B
- JP8: value 22PF -> 20PF
Connections:
- net GND: now also C34.1, JP28.1 (A), JP29.1 (A), JP30.1 (A); no longer C2.2, C28.2, C32.2, C33.2, C4.2, C5.2, C6.2, C8.2, L57.2
- net at JP1.1 (A), JP2.1 (A), JP3.1 (A): now also L1.1, L6.1; no longer L16.2, L21.2
- net at JP1.2 (B): now also C7.2; no longer C7.1
- net at C33.1, JP26.1 (A): now also C5.2
- net at L22.1: now also JP31.2 (B); no longer C7.2
- net at J3.1 (Pin_1), J3.2 (Pin_2), J3.3 (Pin_3)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: no longer JP20.2 (B), JP26.2 (B), JP27.2 (B), L1.1, L6.1
- net at C5.1: now also C33.2, JP29.2 (B); no longer JP8.2 (B)
- net at C14.1: now also JP36.2 (B); no longer JP3.2 (B)
- net at C14.2: now also JP3.2 (B); no longer L11.1
- net at C11.1: now also JP35.2 (B); no longer JP2.2 (B)
- net at L23.1, L24.1: now also JP32.2 (B); no longer C13.2
- new net: C2.2, C4.2, C6.2, C8.2
- new net: JP31.1 (A), JP32.1 (A), JP33.1 (A), L16.2, L21.2
- new net: C7.1, JP34.2 (B)
- new net: C28.2, JP28.2 (B)
- new net: JP20.2 (B), JP26.2 (B), JP27.2 (B), JP34.1 (A), JP35.1 (A), JP36.1 (A), L57.2
- new net: C34.2, JP8.2 (B)
- new net: C32.2, JP30.2 (B)
- new net: C13.2, JP2.2 (B)
- new net: JP33.2 (B), L11.1
Other:
- note added: "2% SRF=450MHz Q=45 DCR=1.19Ω I=470mA"
- note added: "5% SRF=140MHz Q=25 DCR=0.5Ω I=1200mA"
- note added: "5% SRF=850MHz Q=40 DCR=1.05Ω÷2=0.525Ω I=400mA×2=800mA"
- note removed: "2% SRF=450MHz DCR=1.19 Q=45 I=470mA"
- note removed: "5% SRF=140MHz RDC=0.5 I=1200mA Q=25"
- moved on the sheet: C10, C11, C12, C13, C14, C15, C16, C17, C18, C19, C2, C20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
