File: kicad-pcbs/adxi-lsm-20m-30m-40m-2/adxi-lsm-20m-30m-40m-2.kicad_sch (KiCad schematic)
At the start: 121 parts, among them J1 ANT, J2 PA-DRAIN, J3 PA-SUPPLY, J4 C1-GND

Commit message: Final board
Parts:
- removed L10, L12, L13, L14, L15, L16, L17, L18, L19, L20, L21, L5, L6, L7, L73, L74, L75, L8, L9: 6.8uH, Inductor_SMD:L_0805_2012Metric, symbol Device:L
- removed L27, L28, L29, L30, L31, L32, L33, L34, L35, L36, L37, L38, L39, L40, L41, L42, L43, L44, L45, L46, L47, L48, L49, L50, L51, L52, L53, L54, L55, L56, L57: 470nH, Inductor_SMD:L_1008_2520Metric, symbol Device:L
- removed L76: 5.6uH, Inductor_SMD:L_0805_2012Metric, symbol Device:L
- removed L86, L87, L89: 680nH, Inductor_SMD:L_0603_1608Metric, symbol Device:L
- added L24, L58, L59, L60, L61, L62, L63, L64, L65, L66, L67, L68: 680nH, Inductor_SMD:L_0603_1608Metric, symbol Device:L
- added L69, L70: 2.2uH, Inductor_SMD:L_0603_1608Metric, symbol Device:L
- L25, L26: value 470nH -> 3.9uH; footprint Inductor_SMD:L_1008_2520Metric -> Inductor_SMD:L_1812_4532Metric; LCSC Part # C316369 -> C394117; MPN SPH252012HR47MT -> FHW1812IF3R9JST; Manufacturer Sunlord -> Fenghua
- L3, L4: value 6.8uH -> 22uH; footprint Inductor_SMD:L_0805_2012Metric -> Inductor_SMD:L_Sunlord_SWPA3015S; LCSC Part # C223247 -> C83438; MPN LB2012T6R8M -> SWPA3015S220MT; Manufacturer Taiyo-Yuden -> Sunlord
Connections:
- net at C41.1, L93.1: now also L24.2, L59.2, L69.2, L70.2; no longer L11.2, L23.2
- net at C20.1, L84.2: now also L60.1, L61.1
- net at C37.1, JP5.1 (A): now also L67.2, L68.2
- net at L3.1: now also C12.2, C33.2
- net at C21.1, L88.1: now also L62.2, L63.2
- net at C36.1, L88.2: now also L64.1, L66.1
- net at C38.1, L11.1, L23.1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: now also L58.1, L65.1
- net at L85.1: now also L4.2
- net at JP20.2 (B), JP26.2 (B), JP27.2 (B)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: now also L26.2
- new net: L58.2, L59.1
- new net: L64.2, L67.1
- new net: L60.2, L62.1
- new net: L11.2, L69.1
- new net: L23.2, L70.1
- new net: L61.2, L63.1
- new net: L66.2, L68.1
- new net: L24.1, L65.2
Other:
- note added: "$0.10 SRF>23MHz / 1.3Ω / 520mA"
- note added: "$0.21 7.8uH SRF 135MHz / 2x0.6=1.2Ω / 750mA"
- note added: "20m 30m 40m SOLDER SELECTABLE LATE STAGE MODULE (CLASS E PA + LOW PASS FILTER)"
- note added: "5.95% error, 4 parts L_match: 0.519µH (0.68µH || 2.2µH) Series-parallel are for higher current. C_match: 680pF (680pF)"
- note added: "7th order Butterworth approximation (12.62% error, 7 parts): C1_lpf=100pF L1_lpf=0.68µH C2_lpf=330pF L2_lpf=1µH C3_lpf=330pF L3_lpf=0.68µH C4_lpf=100pF Series-parallel are for higher current."
- note added: "Class E Power Amplifier (PA) and low pass filter module schematic component specifications were generated using https://github.com/vk2diy/classe2-calculator $ ./classe2 -p 5 -v 12 -b 20m 30m 40m -q 40 -t infinite --l1 7.755uh -m SI2304DDS ..."
- note added: "RF choke configuration was regenerated using https://github.com/vk2diy/classe2-calculator from after a previous inefficient (high SRF target) design was discarded. This approach saved reconfiguration/respecification of all other components. $ ./classe2 --equivalent-inductor 7.755uh -b 20m 30m 40m --equivalent-inductor-max-components 3 --equivalent-inductor-max-configurations 15 Configurations for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"
- note added: "VK2DIY"
- note removed: "$0.02 SRF>32MHz 0.5Ω 250mA"
- note removed: "$0.04 SRF>38MHz 0.47Ω 135mA"
- note removed: "$0.78 SRF>~18MHz / 3.32Ω / 470mA"
- note removed: "2x (33 x 0.47uH = 15.51uH @ 1.188Ω) = 7.755μH @ 0.594Ω SRF=170MHz I>3A"
- note removed: "5.95% error, 4 parts L_match: 0.519µH (0.68µH || 2.2µH) This was made 2.2µH || 2.2µH for higher current. C_match: 680pF (680pF)"
- note removed: "7th order Butterworth approximation (12.62% error, 7 parts): C1_lpf=100pF L1_lpf=0.68µH C2_lpf=330pF L2_lpf=1µH C3_lpf=330pF L3_lpf=0.68µH C4_lpf=100pF"
- moved on the sheet: C11, C12, C13, C14, C16, C17, C18, C19, C20, C21, C28, C29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

Commit message: Fix 150pF 0603 footprint incorrectly specified as 0201
Parts:
- C29, C41, C42: footprint Capacitor_SMD:C_0201_0603Metric -> Capacitor_SMD:C_0603_1608Metric
Changed lines of the file:
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@@
 			)
 		)
-		(property "Footprint" "Capacitor_SMD:C_0201_0603Metric"
+		(property "Footprint" "Capacitor_SMD:C_0603_1608Metric"
 			(at 389.89 207.01 0)
 			(effects
@@
 			)
 		)
-		(property "Footprint" "Capacitor_SMD:C_0201_0603Metric"
+		(property "Footprint" "Capacitor_SMD:C_0603_1608Metric"
 			(at 148.59 231.14 0)
 			(effects
@@
 			)
 		)
-		(property "Footprint" "Capacitor_SMD:C_0201_0603Metric"
+		(property "Footprint" "Capacitor_SMD:C_0603_1608Metric"
 			(at 427.99 207.01 0)
 			(effects
