File: kicad-pcbs/ADX/ADX.kicad_pcb (KiCad board)
At the start: 2 copper layers, 97.1 x 97 mm, 82 parts, among them CON1 SPK, CON2 MIC, J1 SMA, J1A1 BNC, J2 PJ-102A, Q1 BS170, Q2 BS170, Q3 BS170, Q4 BS170, SW1 UP(BAND)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

Commit message: Commit outstanding files related to Kicad v8 updates
Other:
- net class Default removed
